File: OBC-Attempt-1/OBC-Attempt-1.kicad_pcb (KiCad board)
At the start: 4 copper layers, 76 parts, among them J1 Screw_Terminal_01x08, J2 Screw_Terminal_01x08, J3 USB_B_Micro, J4 Screw_Terminal_01x08, J5 Conn_01x04, J6 Micro_SD_Card, J7 Screw_Terminal_01x02, J8 Screw_Terminal_01x02, Q1 2N7002K, Q2 2N7002K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

Commit message: Basic Pcb layout
Parts:
- moved J2 130.2 mm to (210.7, 147.1), turned to 90 degrees
- moved J7 113.4 mm to (207.5, 32.2), turned to 90 degrees
- moved J6 94.9 mm to (210.9, 80.8), turned to -90 degrees
- moved U9 87.4 mm to (166.5, 80.2), turned to -45 degrees
- moved J4 78.9 mm to (186.9, 29.6), turned to 180 degrees
- moved U1 77.2 mm to (147.7, 82.0)
- moved J3 71.2 mm to (205.9, 63.1), turned to 90 degrees
- moved J1 63.3 mm to (140.0, 113.3), turned to -90 degrees
- moved J5 52.6 mm to (65.7, 66.1)
- moved BZ1 51.8 mm to (179.2, 81.4)
- moved U6 49.0 mm to (193.2, 68.2), turned to 180 degrees
- moved U12 48.4 mm to (190.1, 53.5), turned to 180 degrees
- moved SW1 47.0 mm to (186.3, 103.0), turned to 90 degrees
- moved C16 46.6 mm to (143.6, 77.1)
- moved C17 46.6 mm to (111.2, 109.1)
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Connections:
- J7 pad 1: GND -> BATT+
- J7 pad 2: BATT+ -> GND
- J8 pad 1: BATT+ -> PWR
- J8 pad 2: PWR -> BATT+
Routing:
- net BATT+: track 0.00 -> 24.3 mm

Commit message: PCB work
Parts:
- removed C14: 100nF, Capacitor_SMD:C_01005_0402Metric
- moved J2 137.4 mm to (75.9, 120.4), turned to -90 degrees
- moved J4 133.8 mm to (163.7, 161.3), turned to 90 degrees
- moved SW1 92.0 mm to (101.1, 68.1), turned to -90 degrees
- moved D7 83.6 mm to (150.5, 159.3), turned to -90 degrees
- moved J1 77.9 mm to (128.1, 36.4), turned to 180 degrees
- moved D5 75.7 mm to (150.5, 146.7), turned to -90 degrees
- moved D2 75.2 mm to (87.7, 154.2), turned to 90 degrees
- moved BZ1 74.0 mm to (107.1, 98.1), turned to -135 degrees
- moved U3 72.6 mm to (102.7, 145.8), turned to 90 degrees
- moved Q4 72.0 mm to (124.2, 52.4), turned to -90 degrees
- moved J5 72.0 mm to (133.0, 91.6), turned to 180 degrees
- moved D3 69.6 mm to (87.7, 131.4), turned to 90 degrees
- moved Q3 69.3 mm to (114.0, 52.5), turned to -90 degrees
- moved R18 68.7 mm to (149.6, 62.7), turned to -135 degrees
- moved R5 68.1 mm to (97.6, 53.3), turned to 90 degrees
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Connections:
- J2 pad 5: Net-(D4-Pad1) -> GND
- J2 pad 6: GND -> Net-(D4-Pad1)
- J2 pad 7: Net-(D2-Pad1) -> GND
- J2 pad 8: GND -> Net-(D2-Pad1)
- J4 pad 5: Net-(D6-Pad1) -> GND
- J4 pad 6: GND -> Net-(D6-Pad1)
- J4 pad 7: Net-(D8-Pad1) -> GND
- J4 pad 8: GND -> Net-(D8-Pad1)
- U9 pad 21: unconnected-(U9-Pad21) -> BUZZER
- U9 pad 50: BUZZER -> unconnected-(U9-Pad50)
Routing:
- net BATT+: track 24.3 -> 0.00 mm

Commit message: PCB Layout
Parts:
- moved R14 9.18 mm to (127.0, 148.7), turned to 180 degrees
- moved D2 9.18 mm to (87.7, 145.1)
- moved D4 9.18 mm to (87.6, 134.0)
- moved D5 9.18 mm to (150.5, 137.5)
- moved D7 9.18 mm to (150.5, 150.2)
- moved R11 9.18 mm to (111.9, 113.2)
- moved R16 9.18 mm to (126.8, 136.4)
- moved R17 9.18 mm to (126.0, 124.8)
- moved U2 9.18 mm to (103.0, 122.4)
- moved U3 9.18 mm to (102.7, 136.6)
- moved U5 9.18 mm to (102.8, 147.4)
- moved U7 9.18 mm to (135.8, 150.3)
- moved U8 9.18 mm to (135.4, 114.1)
- moved D1 9.17 mm to (87.6, 111.2)
- moved D3 9.17 mm to (87.7, 122.2)
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Routing:
- net PWR: track 0.00 -> 87.5 mm
- net BATT+: track 0.00 -> 7.18 mm
- added copper zone on In1.Cu, net GND

Commit message: More PCB Work Might restart wiring
Parts:
- moved SW1 32.4 mm to (132.6, 75.9), turned to 135 degrees
- moved D2 8.91 mm to (88.1, 154.0)
- moved D4 8.91 mm to (88.0, 142.9)
- moved D1 8.91 mm to (87.9, 120.1)
- moved D3 8.91 mm to (88.0, 131.1)
- moved R6 3.51 mm to (107.2, 56.8), turned to 0 degrees
- moved R8 3.49 mm to (127.4, 56.5), turned to 0 degrees
- moved R5 3.39 mm to (97.3, 56.6), turned to 0 degrees
- moved R7 3.31 mm to (116.7, 56.6), turned to 0 degrees
- moved D7 3.17 mm to (148.1, 152.2)
- moved D5 3.17 mm to (148.0, 139.5)
- moved D6 3.17 mm to (148.0, 128.4)
- moved D8 3.17 mm to (148.3, 116.1)
- moved C7 2.36 mm to (115.8, 97.2), turned to 0 degrees
- moved U1 2.07 mm to (118.8, 68.7)
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Routing:
- net PWR: track 87.5 -> 2.96 mm
- net SOL4: track 0.00 -> 56.5 mm
- net SOL3: track 0.00 -> 45.7 mm
- net SOL2: track 0.00 -> 31.5 mm
- net SOL1: track 0.00 -> 21.2 mm
- net 3.3V: track 0.00 -> 21.0 mm, vias 0 -> 2
- net GND: track 0.00 -> 20.5 mm, vias 0 -> 2
- net SYS_JTMS-SWDIO: track 0.00 -> 14.3 mm
- net SYS_JTCK_SWCLK: track 0.00 -> 12.4 mm
- net Net-(J1-Pad4): track 0.00 -> 8.47 mm
- net Net-(J1-Pad2): track 0.00 -> 8.40 mm
- net Net-(J1-Pad6): track 0.00 -> 8.20 mm
- net Net-(J1-Pad8): track 0.00 -> 8.02 mm
- net BATT+: track 7.18 -> 0.00 mm
- net Net-(Q1-Pad2): track 0.00 -> 7.06 mm
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- removed copper zone on In1.Cu, net GND

Commit message: Restart PCBdesign
Why why why why why
Parts:
- removed the C18 at (90.5, 91.0)
- added C14: 26pf, Capacitor_SMD:C_01005_0402Metric, F.Cu at (63.3, 44.0)
- added C18: 20pf, Capacitor_SMD:C_0201_0603Metric, F.Cu at (187.4, 77.2)
- added C18: 26uf, Capacitor_SMD:C_01005_0402Metric, F.Cu at (62.4, 45.0)
- C16: value 15pf -> 26pf; footprint Capacitor_SMD:C_0201_0603Metric -> Capacitor_SMD:C_01005_0402Metric
- C17: value 15pf -> 26uf; footprint Capacitor_SMD:C_0201_0603Metric -> Capacitor_SMD:C_01005_0402Metric
- Y1: value 32.768kHz -> ABMM2-25MHZ-D1-T; footprint Crystal:Crystal_HC49-4H_Vertical -> ABMM2_6mm_3_6mm:XTAL_ABMM2-25.000MHZ-D1-T
- Y2: value 25MHz -> ABMM2-32.768MHZ-E2F-T; footprint Crystal:Crystal_HC49-4H_Vertical -> ABMM2_6mm_3_6mm:XTAL_ABMM2-32.768MHZ-E2F-T
- moved J4 107.8 mm to (116.1, 58.7), turned to 0 degrees
- moved D3 106.9 mm to (174.5, 68.2), turned to 0 degrees
- moved U4 105.1 mm to (198.5, 68.2), turned to 0 degrees
- moved R6 102.9 mm to (209.9, 62.4)
- moved U3 101.1 mm to (183.6, 76.0), turned to 0 degrees
- moved R4 97.3 mm to (182.2, 82.6), turned to 0 degrees
- moved U1 96.5 mm to (214.4, 56.0), turned to 0 degrees
- moved D2 95.6 mm to (148.7, 80.0), turned to 0 degrees
- moved R2 95.3 mm to (193.8, 73.1), turned to 0 degrees
- moved R9 91.7 mm to (188.2, 73.3)
- moved C7 91.5 mm to (202.2, 66.8)
- moved C15 90.8 mm to (202.2, 65.1)
- moved R5 90.7 mm to (184.7, 80.8)
- moved U2 84.7 mm to (178.4, 83.9), turned to 0 degrees
- moved R12 81.1 mm to (167.0, 90.3)
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Connections:
- C16 pad 1: RCC_OSC32_OUT -> RCC_OSC_IN
- C17 pad 1: RCC_OSC32_IN -> RCC_OSC_OUT
- Y1 pad 1: RCC_OSC32_OUT -> RCC_OSC_IN
- Y1 pad 2: RCC_OSC32_IN -> GND
- Y2 pad 1: RCC_OSC_IN -> RCC_OSC32_IN
- Y2 pad 2: RCC_OSC_OUT -> GND
Routing:
- net SOL4: track 56.5 -> 0.00 mm
- net SOL3: track 45.7 -> 0.00 mm
- net SOL2: track 31.5 -> 0.00 mm
- net GND: track 20.5 -> 48.9 mm, vias 2 -> 0
- net SOL1: track 21.2 -> 0.00 mm
- net 3.3V: track 21.0 -> 0.00 mm, vias 2 -> 0
- net SYS_JTMS-SWDIO: track 14.3 -> 0.00 mm
- net SYS_JTCK_SWCLK: track 12.4 -> 0.00 mm
- net RCC_OSC_IN: track 0.00 -> 11.9 mm
- net RCC_OSC_OUT: track 0.00 -> 10.9 mm
- net RCC_OSC32_IN: track 0.00 -> 10.9 mm
- net Net-(J1-Pad4): track 8.47 -> 0.00 mm
- net Net-(J1-Pad2): track 8.40 -> 0.00 mm
- net Net-(J1-Pad6): track 8.20 -> 0.00 mm
- net Net-(J1-Pad8): track 8.02 -> 0.00 mm
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
Commit message: More work
Parts:
- C12, C5, J3, U6: moved to B.Cu
- moved R6 123.9 mm to (90.0, 31.3)
- moved C19 116.8 mm to (51.8, 70.9)
- moved D2 116.8 mm to (36.5, 47.5)
- moved D3 116.8 mm to (62.3, 35.7)
- moved D5 116.8 mm to (36.5, 55.3)
- moved D6 116.8 mm to (73.1, 35.7)
- moved J2 116.8 mm to (3.89, 38.0)
- moved J4 116.8 mm to (3.89, 26.2)
- moved Q1 116.8 mm to (30.4, 75.8)
- moved Q4 116.8 mm to (19.5, 77.2)
- moved R1 116.8 mm to (77.7, 42.9)
- moved R10 116.8 mm to (19.6, 58.5)
- moved R12 116.8 mm to (54.8, 57.8)
- moved R16 116.8 mm to (54.8, 55.2)
- moved R18 116.8 mm to (26.8, 58.1)
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Routing:
- net SDIO_CMD: track 0.00 -> 34.0 mm
- net SDIO_D3: track 0.00 -> 30.3 mm
- net SDIO_D0: track 0.00 -> 29.8 mm
- net SDIO_CK: track 0.00 -> 26.7 mm
- net SDIO_D1: track 0.00 -> 25.6 mm
- net SDIO_D2: track 0.00 -> 24.2 mm
- net BATT+: track 0.00 -> 17.3 mm
- net Net-(C5-Pad1): track 0.00 -> 9.08 mm
- net SYS_JTCK_SWCLK: track 0.00 -> 8.37 mm
- net SYS_JTMS-SWDIO: track 0.00 -> 8.16 mm
- net Net-(R13-Pad2): track 0.00 -> 8.01 mm
- net GND: track 48.9 -> 55.0 mm
- net 3.3V: track 0.00 -> 4.40 mm
- net USB_OTG_FS_ID: track 0.00 -> 2.72 mm, vias 0 -> 1
- net Net-(C11-Pad1): track 0.00 -> 2.45 mm
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
Commit message: PCB Work
Parts:
- removed the C18 at (75.2, 44.7)
- removed C19: 20pf, Capacitor_SMD:C_0201_0603Metric
- moved R18 145.6 mm to (172.3, 52.4), turned to 180 degrees
- moved Q4 135.1 mm to (150.4, 43.7), turned to -90 degrees
- moved Q3 120.9 mm to (140.6, 43.7), turned to -90 degrees
- moved R19 111.2 mm to (169.1, 52.4), turned to 180 degrees
- moved U12 111.0 mm to (162.3, 49.1), turned to 180 degrees
- moved BZ1 109.7 mm to (127.5, 75.0), turned to 180 degrees
- moved C20 98.8 mm to (168.9, 47.2), turned to -90 degrees
- moved Q1 95.7 mm to (120.4, 43.2), turned to -90 degrees
- moved C21 92.3 mm to (155.9, 49.6), turned to -90 degrees
- moved R3 88.1 mm to (139.7, 39.2), turned to 90 degrees
- moved R7 83.0 mm to (143.5, 43.5), turned to 90 degrees
- moved J1 81.5 mm to (154.6, 32.2), turned to 180 degrees
- moved R8 78.3 mm to (153.5, 43.4), turned to 90 degrees
- moved R1 71.9 mm to (149.5, 39.0), turned to 90 degrees
- moved Q2 71.2 mm to (130.5, 43.4), turned to -90 degrees
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Connections:
- U9 pad 10: PYRO1 -> unconnected-(U9-Pad10)
- U9 pad 11: PYRO2 -> PYRO1
- U9 pad 14: PYRO3 -> PYRO2
- U9 pad 15: PYRO4 -> PYRO3
- U9 pad 16: unconnected-(U9-Pad16) -> PYRO4
- U9 pad 17: VMON -> BUZZER
- U9 pad 21: BUZZER -> SCK
- U9 pad 22: unconnected-(U9-Pad22) -> MISO
- U9 pad 23: unconnected-(U9-Pad23) -> MOSI
- U9 pad 24: unconnected-(U9-Pad24) -> CS2_GYRO
- U9 pad 25: unconnected-(U9-Pad25) -> CS1_ACC
- U9 pad 37: unconnected-(U9-Pad37) -> INT_ACC1
- U9 pad 38: unconnected-(U9-Pad38) -> INT_ACC2
- U9 pad 41: unconnected-(U9-Pad41) -> INT_GYRO1
- U9 pad 42: unconnected-(U9-Pad42) -> INT_GYRO2
- U9 pad 55: SCK -> unconnected-(U9-Pad55)
- U9 pad 56: MISO -> VMON
- U9 pad 57: MOSI -> unconnected-(U9-Pad57)
- U9 pad 58: INT_ACC1 -> unconnected-(U9-Pad58)
- U9 pad 59: INT_ACC2 -> unconnected-(U9-Pad59)
- U9 pad 61: INT_GYRO1 -> unconnected-(U9-Pad61)
- U9 pad 62: INT_GYRO2 -> unconnected-(U9-Pad62)
- U9 pad 8: CS1_ACC -> unconnected-(U9-Pad8)
- U9 pad 9: CS2_GYRO -> unconnected-(U9-Pad9)
Routing:
- net GND: track 55.0 -> 174.6 mm, vias 0 -> 5
- net PWR: track 0.00 -> 87.8 mm
- net 3.3V: track 4.40 -> 39.3 mm, vias 0 -> 4
- net VMON: track 0.00 -> 33.4 mm
- net USB_OTG_FS_ID: track 2.72 -> 35.0 mm
- net USB_OTG_FS_DP: track 2.31 -> 32.4 mm
- net USB_OTG_FS_DM: track 2.20 -> 25.7 mm
- net INT_ACC2: track 0.00 -> 15.4 mm
- net BUZZER: track 0.00 -> 10.0 mm
- net INT_ACC1: track 0.00 -> 9.91 mm
- net PYRO2: track 0.00 -> 8.77 mm, vias 0 -> 2
- net PYRO1: track 0.00 -> 7.58 mm, vias 0 -> 2
- net PYRO4: track 0.00 -> 7.33 mm, vias 0 -> 2
- net PYRO3: track 0.00 -> 7.20 mm, vias 0 -> 2
- net Net-(J1-Pad8): track 0.00 -> 6.71 mm
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