File: OBC-Attempt-3_Dual_Deploy/OBC-Attempt-3_Dual_Deploy.kicad_sch (KiCad schematic)
At the start: 31 parts, among them J1 Bat, J2 Bat, J3 PWR, J4 DEBUG, J5 CAN Header, SW1 SW_SPDT, SW2 SW_SPST, U1 LD1117S33TR_SOT223, U2 STM32F042G4Ux, U3 SN65HVD230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

Commit message: Re org da files
Parts:
- removed C10: 1uF, Capacitor_SMD:C_0402_1005Metric, symbol Device:C
- removed C11: 10uF, Capacitor_SMD:C_0402_1005Metric, symbol Device:C
- removed C12, C13, C14: 100nF, Capacitor_SMD:C_0402_1005Metric, symbol Device:C
- removed U4: MS560702BA03-50, MS5607:SON125P300X500X100-8N, symbol MS5607-02BA03:MS560702BA03-50
- removed U5: BMI088, BMI088:PQFN50P450X300X100-16N, symbol BMI088:BMI088
- removed U6: MMC5983MA, MMC5983MA:PQFN50P300X300X100-16N, symbol MMC5983MA:MMC5983MA
Connections:
- net IMU_INT1: no longer names the net of U2.6 (PA0)
- net IMU_INT2: no longer names the net of U2.7 (PA1)
- net IMU_INT3: no longer names the net of U2.8 (PA2)
- net IMU_INT4: no longer names the net of U2.9 (PA3)
- net MAG_INT1: no longer names the net of U2.10 (PA4)
- net SPI1_MISO: no longer names the net of U2.12 (PA6)
- net SPI1_MOSI: no longer names the net of U2.13 (PA7)
- net SPI1_SCK: no longer names the net of U2.11 (PA5)
- net USART1_RX: no longer names the net of U2.28 (PB7)
- net USART1_TX: no longer names the net of U2.27 (PB6)
Other:
- note removed: "Barometric Altimeter (SPI)"
- note removed: "IMU (SPI)"
- note removed: "Magnetometer (SPI)"

Commit message: Work on board
Parts:
- added J6, J7: Conn_01x02_Female, Connector_PinHeader_1.00mm:PinHeader_1x02_P1.00mm_Vertical, symbol Connector:Conn_01x02_Female
- added R4, R5: 270, Resistor_SMD:R_01005_0402Metric, symbol Device:R
- added U4, U5: CPC1002N, Package_SO:SOP-4_3.8x4.1mm_P2.54mm, symbol Relay_SolidState:CPC1002N
Connections:
- net 12V+: now also U4.3, U5.3
- net GND: now also J6.2 (Pin_2), J7.2 (Pin_2), U4.2, U5.2
- net Pyro1: now reaches U2.8 (PA2)
- net Pyro1: now also R4.2
- net Pyro2: now reaches U2.9 (PA3)
- net Pyro2: now also R5.1
- new net: R5.2, U5.1
- new net: J7.1 (Pin_1), U5.4
- new net: R4.1, U4.1
- new net: J6.1 (Pin_1), U4.4
- no-connect marks 0 -> 16

Commit message: Cherry Rework
Parts:
- removed J6, J7: Conn_01x02_Female, Connector_PinHeader_1.00mm:PinHeader_1x02_P1.00mm_Vertical, symbol Connector:Conn_01x02_Female
- added J6: Conn_01x03_Female, Connector_PinSocket_2.54mm:PinSocket_1x03_P2.54mm_Vertical, symbol Connector:Conn_01x03_Female
Connections:
- net GND: now also J6.3 (Pin_3)
- net at U5.4: now also J6.1 (Pin_1)
- net at U4.4: now also J6.2 (Pin_2)
Other:
- moved on the sheet: R4, R5, U4, U5

Commit message: Yas
Parts:
- J6: value Conn_01x03_Female -> Deployment; symbol Connector:Conn_01x03_Female -> Connector:Conn_01x03_Male
- R4, R5: footprint Resistor_SMD:R_01005_0402Metric -> Resistor_SMD:R_0402_1005Metric
Connections:
- net GND: now also J6.1 (Pin_1); no longer J6.3 (Pin_3)
- net at U5.4: now also J6.3 (Pin_3); no longer J6.1 (Pin_1)
Changed lines of the file:
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@@
     (property "Reference" "R4" (id 0) (at 190.5 64.135 90))
     (property "Value" "270" (id 1) (at 190.5 69.215 90))
-    (property "Footprint" "Resistor_SMD:R_01005_0402Metric" (id 2) (at 190.5 64.897 90)
+    (property "Footprint" "Resistor_SMD:R_0402_1005Metric" (id 2) (at 190.5 64.897 90)
       (effects (font (size 1.27 1.27)) hide)
     )
@@
     (property "Reference" "R5" (id 0) (at 190.5 48.895 90))
     (property "Value" "270" (id 1) (at 190.5 53.975 90))
-    (property "Footprint" "Resistor_SMD:R_01005_0402Metric" (id 2) (at 190.5 53.213 90)
+    (property "Footprint" "Resistor_SMD:R_0402_1005Metric" (id 2) (at 190.5 53.213 90)
       (effects (font (size 1.27 1.27)) hide)
     )
@@
     (pin "4")
   )
-  (symbol (lib_id "Connector:Conn_01x03_Female") (at 226.695 66.675 0) (unit 1)
+  (symbol (lib_id "Connector:Conn_01x03_Male") (at 226.695 66.675 180) (unit 1)
     (in_bom yes) (on_board yes) (fields_autoplaced)
     (property "Reference" "J6" (id 0) (at 228.6 65.4049 0)
-      (effects (font (size 1.27 1.27)) (justify left))
-    )
-    (property "Value" "Conn_01x03_Female" (id 1) (at 228.6 67.9449 0)
-      (effects (font (size 1.27 1.27)) (justify left))
+      (effects (font (size 1.27 1.27)) (justify right))
+    )
+    (property "Value" "Deployment" (id 1) (at 228.6 67.9449 0)
+      (effects (font (size 1.27 1.27)) (justify right))
     )
     (property "Footprint" "Connector_PinSocket_2.54mm:PinSocket_1x03_P2.54mm_Vertical" (id 2) (at 226.695 66.675 0)
@@
     )
     (path "/93b6177e-cd4a-48d0-8275-f4c681696203"
-      (reference "J6") (unit 1) (value "Conn_01x03_Female") (footprint "Connector_PinSocket_2.54mm:PinSocket_1x03_P2.54mm_Vertical")
+      (reference "J6") (unit 1) (value "Deployment") (footprint "Connector_PinSocket_2.54mm:PinSocket_1x03_P2.54mm_Vertical")
     )
     (path "/47a92c95-42ee-4ec5-a9ff-dc99e2f1e276"
@@
     )
     (path "/1b70d0c9-8dc8-4f1e-82be-f9e70b316b96"
-      (reference "R4") (unit 1) (value "270") (footprint "Resistor_SMD:R_01005_0402Metric")
+      (reference "R4") (unit 1) (value "270") (footprint "Resistor_SMD:R_0402_1005Metric")
     )
     (path "/609c4447-7d40-4517-a6b9-252b3d8ebec1"
-      (reference "R5") (unit 1) (value "270") (footprint "Resistor_SMD:R_01005_0402Metric")
+      (reference "R5") (unit 1) (value "270") (footprint "Resistor_SMD:R_0402_1005Metric")
     )
     (path "/c5dff228-5c1d-408a-911b-f90b11fa9704"
