File: OBC-Attempt-6_Matcha_2_Layer_4/OBC-Attempt-6_Matcha_2_Layer_4.kicad_sch (KiCad schematic)
At the start: 59 parts, among them J2 Screw_Terminal_01x08, J3 Screw_Terminal_01x08, J5 Conn_01x04, J6 Micro_SD_Card, J7 Screw_Terminal_01x02, J8 Screw_Terminal_01x02, SW1 PCM12SMTR, U1 BMI088, U10 CPC1020NTR, U11 CPC1020NTR, U12 NCP1117-3.3_SOT223, U2 CPC1020NTR, U3 CPC1020NTR, U4 CPC1020NTR, U5 CPC1020NTR, U7 CPC1020NTR, U8 CPC1020NTR, U9 STM32F401RDTx, Y1 ABMM2-25MHZ-D1-T

Commit message: Some Changes
Parts:
- removed C1, C11, C13, C2, C3, C4, C6, C8, C9: 100nF, Capacitor_SMD:C_0402_1005Metric, symbol Device:C_Small
- removed C10: 1uF, Capacitor_SMD:C_0603_1608Metric, symbol Device:C_Small
- removed C15: 4.7uF, Capacitor_SMD:C_0603_1608Metric, symbol Device:C_Small
- removed C16, C17: 26pf, Capacitor_SMD:C_0402_1005Metric, symbol pspice:C
- removed C7: 4.7uF, Capacitor_SMD:C_0402_1005Metric, symbol Device:C_Small
- removed D5, D6, D7, D8: B330, Diode_SMD:D_SMA, symbol Diode:B330
- removed J3: Screw_Terminal_01x08, TerminalBlock_Phoenix:TerminalBlock_Phoenix_MPT-0,5-8-2.54_1x08_P2.54mm_Horizontal, symbol Connector:Screw_Terminal_01x08
- removed R13: 10k, Resistor_SMD:R_0603_1608Metric, symbol Device:R
- removed R14, R15, R16, R17: 270, Resistor_SMD:R_0603_1608Metric, symbol Device:R_Small
- removed SW1: PCM12SMTR, PCM12SMTR:SW_PCM12SMTR, symbol PCM12SMTR:PCM12SMTR
- removed U1: BMI088, BMI088:BMI088, symbol BMI088:BMI088
- removed U10, U11, U7, U8: CPC1020NTR, CPC1020NTR:4-SOP, symbol CPC1020NTR:CPC1020NTR
- removed U9: STM32F401RDTx, Package_QFP:LQFP-64_10x10mm_P0.5mm, symbol MCU_ST_STM32F4:STM32F401RDTx
- removed Y1: ABMM2-25MHZ-D1-T, ABMM2_6mm_3_6mm:XTAL_ABMM2-25.000MHZ-D1-T, symbol ABMM2_25MHZ:ABMM2-25.000MHZ-D1-T
- added C?: 1uF, Capacitor_SMD:C_0402_1005Metric, symbol Device:C
- added C?: .1uF, Capacitor_SMD:C_0402_1005Metric, symbol Device:C
- added C?: 4.7nF, Capacitor_SMD:C_0402_1005Metric, symbol Device:C
- added C? (x2): 20pF, Capacitor_SMD:C_0402_1005Metric, symbol Device:C
- added C?: 4u7, Capacitor_SMD:C_0402_1005Metric, symbol Device:C
- added C?: 10nF, Capacitor_SMD:C_0402_1005Metric, symbol Device:C
- added J?: CAN Header, Connector_PinHeader_1.00mm:PinHeader_1x04_P1.00mm_Vertical, symbol Connector:Conn_01x04_Female
- added J?: Screw_Terminal_01x04, symbol Connector:Screw_Terminal_01x04
- added R? (x2): 60 ohm, Resistor_SMD:R_0805_2012Metric, symbol Device:R
- added R?: 10k, Resistor_SMD:R_0402_1005Metric, symbol Device:R
- added SW?: SW_SPDT, Jumper:SolderJumper-3_P1.3mm_Open_RoundedPad1.0x1.5mm_NumberLabels, symbol Switch:SW_SPDT
- added SW?: SW_SPST, Jumper:SolderJumper-2_P1.3mm_Open_RoundedPad1.0x1.5mm, symbol Switch:SW_SPST
- added U?: SN65HVD230, Package_SO:SOIC-8_3.9x4.9mm_P1.27mm, symbol Interface_CAN_LIN:SN65HVD230
- added U?: STM32F042G4Ux, Package_DFN_QFN:QFN-28_4x4mm_P0.5mm, symbol MCU_ST_STM32F0:STM32F042G4Ux
- added X?: ECS-2520MV-xxx-xx, Oscillator:Oscillator_SMD_ECS_2520MV-xxx-xx-4Pin_2.5x2.0mm, symbol Oscillator:ECS-2520MV-xxx-xx
- J2: value Screw_Terminal_01x08 -> SOL A; footprint TerminalBlock_Phoenix:TerminalBlock_Phoenix_MPT-0,5-8-2.54_1x08_P2.54mm_Horizontal -> TerminalBlock_Phoenix:TerminalBlock_Phoenix_MPT-0,5-4-2.54_1x04_P2.54mm_Horizontal; symbol Connector:Screw_Terminal_01x08 -> Connector:Screw_Terminal_01x04
- renumbered D3 to D2, D4 to D3, D2 to D4, U4 to U1, U5 to U4
Connections:
- net 3.3V: now also J5.3 (Pin_3), C?.1, C?.1, C?.1, C?.1, SW?.3 (C), U?.17 (VDD), U?.18 (VDDIO2), U?.5 (VDDA); no longer J5.2 (Pin_2)
- net BATT+: now also J7.2 (Pin_2), J8.1 (Pin_1); no longer J7.1 (Pin_1), J8.2 (Pin_2)
- net GND: now also J2.1 (Pin_1), J2.3 (Pin_3), J7.1 (Pin_1), C?.2, C?.2, C?.2, C?.2, C?.2, C?.2, C?.2, J?.1 (Pin_1), J?.3 (Pin_3), SW?.1 (A), U?.16 (VSSA), U?.2 (GND), U?.8 (Rs), X?.2 (GND), X?.4 (VDD); no longer D1.2 (A), D2.2 (A), D3.2 (A), D4.2 (A), J2.2 (Pin_2), J2.4 (Pin_4), J2.6 (Pin_6), J2.8 (Pin_8), J7.2 (Pin_2)
- net PWR: now also J8.2 (Pin_2); no longer J8.1 (Pin_1)
- net RCC_OSC_IN: now also C?.1, U?.2 (PF0), X?.1 (Tri-State)
- net RCC_OSC_OUT: now also C?.1, U?.3 (PF1), X?.3 (OUT)
- net SYS_JTMS-SWDIO: now also J5.2 (Pin_2); no longer J5.3 (Pin_3)
- new net: D3.1 (K), J?.2 (Pin_2)
- new net: D3.2 (A), U3.4
- new net: D2.1 (K), J2.2 (Pin_2)
- new net: D1.1 (K), J2.4 (Pin_4)
- new net: R?.1, SW?.1 (A)
- new net: C?.1, R?.1, R?.2
- new net: D1.2 (A), U1.4
- new net: D2.2 (A), U2.4
- new net: R?.2, SW?.2 (B)
- new net: D4.2 (A), U4.4
- new net: D4.1 (K), J?.4 (Pin_4)
- new net +3.3V: U?.3 (VCC)
- new net BOOT0: R?.1, U?.4 (NRST)
- new net CAN_H: J?.3 (Pin_3), J?.4 (Pin_4), SW?.2 (B), U?.7 (CANH)
- new net CAN_L: J?.1 (Pin_1), J?.2 (Pin_2), R?.2, U?.6 (CANL)
- new net CAN_RX: U?.1 (PB8), U?.4 (R)
- new net CAN_TX: U?.1 (D), U?.20 (PA10/PA12)
- new net SYS_SWCLK: U?.22 (PA14)
- new net SYS_SWDIO: U?.21 (PA13)
- no-connect marks 26 -> 19
Other:
- note added: "MICROCHIP: STM32F042G4Ux"
- note added: "Transciever (CAN)"
- note removed: "LSE CYRSTAL OSCILLATOR"
- note removed: "MICROCHIP: STM32F401RDT6TR"
- moved on the sheet: D1, D2, D3, D4, J5, J7, J8, R10, R11, R12, R9, U1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

Commit message: PCB LAYOUT
Parts:
- removed BZ1: Buzzer, Buzzer_Beeper:Buzzer_TDK_PS1240P02BT_D12.2mm_H6.5mm, symbol Device:Buzzer
- removed J6: Micro_SD_Card, Connector_Card:microSD_HC_Wuerth_693072010801, symbol Connector:Micro_SD_Card
- J3: renamed from J?; footprint (none) -> TerminalBlock_Phoenix:TerminalBlock_Phoenix_MPT-0,5-4-2.54_1x04_P2.54mm_Horizontal
- U1, U2, U3, U4: footprint CPC1020NTR:4-SOP -> 4-SOP
- gave numbers to parts that had none: 16
Connections:
- no-connect marks 19 -> 18

Commit message: Open
Parts:
- J3: value Screw_Terminal_01x04 -> SOL B
Other:
- moved on the sheet: D3, D4, R10, R12, U3, U4

Commit message: Working on schematic
Parts:
- removed D1, D2, D3, D4: B330, Diode_SMD:D_SMA, symbol Diode:B330
- removed R10, R11, R12, R9: 270, Resistor_SMD:R_0603_1608Metric, symbol Device:R_Small
- removed U1, U2, U3, U4: CPC1020NTR, 4-SOP, symbol CPC1020NTR:CPC1020NTR
- added R? (x8): R, symbol Device:R
- added U? (x4): ACPL-244-500E, SOIC127P700X242-16N, symbol ACPL-244:ACPL-244-500E
Connections:
- net GND: now also R?.1, R?.1, R?.1, R?.1; no longer J2.1 (Pin_1), J2.3 (Pin_3), J3.1 (Pin_1), J3.3 (Pin_3)
- net PWR: now also U?.10, U?.12, U?.14, U?.16
- new net: R?.2, U?.15
- new net: R?.2, U?.13
- new net: R?.2, U?.11
- new net: R?.2, U?.9

Commit message: Complete chematic
Might have to change the optocouplers
Parts:
- removed H1, H2, H3, H4: MountingHole, MountingHole:MountingHole_3mm, symbol Mechanical:MountingHole
- removed U? (x4): ACPL-244-500E, SOIC127P700X242-16N, symbol ACPL-244:ACPL-244-500E
- added D1, D2: CVJ10F30, CVJ10F30:CVJ10F30, symbol CVJ10F30:CVJ10F30
- added H1, H2, H3, H4: MountingHole_Pad, MountingHole:MountingHole_2.2mm_M2_Pad_TopBottom, symbol Mechanical:MountingHole_Pad
- added U1, U2: LTV-827S, Package_DIP:SMDIP-8_W9.53mm, symbol Isolator:LTV-827S
- added U3, U4: QS5K2TR, QS5K2TR:SOT95P280X100-5N, symbol QS5K2TR:QS5K2TR
- R10, R11, R8, R9: renamed from R?; footprint (none) -> Resistor_SMD:R_0603_1608Metric
- R4, R5, R6, R7: renamed from R?; footprint (none) -> Resistor_SMD:R_0402_1005Metric
Connections:
- net SYS_SWCLK is gone; now on net SYS_JTCK_SWCLK: U6.22 (PA14)
- net SYS_SWDIO is gone; now on net SYS_JTMS-SWDIO: U6.21 (PA13)
- net GND: now also H1.1, H2.1, H3.1, H4.1, U1.2, U1.4, U2.2, U2.4, U3.2, U4.2
- net PWR: now also J2.1 (Pin_1), J2.3 (Pin_3), J3.1 (Pin_1), J3.3 (Pin_3), D1.4 (D2OUT), D1.5 (D1OUT), D2.4 (D2OUT), D2.5 (D1OUT), U1.6, U1.8, U2.6, U2.8
- net SOL1: now also R4.2
- net SOL2: now also R5.2
- net SOL3: now also R6.2
- net SOL4: now also R7.2
- net at R8.2: now also U1.7, U3.1
- net SOLA: now reaches J2.2 (Pin_2)
- net SOLA: now also D1.1 (D1IN), U3.5
- net SOLB: now reaches J2.4 (Pin_4)
- net SOLB: now also D1.3 (D2IN), U3.4
- net at R9.2: now also U1.5, U3.3
- net at R7.1: now also U2.3
- net at R6.1: now also U2.1
- net at R4.1: now also U1.1
- net at R10.2: now also U2.7, U4.1
- net at R11.2: now also U2.5, U4.3
- net SOLC: now reaches J3.2 (Pin_2)
- net SOLC: now also D2.1 (D1IN), U4.5
- net SOLD: now reaches J3.4 (Pin_4)
- net SOLD: now also D2.3 (D2IN), U4.4
- net at R5.1: now also U1.3
Other:
- moved on the sheet: R4, R5, R6, R7

Commit message: Some late night pcb work
Parts:
- removed J7, J8: Screw_Terminal_01x02, TerminalBlock_Phoenix:TerminalBlock_Phoenix_MPT-0,5-2-2.54_1x02_P2.54mm_Horizontal, symbol Connector:Screw_Terminal_01x02
- removed U1, U2: LTV-827S, Package_DIP:SMDIP-8_W9.53mm, symbol Isolator:LTV-827S
- added J4: Screw_Terminal_01x04, TerminalBlock_Phoenix:TerminalBlock_Phoenix_MPT-0,5-4-2.54_1x04_P2.54mm_Horizontal, symbol Connector:Screw_Terminal_01x04
- added U1: LTV-247, Package_SO:SOP-16_4.4x10.4mm_P1.27mm, symbol Isolator:LTV-247
- J5: footprint Connector_PinHeader_2.54mm:PinHeader_1x04_P2.54mm_Vertical -> Connector_PinHeader_1.00mm:PinHeader_1x04_P1.00mm_Vertical
Connections:
- net +3.3V is gone; now on net 3.3V: U5.3 (VCC)
- net BATT+: now also J4.2 (Pin_2), J4.3 (Pin_3)
- net GND: now also J4.1 (Pin_1), U1.2, U1.4, U1.6, U1.8
- net PWR: now also J4.4 (Pin_4), U1.10, U1.12, U1.14, U1.16
- net at R8.2, U3.1: now also U1.15
- net at R4.1: now also U1.1
- net at R9.2, U3.3: now also U1.13
- net at R7.1: now also U1.7
- net at R6.1: now also U1.5
- net at R10.2, U4.1: now also U1.11
- net at R5.1: now also U1.3
- net at R11.2, U4.3: now also U1.9

Commit message: Wired Everything in the board
Parts:
- removed H4: MountingHole_Pad, MountingHole:MountingHole_2.2mm_M2_Pad_TopBottom, symbol Mechanical:MountingHole_Pad
- removed J5: Conn_01x04, Connector_PinHeader_1.00mm:PinHeader_1x04_P1.00mm_Vertical, symbol Connector_Generic:Conn_01x04
- added J5: Conn_01x02_Male, symbol Connector:Conn_01x02_Male
- added J6: Conn_01x02_Male, Connector_PinHeader_1.00mm:PinHeader_1x02_P1.00mm_Vertical, symbol Connector:Conn_01x02_Male
Connections:
- net 3.3V: now also J6.1 (Pin_1)
- net GND: now also J4.4 (Pin_4), J6.2 (Pin_2); no longer J4.1 (Pin_1)
- net PWR: now also J2.2 (Pin_2), J2.4 (Pin_4), J3.2 (Pin_2), J3.4 (Pin_4), J4.1 (Pin_1); no longer J2.1 (Pin_1), J2.3 (Pin_3), J3.1 (Pin_1), J3.3 (Pin_3), J4.4 (Pin_4)
- net SOL1: now also U6.13 (PA7)
- net SOL2: now also U6.15 (PB1)
- net SOL3: now also U6.11 (PA5)
- net SOL4: now also U6.9 (PA3)
- net SOLA: now also J2.3 (Pin_3); no longer J2.2 (Pin_2)
- net SOLB: now also J2.1 (Pin_1); no longer J2.4 (Pin_4)
- net SOLC: now also J3.3 (Pin_3); no longer J3.2 (Pin_2)
- net SOLD: now also J3.1 (Pin_1); no longer J3.4 (Pin_4)
- net SYS_JTCK_SWCLK: now also J5.2 (Pin_2)
- net SYS_JTMS-SWDIO: now also J5.1 (Pin_1)
- net VMON: now also U6.7 (PA1)
- no-connect marks 18 -> 13
