File: OBC-Attempt-6_Matcha_2_Layer_4/OBC-Attempt-6_Matcha_2_Layer_4.kicad_pcb (KiCad board)
At the start: 4 copper layers, 25.4 x 31.8 mm, 42 parts, among them J1 CAN Header, J2 SOL A, J3 SOL B, J4 Screw_Terminal_01x04, J5 Conn_01x02_Male, J6 Conn_01x02_Male, SW1 SW_SPST, SW2 SW_SPDT, U1 LTV-247, U12 NCP1117-3.3_SOT223, U3 QS5K2TR, U4 QS5K2TR, U5 SN65HVD230, U6 STM32F042G4Ux, X1 ECS-2520MV-xxx-xx

Commit message: Added front stuff
Other:
- board text added: "+BATT-"
- board text added: "- RCS"
- board text added: "-SOL A+"
- board text added: "-SOL B+"
- board text added: "-SOL C+"
- board text added: "-SOL D+"
- board text added: "3"
- board text added: "3.3V"
- board text added: "ALEX AARHUS"
- board text added: "CAN H"
- board text added: "CAN L"
- board text added: "CLK"
- board text added: "DIO"
- board text added: "G"
- board text added: "GND"
- board text added: "GO KARMAN!"
- board text added: "GO SAN DIEGO!"
- board text added: "MATCHA V4.0"
- board text added: "PSHHHHHHHH!"
- board text added: "SDSURP 2023"
- board text added: "SWITCH"
Changed lines of the file:
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@@
 (kicad_pcb (version 20211014) (generator pcbnew)
   (general
-    (thickness 4.69)
+    (thickness 1.58)
   )
   (paper "A4")
@@
       (layer "F.Mask" (type "Top Solder Mask") (thickness 0.01))
       (layer "F.Cu" (type "copper") (thickness 0.035))
-      (layer "dielectric 1" (type "core") (thickness 1.51) (material "FR4") (epsilon_r 4.5) (loss_tangent 0.02))
+      (layer "dielectric 1" (type "prepreg") (thickness 0.11) (material "FR4") (epsilon_r 4.5) (loss_tangent 0.02))
       (layer "In1.Cu" (type "copper") (thickness 0.035))
-      (layer "dielectric 2" (type "prepreg") (thickness 1.51) (material "FR4") (epsilon_r 4.5) (loss_tangent 0.02))
+      (layer "dielectric 2" (type "core") (thickness 1.2) (material "FR4") (epsilon_r 4.5) (loss_tangent 0.02))
       (layer "In2.Cu" (type "copper") (thickness 0.035))
-      (layer "dielectric 3" (type "core") (thickness 1.51) (material "FR4") (epsilon_r 4.5) (loss_tangent 0.02))
+      (layer "dielectric 3" (type "prepreg") (thickness 0.11) (material "FR4") (epsilon_r 4.5) (loss_tangent 0.02))
       (layer "B.Cu" (type "copper") (thickness 0.035))
       (layer "B.Mask" (type "Bottom Solder Mask") (thickness 0.01))
@@
   )
   (gr_rect (start 25.4 25.4) (end 50.8 57.15) (layer "Edge.Cuts") (width 0.1) (fill none))
+  (gr_text "SWITCH" (at 35.52 26.7) (layer "F.SilkS")
+    (effects (font (size 0.5 0.5) (thickness 0.1)))
+  )
+  (gr_text "DIO" (at 48.99 45.79 -90) (layer "F.SilkS")
+    (effects (font (size 0.5 0.5) (thickness 0.1)))
+  )
+  (gr_text "ALEX AARHUS" (at 33.18 51.194) (layer "F.SilkS")
+    (effects (font (size 0.5 0.5) (thickness 0.1)))
+  )
+  (gr_text "G" (at 41.64 34.61) (layer "F.SilkS")
+    (effects (font (size 0.5 0.5) (thickness 0.1)))
+  )
+  (gr_text "-SOL B+" (at 26.75 53.94 90) (layer "F.SilkS")
+    (effects (font (size 0.5 0.5) (thickness 0.1)))
+  )
+  (gr_text "- RCS" (at 42.37 53.35 -90) (layer "F.SilkS")
+    (effects (font (size 0.75 0.75) (thickness 0.15)))
+  )
+  (gr_text "CAN H" (at 28.68 44.15) (layer "F.SilkS")
+    (effects (font (size 0.5 0.5) (thickness 0.1)))
+  )
+  (gr_text "GND" (at 29.55 40.51) (layer "F.SilkS")
+    (effects (font (size 0.5 0.5) (thickness 0.1)))
+  )
+  (gr_text "GO KARMAN! " (at 40.36 39.909999) (layer "F.SilkS")
+    (effects (font (size 0.5 0.5) (thickness 0.1)))
+  )
+  (gr_text "-SOL A+" (at 26.84 49.03 90) (layer "F.SilkS")
+    (effects (font (size 0.5 0.5) (thickness 0.1)))
+  )
+  (gr_text "CAN L" (at 30.67 41.76) (layer "F.SilkS")
+    (effects (font (size 0.5 0.5) (thickness 0.1)))
+  )
+  (gr_text "-SOL C+" (at 49.19 53.87 270) (layer "F.SilkS")
+    (effects (font (size 0.5 0.5) (thickness 0.1)))
+  )
+  (gr_text "+BATT- " (at 40.55 26.71) (layer "F.SilkS")
+    (effects (font (size 0.5 0.5) (thickness 0.1)))
+  )
+  (gr_text "3" (at 46.16 34.61) (layer "F.SilkS")
+    (effects (font (size 0.5 0.5) (thickness 0.1)))
+  )
+  (gr_text "CLK" (at 50.06 45.87 270) (layer "F.SilkS")
+    (effects (font (size 0.5 0.5) (thickness 0.1)))
+  )
+  (gr_text "SDSURP 2023" (at 33.18 51.92) (layer "F.SilkS")
+    (effects (font (size 0.5 0.5) (thickness 0.1)))
+  )
+  (gr_text "3.3V" (at 29.52 39.41) (layer "F.SilkS")
+    (effects (font (size 0.5 0.5) (thickness 0.1)))
+  )
+  (gr_text "-SOL D+" (at 49.28 48.96 270) (layer "F.SilkS")
+    (effects (font (size 0.5 0.5) (thickness 0.1)))
+  )
+  (gr_text "MATCHA V4.0" (at 33.18 50.48) (layer "F.SilkS")
+    (effects (font (size 0.5 0.5) (thickness 0.1)))
+  )
+  (gr_text "PSHHHHHHHH!" (at 43.57 51.29 -90) (layer "F.SilkS")
+    (effects (font (size 1 1) (thickness 0.2)))
+  )
+  (gr_text "GO SAN DIEGO!" (at 40.36 40.73) (layer "F.SilkS")
+    (effects (font (size 0.5 0.5) (thickness 0.1)))
+  )
   (segment (start 33.619999 43.699999) (end 33.619999 44.749999) (width 0.5) (layer "F.Cu") (net 1))
   (segment (start 33.619999 45.810001) (end 33.619999 44.749999) (width 0.5) (layer "F.Cu") (net 1))
@@
   (segment (start 34.475 49.835) (end 35.255 49.055) (width 0.5) (layer "B.Cu") (net 9))
   (segment (start 28.99 55.16) (end 33.68 55.16) (width 0.5) (layer "B.Cu") (net 9))
+  (segment (start 47.98 55.3) (end 47.16 55.3) (width 0.7) (layer "F.Cu") (net 10))
+  (segment (start 49.21 50.95) (end 49.21 54.07) (width 0.7) (layer "F.Cu") (net 10))
+  (segment (start 29.55 52.62) (end 33.31 56.38) (width 0.7) (layer "F.Cu") (net 10))
   (segment (start 47.16 50.22) (end 48.48 50.22) (width 0.7) (layer "F.Cu") (net 10))
-  (segment (start 49.21 50.95) (end 49.21 53.25) (width 0.7) (layer "F.Cu") (net 10))
-  (segment (start 29.55 52.62) (end 33.31 56.38) (width 0.7) (layer "F.Cu") (net 10))
+  (segment (start 48.48 50.22) (end 49.21 50.95) (width 0.7) (layer "F.Cu") (net 10))
   (segment (start 33.31 56.38) (end 45.39 56.38) (width 0.7) (layer "F.Cu") (net 10))
-  (segment (start 48.48 50.22) (end 49.21 50.95) (width 0.7) (layer "F.Cu") (net 10))
+  (segment (start 49.21 54.07) (end 47.98 55.3) (width 0.7) (layer "F.Cu") (net 10))
   (segment (start 45.39 56.38) (end 46.47 55.3) (width 0.7) (layer "F.Cu") (net 10))
   (segment (start 46.47 55.3) (end 47.16 55.3) (width 0.7) (layer "F.Cu") (net 10))
   (segment (start 28.99 52.62) (end 29.55 52.62) (width 0.7) (layer "F.Cu") (net 10))
-  (segment (start 49.21 53.25) (end 47.16 55.3) (width 0.7) (layer "F.Cu") (net 10))
   (segment (start 38.38 42.14) (end 37.89 41.65) (width 0.5) (layer "B.Cu") (net 10))
   (segment (start 26.19 41.76) (end 26.19 46.3) (width 0.7) (layer "B.Cu") (net 10))
@@
   (segment (start 43.803334 40.66) (end 43.8 40.656666) (width 0.3) (layer "F.Cu") (net 22))
   (via (at 43.8 40.656666) (size 0.7) (drill 0.3) (layers "F.Cu" "B.Cu") (free) (net 22))
+  (segment (start 34.3 34.39) (end 32.37 34.39) (width 0.5) (layer "B.Cu") (net 22))
+  (segment (start 32.37 34.39) (end 32.12 34.64) (width 0.5) (layer "B.Cu") (net 22))
+  (segment (start 34.48 34.57) (end 34.3 34.39) (width 0.5) (layer "B.Cu") (net 22))
   (segment (start 32.12 34.64) (end 32.12 38.91) (width 0.5) (layer "B.Cu") (net 22))
-  (segment (start 32.6 34.16) (end 32.12 34.64) (width 0.5) (layer "B.Cu") (net 22))
-  (segment (start 34.08 34.17) (end 34.08 34.16) (width 0.5) (layer "B.Cu") (net 22))
-  (segment (start 34.48 34.57) (end 34.08 34.17) (width 0.5) (layer "B.Cu") (net 22))
+  (segment (start 32.48 39.27) (end 41.64 39.27) (width 0.5) (layer "B.Cu") (net 22))
+  (segment (start 41.64 39.27) (end 43.026666 40.656666) (width 0.5) (layer "B.Cu") (net 22))
+  (segment (start 32.12 38.91) (end 32.48 39.27) (width 0.5) (layer "B.Cu") (net 22))
   (segment (start 34.48 35.28) (end 34.48 34.57) (width 0.5) (layer "B.Cu") (net 22))
-  (segment (start 34.08 34.16) (end 32.6 34.16) (width 0.5) (layer "B.Cu") (net 22))
-  (segment (start 32.48 39.27) (end 41.64 39.27) (width 0.5) (layer "B.Cu") (net 22))
   (segment (start 43.026666 40.656666) (end 43.8 40.656666) (width 0.5) (layer "B.Cu") (net 22))
-  (segment (start 32.12 38.91) (end 32.48 39.27) (width 0.5) (layer "B.Cu") (net 22))
-  (segment (start 41.64 39.27) (end 43.026666 40.656666) (width 0.5) (layer "B.Cu") (net 22))
   (segment (start 35.83 35.88) (end 35.83 36.73) (width 0.5) (layer "B.Cu") (net 23))
   (segment (start 36.02 35.69) (end 35.83 35.88) (width 0.5) (layer "B.Cu") (net 23))

Commit message: Open multiple
Routing:
- net PWR: track 101.8 -> 103.0 mm
Changed lines of the file:
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@@
   (segment (start 40.91 42.17) (end 40.39 41.65) (width 0.5) (layer "B.Cu") (net 10))
   (segment (start 28.99 52.62) (end 33.135 52.62) (width 0.7) (layer "B.Cu") (net 10))
-  (segment (start 26.19 27.02) (end 26.19 41.76) (width 0.7) (layer "B.Cu") (net 10))
   (segment (start 35.83 42.03) (end 35.45 41.65) (width 0.5) (layer "B.Cu") (net 10))
+  (segment (start 34.08 28.92) (end 34.08 26.84) (width 0.7) (layer "B.Cu") (net 10))
   (segment (start 32.82 41.65) (end 26.3 41.65) (width 0.5) (layer "B.Cu") (net 10))
   (segment (start 38.38 43.03) (end 38.38 42.14) (width 0.5) (layer "B.Cu") (net 10))
@@
   (segment (start 28.99 47.54) (end 27.43 47.54) (width 0.7) (layer "B.Cu") (net 10))
   (segment (start 40.39 41.65) (end 37.67 41.65) (width 0.5) (layer "B.Cu") (net 10))
-  (segment (start 31.35 26.19) (end 27.02 26.19) (width 0.7) (layer "B.Cu") (net 10))
-  (segment (start 34.08 28.92) (end 31.35 26.19) (width 0.7) (layer "B.Cu") (net 10))
   (segment (start 35.45 41.65) (end 32.82 41.65) (width 0.5) (layer "B.Cu") (net 10))
   (segment (start 40.91 43.03) (end 40.91 42.17) (width 0.5) (layer "B.Cu") (net 10))
+  (segment (start 27.02 26.19) (end 26.19 27.02) (width 0.7) (layer "B.Cu") (net 10))
   (segment (start 27.434366 52.62) (end 28.99 52.62) (width 0.7) (layer "B.Cu") (net 10))
   (segment (start 33.29 42.12) (end 32.82 41.65) (width 0.5) (layer "B.Cu") (net 10))
@@
   (segment (start 26.19 46.3) (end 26.19 51.375634) (width 0.7) (layer "B.Cu") (net 10))
   (segment (start 37.89 41.65) (end 37.67 41.65) (width 0.5) (layer "B.Cu") (net 10))
+  (segment (start 26.19 27.02) (end 26.19 41.76) (width 0.7) (layer "B.Cu") (net 10))
   (segment (start 44.91 55.3) (end 47.16 55.3) (width 0.7) (layer "B.Cu") (net 10))
-  (segment (start 27.02 26.19) (end 26.19 27.02) (width 0.7) (layer "B.Cu") (net 10))
+  (segment (start 34.08 26.84) (end 33.43 26.19) (width 0.7) (layer "B.Cu") (net 10))
   (segment (start 37.67 41.65) (end 35.45 41.65) (width 0.5) (layer "B.Cu") (net 10))
   (segment (start 26.19 51.375634) (end 27.434366 52.62) (width 0.7) (layer "B.Cu") (net 10))
@@
   (segment (start 33.29 43.03) (end 33.29 42.12) (width 0.5) (layer "B.Cu") (net 10))
   (segment (start 42.99 53.38) (end 44.91 55.3) (width 0.7) (layer "B.Cu") (net 10))
+  (segment (start 33.43 26.19) (end 27.02 26.19) (width 0.7) (layer "B.Cu") (net 10))
   (segment (start 35.83 43.03) (end 35.83 42.03) (width 0.5) (layer "B.Cu") (net 10))
   (segment (start 40.8225 49.095) (end 40.8225 49.3825) (width 0.5) (layer "B.Cu") (net 11))
