File: PT Board Ground Systems/PT Board Ground Systems.kicad_pcb (KiCad board)
At the start: 2 copper layers, 58.4 x 25.4 mm, 31 parts, among them J1 OUT CHAN 1, J2 CHAN IN, J3 OUT CHAN 2

Commit message: AGS Board Work
Parts:
- removed D10, D12, D14, D16, D2, D4, D6, D8: D_Small, Diode_SMD:D_SMA
- removed D11, D13, D15, D3, D5, D7, D9: LED, LED_SMD:LED_0805_2012Metric
- removed R2, R3, R4, R5, R6, R7, R8: 2.9K, Resistor_SMD:R_0603_1608Metric
- J1: value OUT CHAN 1 -> POWER IN; footprint TerminalBlock_Phoenix:TerminalBlock_Phoenix_MPT-0,5-8-2.54_1x08_P2.54mm_Horizontal -> TerminalBlock_Phoenix:TerminalBlock_Phoenix_MPT-0,5-2-2.54_1x02_P2.54mm_Horizontal
- J2: value CHAN IN -> OUT CHAN A; footprint TerminalBlock_Phoenix:TerminalBlock_Phoenix_MPT-0,5-2-2.54_1x02_P2.54mm_Horizontal -> TerminalBlock_Phoenix:TerminalBlock_Phoenix_MPT-0,5-8-2.54_1x08_P2.54mm_Horizontal
- J3: value OUT CHAN 2 -> OUT CHAN B
- moved J2 26.2 mm to (74.7, 30.9), turned to 180 degrees
- moved D1 24.8 mm to (46.4, 39.3), turned to 0 degrees
- moved J1 23.0 mm to (53.4, 39.3), turned to 0 degrees
- moved R1 21.3 mm to (49.7, 39.3), turned to 0 degrees
- moved H2 3.18 mm to (29.3, 41.3)
- moved H4 3.18 mm to (80.0, 41.3)
- moved H1 3.18 mm to (29.2, 28.6)
- moved H3 3.18 mm to (80.0, 28.6)
- moved J3 0.50 mm to (52.4, 30.9)
Connections:
- D1 pad 1: Net-(D1-Pad1) -> GND
- J1 pad 1: GND -> POWER IN
- J1 pad 2: Net-(D1-Pad1) -> GND
- J2 pad 1: Net-(D16-Pad2) -> GND
- J2 pad 2: GND -> POWER IN
- J3 pad 2: Net-(D10-Pad1) -> POWER IN
- J3 pad 4: Net-(D11-Pad1) -> POWER IN
- J3 pad 6: Net-(D13-Pad1) -> POWER IN
- J3 pad 8: Net-(D15-Pad1) -> POWER IN
- R1 pad 2: Net-(D16-Pad2) -> POWER IN
Routing:
- net Net-(D16-Pad2): track 103.8 -> 0.00 mm
- net Net-(D1-Pad1): track 9.09 -> 0.00 mm
- net Net-(D15-Pad1): track 8.93 -> 0.00 mm
- net Net-(D3-Pad1): track 8.82 -> 0.00 mm
- net Net-(D10-Pad1): track 8.67 -> 0.00 mm
- net Net-(D13-Pad1): track 8.67 -> 0.00 mm
- net Net-(D5-Pad1): track 8.60 -> 0.00 mm
- net Net-(D7-Pad1): track 8.57 -> 0.00 mm
- net Net-(D11-Pad1): track 8.43 -> 0.00 mm
- net Net-(D5-Pad2): track 1.57 -> 0.00 mm
- net Net-(D3-Pad2): track 1.54 -> 0.00 mm
- net Net-(D7-Pad2): track 1.52 -> 0.00 mm
- net Net-(D15-Pad2): track 1.51 -> 0.00 mm
- net Net-(D13-Pad2): track 1.48 -> 0.00 mm
- net Net-(D9-Pad2): track 1.44 -> 0.00 mm
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- added copper zone on F.Cu, net POWER IN
Other:
- board size 58.4 x 25.4 mm -> 58.4 x 19.1 mm
- board text removed: "AARHUS WUZ HERE"
