File: OBC-Attempt-5_Matcha_2_Layer_3/OBC-Attempt-5_Matcha_2_Layer_3.kicad_pcb (KiCad board)
At the start: 2 copper layers, 57.1 x 57.1 mm, 59 parts, among them J2 Screw_Terminal_01x08, J3 Screw_Terminal_01x08, J5 Conn_01x04, J6 Micro_SD_Card, J7 Screw_Terminal_01x02, J8 Screw_Terminal_01x02, SW1 PCM12SMTR, U1 BMI088, U10 CPC1020NTR, U11 CPC1020NTR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

Commit message: Some 4 Layer Work :)
Routing:
- net GND: track 59.9 -> 57.9 mm

Commit message: Some Gerbs Some Work
Parts:
- H1, H2, H3, H4: footprint MountingHole:MountingHole_3mm -> MountingHole:MountingHole_3.2mm_M3
Changed lines of the file:
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@@
       (drillshape 0)
       (scaleselection 1)
-      (outputdirectory "")
+      (outputdirectory "Gerb/")
     )
   )
@@
     )
   )
-  (footprint "MountingHole:MountingHole_3mm" (layer "F.Cu")
+  (footprint "MountingHole:MountingHole_3.2mm_M3" (layer "F.Cu")
     (at 76.2 31.75)
-    (descr "Mounting Hole 3mm, no annular")
-    (tags "mounting hole 3mm no annular")
+    (descr "Mounting Hole 3.2mm, no annular, M3")
+    (tags "mounting hole 3.2mm no annular m3")
     (property "Sheetfile" "OBC-Attempt-5_Matcha_2_Layer_3.kicad_sch")
     (property "Sheetname" "")
     (attr exclude_from_pos_files)
-    (fp_text reference "H2" (at 0 -4) (layer "F.Fab")
-      (effects (font (size 1 1) (thickness 0.15)))
-    )
-    (fp_text value "MountingHole" (at 0 4) (layer "F.Fab")
+    (fp_text reference "H2" (at 0 -4.2) (layer "F.SilkS")
+      (effects (font (size 1 1) (thickness 0.15)))
+    )
+    (fp_text value "MountingHole" (at 0 4.2) (layer "F.Fab")
       (effects (font (size 1 1) (thickness 0.15)))
     )
@@
       (effects (font (size 1 1) (thickness 0.15)))
     )
-    (fp_circle (center 0 0) (end 3 0) (layer "Cmts.User") (width 0.15) (fill none))
-    (fp_circle (center 0 0) (end 3.25 0) (layer "F.CrtYd") (width 0.05) (fill none))
-    (pad "" np_thru_hole circle (at 0 0) (size 3 3) (drill 3) (layers *.Cu *.Mask))
+    (fp_circle (center 0 0) (end 3.2 0) (layer "Cmts.User") (width 0.15) (fill none))
+    (fp_circle (center 0 0) (end 3.45 0) (layer "F.CrtYd") (width 0.05) (fill none))
+    (pad "" np_thru_hole circle (at 0 0) (size 3.2 3.2) (drill 3.2) (layers *.Cu *.Mask))
   )
   (footprint "CPC1020NTR:4-SOP" (layer "F.Cu")
@@
     )
   )
-  (footprint "MountingHole:MountingHole_3mm" (layer "F.Cu")
+  (footprint "MountingHole:MountingHole_3.2mm_M3" (layer "F.Cu")
     (at 76.2 76.2)
-    (descr "Mounting Hole 3mm, no annular")
-    (tags "mounting hole 3mm no annular")
+    (descr "Mounting Hole 3.2mm, no annular, M3")
+    (tags "mounting hole 3.2mm no annular m3")
     (property "Sheetfile" "OBC-Attempt-5_Matcha_2_Layer_3.kicad_sch")
     (property "Sheetname" "")
     (attr exclude_from_pos_files)
-    (fp_text reference "H4" (at 0 -4) (layer "F.Fab")
-      (effects (font (size 1 1) (thickness 0.15)))
-    )
-    (fp_text value "MountingHole" (at 0 4) (layer "F.Fab")
+    (fp_text reference "H4" (at 0 -4.2) (layer "F.SilkS")
+      (effects (font (size 1 1) (thickness 0.15)))
+    )
+    (fp_text value "MountingHole" (at 0 4.2) (layer "F.Fab")
       (effects (font (size 1 1) (thickness 0.15)))
     )
@@
       (effects (font (size 1 1) (thickness 0.15)))
     )
-    (fp_circle (center 0 0) (end 3 0) (layer "Cmts.User") (width 0.15) (fill none))
-    (fp_circle (center 0 0) (end 3.25 0) (layer "F.CrtYd") (width 0.05) (fill none))
-    (pad "" np_thru_hole circle (at 0 0) (size 3 3) (drill 3) (layers *.Cu *.Mask))
+    (fp_circle (center 0 0) (end 3.2 0) (layer "Cmts.User") (width 0.15) (fill none))
+    (fp_circle (center 0 0) (end 3.45 0) (layer "F.CrtYd") (width 0.05) (fill none))
+    (pad "" np_thru_hole circle (at 0 0) (size 3.2 3.2) (drill 3.2) (layers *.Cu *.Mask))
   )
   (footprint "Capacitor_SMD:C_0402_1005Metric" (layer "F.Cu")
@@
     )
   )
-  (footprint "MountingHole:MountingHole_3mm" (layer "F.Cu")
+  (footprint "MountingHole:MountingHole_3.2mm_M3" (layer "F.Cu")
     (at 31.75 76.2)
-    (descr "Mounting Hole 3mm, no annular")
-    (tags "mounting hole 3mm no annular")
+    (descr "Mounting Hole 3.2mm, no annular, M3")
+    (tags "mounting hole 3.2mm no annular m3")
     (property "Sheetfile" "OBC-Attempt-5_Matcha_2_Layer_3.kicad_sch")
     (property "Sheetname" "")
     (attr exclude_from_pos_files)
-    (fp_text reference "H1" (at 0 -4) (layer "F.Fab")
-      (effects (font (size 1 1) (thickness 0.15)))
-    )
-    (fp_text value "MountingHole" (at 0 4) (layer "F.Fab")
+    (fp_text reference "H1" (at 0 -4.2) (layer "F.SilkS")
+      (effects (font (size 1 1) (thickness 0.15)))
+    )
+    (fp_text value "MountingHole" (at 0 4.2) (layer "F.Fab")
       (effects (font (size 1 1) (thickness 0.15)))
     )
@@
       (effects (font (size 1 1) (thickness 0.15)))
     )
-    (fp_circle (center 0 0) (end 3 0) (layer "Cmts.User") (width 0.15) (fill none))
-    (fp_circle (center 0 0) (end 3.25 0) (layer "F.CrtYd") (width 0.05) (fill none))
-    (pad "" np_thru_hole circle (at 0 0) (size 3 3) (drill 3) (layers *.Cu *.Mask))
+    (fp_circle (center 0 0) (end 3.2 0) (layer "Cmts.User") (width 0.15) (fill none))
+    (fp_circle (center 0 0) (end 3.45 0) (layer "F.CrtYd") (width 0.05) (fill none))
+    (pad "" np_thru_hole circle (at 0 0) (size 3.2 3.2) (drill 3.2) (layers *.Cu *.Mask))
   )
   (footprint "Resistor_SMD:R_0603_1608Metric" (layer "F.Cu")
@@
     )
   )
-  (footprint "MountingHole:MountingHole_3mm" (layer "F.Cu")
+  (footprint "MountingHole:MountingHole_3.2mm_M3" (layer "F.Cu")
     (at 31.75 31.75)
-    (descr "Mounting Hole 3mm, no annular")
-    (tags "mounting hole 3mm no annular")
+    (descr "Mounting Hole 3.2mm, no annular, M3")
+    (tags "mounting hole 3.2mm no annular m3")
     (property "Sheetfile" "OBC-Attempt-5_Matcha_2_Layer_3.kicad_sch")
     (property "Sheetname" "")
     (attr exclude_from_pos_files)
-    (fp_text reference "H3" (at 0 -4) (layer "F.Fab")
-      (effects (font (size 1 1) (thickness 0.15)))
-    )
-    (fp_text value "MountingHole" (at 0 4) (layer "F.Fab")
+    (fp_text reference "H3" (at 0 -4.2) (layer "F.SilkS")
+      (effects (font (size 1 1) (thickness 0.15)))
+    )
+    (fp_text value "MountingHole" (at 0 4.2) (layer "F.Fab")
       (effects (font (size 1 1) (thickness 0.15)))
     )
@@
       (effects (font (size 1 1) (thickness 0.15)))
     )
-    (fp_circle (center 0 0) (end 3 0) (layer "Cmts.User") (width 0.15) (fill none))
-    (fp_circle (center 0 0) (end 3.25 0) (layer "F.CrtYd") (width 0.05) (fill none))
-    (pad "" np_thru_hole circle (at 0 0) (size 3 3) (drill 3) (layers *.Cu *.Mask))
+    (fp_circle (center 0 0) (end 3.2 0) (layer "Cmts.User") (width 0.15) (fill none))
+    (fp_circle (center 0 0) (end 3.45 0) (layer "F.CrtYd") (width 0.05) (fill none))
+    (pad "" np_thru_hole circle (at 0 0) (size 3.2 3.2) (drill 3.2) (layers *.Cu *.Mask))
   )
   (footprint "ABMM2_6mm_3_6mm:XTAL_ABMM2-25.000MHZ-D1-T" (layer "F.Cu")
