File: Solenoid Board Ground Systems/Solenoid Board Ground Systems.kicad_sch (KiCad schematic)
At the start: 32 parts, among them J1 OUT CHAN 1, J2 IN CHAN 1, J3 OUT CHAN 2, J4 IN CHAN 2

Commit message: Lots of changes
Parts:
- removed J2: IN CHAN 1, TerminalBlock_Phoenix:TerminalBlock_Phoenix_MPT-0,5-8-2.54_1x08_P2.54mm_Horizontal, symbol Connector:Screw_Terminal_01x08
- removed J4: IN CHAN 2, TerminalBlock_Phoenix:TerminalBlock_Phoenix_MPT-0,5-8-2.54_1x08_P2.54mm_Horizontal, symbol Connector:Screw_Terminal_01x08
- added J2: CHAN IN, TerminalBlock_Phoenix:TerminalBlock_Phoenix_MPT-0,5-9-2.54_1x09_P2.54mm_Horizontal, symbol Connector:Screw_Terminal_01x09
- H1, H2, H3, H4: footprint MountingHole:MountingHole_2.5mm_Pad_TopBottom -> MountingHole:MountingHole_3.2mm_M3_DIN965_Pad_TopBottom
Connections:
- net GND: now also J2.9 (Pin_9)
- net at D16.2 (A), R8.2: now also J2.1 (Pin_1)
- net at D6.2 (A), R3.2: now also J2.6 (Pin_6)
- net at D14.2 (A), R7.2: now also J2.2 (Pin_2)
- net at D12.2 (A), R6.2: now also J2.3 (Pin_3)
- net at D10.2 (A), R5.2: now also J2.4 (Pin_4)
- net at D2.2 (A), R1.2: now also J2.8 (Pin_8)
- net at D8.2 (A), R4.2: now also J2.5 (Pin_5)
- net at D4.2 (A), R2.2: now also J2.7 (Pin_7)

Commit message: Ground System Work
Parts:
- J1: value OUT CHAN 1 -> OUT CHAN A
- J2: value CHAN IN -> POWER IN
- J3: value OUT CHAN 2 -> OUT CHAN B
Connections:
- net GND: now also D10.2 (A), D12.2 (A), D14.2 (A), D16.2 (A), D2.2 (A), D4.2 (A), D6.2 (A), D8.2 (A)
- net POW IN E: now reaches D10.1 (K), D9.1 (K), J3.2 (Pin_2)
- net POW IN E: now also J2.4 (Pin_4), R5.2
- net POW IN F: now reaches D11.1 (K), D12.1 (K), J3.4 (Pin_4)
- net POW IN F: now also J2.3 (Pin_3), R6.2
- net POW IN G: now reaches D13.1 (K), D14.1 (K), J3.6 (Pin_6)
- net POW IN G: now also J2.2 (Pin_2), R7.2
- net POW IN H: now reaches D15.1 (K), D16.1 (K), J3.8 (Pin_8)
- net POW IN H: now also J2.1 (Pin_1), R8.2
- net POW IN D: now reaches J2.5 (Pin_5), R4.2
- net POW IN D: now also D7.1 (K), D8.1 (K), J1.8 (Pin_8); no longer D8.2 (A)
- net POW IN C: now reaches J2.6 (Pin_6), R3.2
- net POW IN C: now also D5.1 (K), D6.1 (K), J1.6 (Pin_6); no longer D6.2 (A)
- net POW IN B: now reaches J2.7 (Pin_7), R2.2
- net POW IN B: now also D3.1 (K), D4.1 (K), J1.4 (Pin_4); no longer D4.2 (A)
- net POW IN A: now reaches J2.8 (Pin_8), R1.2
- net POW IN A: now also D1.1 (K), D2.1 (K), J1.2 (Pin_2); no longer D2.2 (A)
Other:
- note added: "LED BANK"
- note added: "POWER IN"
- note added: "SOLENOIDS OUT"
- note removed: "BOARD SCHEMATIC"
- moved on the sheet: D1, D10, D11, D12, D13, D14, D15, D16, D2, D3, D4, D5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

Commit message: AGS Board Work
Connections:
- net GND: now also D1.1 (K), D11.1 (K), D13.1 (K), D15.1 (K), D3.1 (K), D5.1 (K), D7.1 (K), D9.1 (K)
- net POW IN A: no longer D1.1 (K)
- net POW IN B: no longer D3.1 (K)
- net POW IN C: no longer D5.1 (K)
- net POW IN D: no longer D7.1 (K)
- net POW IN E: no longer D9.1 (K)
- net POW IN F: no longer D11.1 (K)
- net POW IN G: no longer D13.1 (K)
- net POW IN H: no longer D15.1 (K)
Changed lines of the file:
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@@
   (junction (at 195.58 23.495) (diameter 0) (color 0 0 0 0)
   )
+  (junction (at 67.945 24.765) (diameter 0) (color 0 0 0 0)
+  )
   (junction (at 158.75 34.925) (diameter 0) (color 0 0 0 0)
   )
   (junction (at 139.065 46.355) (diameter 0) (color 0 0 0 0)
   )
+  (junction (at 98.425 24.765) (diameter 0) (color 0 0 0 0)
+  )
+  (junction (at 93.345 24.765) (diameter 0) (color 0 0 0 0)
+  )
   (junction (at 123.825 34.925) (diameter 0) (color 0 0 0 0)
   )
+  (junction (at 73.025 24.765) (diameter 0) (color 0 0 0 0)
+  )
   (junction (at 128.905 38.735) (diameter 0) (color 0 0 0 0)
   )
   (junction (at 133.985 42.545) (diameter 0) (color 0 0 0 0)
   )
+  (junction (at 78.105 24.765) (diameter 0) (color 0 0 0 0)
+  )
   (junction (at 190.5 23.495) (diameter 0) (color 0 0 0 0)
   )
+  (junction (at 88.265 24.765) (diameter 0) (color 0 0 0 0)
+  )
   (junction (at 163.83 38.735) (diameter 0) (color 0 0 0 0)
   )
   (junction (at 200.66 23.495) (diameter 0) (color 0 0 0 0)
   )
+  (junction (at 83.185 24.765) (diameter 0) (color 0 0 0 0)
+  )
   (junction (at 173.99 46.355) (diameter 0) (color 0 0 0 0)
   )
@@
     (stroke (width 0) (type default) (color 0 0 0 0))
   )
+  (wire (pts (xy 62.865 24.765) (xy 62.865 25.4))
+    (stroke (width 0) (type default) (color 0 0 0 0))
+  )
   (wire (pts (xy 163.195 42.545) (xy 162.56 42.545))
     (stroke (width 0) (type default) (color 0 0 0 0))
@@
     (stroke (width 0) (type default) (color 0 0 0 0))
   )
+  (wire (pts (xy 93.345 24.765) (xy 88.265 24.765))
+    (stroke (width 0) (type default) (color 0 0 0 0))
+  )
+  (wire (pts (xy 98.425 24.765) (xy 93.345 24.765))
+    (stroke (width 0) (type default) (color 0 0 0 0))
+  )
   (wire (pts (xy 168.275 42.545) (xy 168.91 42.545))
     (stroke (width 0) (type default) (color 0 0 0 0))
@@
     (stroke (width 0) (type default) (color 0 0 0 0))
   )
+  (wire (pts (xy 103.505 24.765) (xy 98.425 24.765))
+    (stroke (width 0) (type default) (color 0 0 0 0))
+  )
   (wire (pts (xy 123.825 34.925) (xy 123.19 34.925))
     (stroke (width 0) (type default) (color 0 0 0 0))
@@
     (stroke (width 0) (type default) (color 0 0 0 0))
   )
+  (wire (pts (xy 88.265 24.765) (xy 83.185 24.765))
+    (stroke (width 0) (type default) (color 0 0 0 0))
+  )
   (wire (pts (xy 171.45 29.21) (xy 171.45 29.845))
     (stroke (width 0) (type default) (color 0 0 0 0))
@@
     (stroke (width 0) (type default) (color 0 0 0 0))
   )
+  (wire (pts (xy 78.105 24.765) (xy 73.025 24.765))
+    (stroke (width 0) (type default) (color 0 0 0 0))
+  )
   (wire (pts (xy 128.27 42.545) (xy 127.635 42.545))
     (stroke (width 0) (type default) (color 0 0 0 0))
@@
     (stroke (width 0) (type default) (color 0 0 0 0))
   )
+  (wire (pts (xy 73.025 24.765) (xy 67.945 24.765))
+    (stroke (width 0) (type default) (color 0 0 0 0))
+  )
   (wire (pts (xy 127.635 42.545) (xy 127.635 43.18))
     (stroke (width 0) (type default) (color 0 0 0 0))
@@
     (stroke (width 0) (type default) (color 0 0 0 0))
   )
+  (wire (pts (xy 67.945 24.765) (xy 62.865 24.765))
+    (stroke (width 0) (type default) (color 0 0 0 0))
+  )
   (wire (pts (xy 173.99 29.21) (xy 173.99 46.355))
     (stroke (width 0) (type default) (color 0 0 0 0))
@@
   )
   (wire (pts (xy 195.58 23.495) (xy 190.5 23.495))
+    (stroke (width 0) (type default) (color 0 0 0 0))
+  )
+  (wire (pts (xy 83.185 24.765) (xy 78.105 24.765))
     (stroke (width 0) (type default) (color 0 0 0 0))
   )
@@
     )
   )
-  (global_label "POW IN G" (shape input) (at 98.425 24.765 90) (fields_autoplaced)
-    (effects (font (size 1 1)) (justify left))
-    (property "Intersheet References" "${INTERSHEET_REFS}" (id 0) (at 98.3625 15.6269 90)
-      (effects (font (size 1 1)) (justify left) hide)
-    )
-  )
   (global_label "POW IN D" (shape input) (at 139.7 46.355 0) (fields_autoplaced)
     (effects (font (size 1 1)) (justify left))
@@
     )
   )
-  (global_label "POW IN E" (shape input) (at 88.265 24.765 90) (fields_autoplaced)
-    (effects (font (size 1 1)) (justify left))
-    (property "Intersheet References" "${INTERSHEET_REFS}" (id 0) (at 88.2025 15.7221 90)
-      (effects (font (size 1 1)) (justify left) hide)
-    )
-  )
   (global_label "POW IN F" (shape input) (at 93.345 40.64 270) (fields_autoplaced)
     (effects (font (size 1 1)) (justify right))
@@
     )
   )
-  (global_label "POW IN H" (shape input) (at 103.505 24.765 90) (fields_autoplaced)
-    (effects (font (size 1 1)) (justify left))
-    (property "Intersheet References" "${INTERSHEET_REFS}" (id 0) (at 103.4425 15.5793 90)
-      (effects (font (size 1 1)) (justify left) hide)
-    )
-  )
   (global_label "POW IN E" (shape input) (at 88.265 40.64 270) (fields_autoplaced)
     (effects (font (size 1 1)) (justify right))
@@
     )
   )
-  (global_label "POW IN B" (shape input) (at 73.025 24.765 90) (fields_autoplaced)
-    (effects (font (size 1 1)) (justify left))
-    (property "Intersheet References" "${INTERSHEET_REFS}" (id 0) (at 72.9625 15.6269 90)
-      (effects (font (size 1 1)) (justify left) hide)
-    )
-  )
-  (global_label "POW IN C" (shape input) (at 78.105 24.765 90) (fields_autoplaced)
-    (effects (font (size 1 1)) (justify left))
-    (property "Intersheet References" "${INTERSHEET_REFS}" (id 0) (at 78.0425 15.6269 90)
-      (effects (font (size 1 1)) (justify left) hide)
-    )
-  )
   (global_label "POW IN A" (shape input) (at 124.46 34.925 0) (fields_autoplaced)
     (effects (font (size 1 1)) (justify left))
     (property "Intersheet References" "${INTERSHEET_REFS}" (id 0) (at 133.4552 34.8625 0)
-      (effects (font (size 1 1)) (justify left) hide)
-    )
-  )
-  (global_label "POW IN A" (shape input) (at 67.945 24.765 90) (fields_autoplaced)
-    (effects (font (size 1 1)) (justify left))
-    (property "Intersheet References" "${INTERSHEET_REFS}" (id 0) (at 67.8825 15.7698 90)
-      (effects (font (size 1 1)) (justify left) hide)
-    )
-  )
-  (global_label "POW IN D" (shape input) (at 83.185 24.765 90) (fields_autoplaced)
-    (effects (font (size 1 1)) (justify left))
-    (property "Intersheet References" "${INTERSHEET_REFS}" (id 0) (at 83.1225 15.6269 90)
-      (effects (font (size 1 1)) (justify left) hide)
-    )
-  )
-  (global_label "POW IN F" (shape input) (at 93.345 24.765 90) (fields_autoplaced)
-    (effects (font (size 1 1)) (justify left))
-    (property "Intersheet References" "${INTERSHEET_REFS}" (id 0) (at 93.2825 15.7698 90)
       (effects (font (size 1 1)) (justify left) hide)
     )
@@
     (pin "2")
   )
+  (symbol (lib_id "power:GND") (at 62.865 25.4 0) (unit 1)
+    (in_bom yes) (on_board yes) (fields_autoplaced)
+    (property "Reference" "#PWR?" (id 0) (at 62.865 31.75 0)
+      (effects (font (size 1.27 1.27)) hide)
+    )
+    (property "Value" "GND" (id 1) (at 62.865 30.48 0)
+      (effects (font (size 1.27 1.27)) hide)
+    )
+    (property "Footprint" "" (id 2) (at 62.865 25.4 0)
+      (effects (font (size 1.27 1.27)) hide)
+    )
+    (property "Datasheet" "" (id 3) (at 62.865 25.4 0)
+      (effects (font (size 1.27 1.27)) hide)
+    )
+    (pin "1")
+  )
   (symbol (lib_id "Device:LED") (at 73.025 29.845 270) (unit 1)
     (in_bom yes) (on_board yes)
@@
       (reference "#PWR?") (unit 1) (value "GND") (footprint "")
     )
+    (path "/d56826c1-00d5-445b-bc3a-5853db726212"
+      (reference "#PWR?") (unit 1) (value "GND") (footprint "")
+    )

Commit message: Some Gerbs Some Work
Parts:
- D10, D12, D14, D16, D2, D4, D6, D8: footprint Diode_SMD:D_SMA -> Diode_THT:D_DO-41_SOD81_P2.54mm_Vertical_AnodeUp
Changed lines of the file:
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@@
       (effects (font (size 1.27 1.27)) (justify left) hide)
     )
-    (property "Footprint" "Diode_SMD:D_SMA" (id 2) (at 120.65 34.925 90)
+    (property "Footprint" "Diode_THT:D_DO-41_SOD81_P2.54mm_Vertical_AnodeUp" (id 2) (at 120.65 34.925 90)
       (effects (font (size 1.27 1.27)) hide)
     )
@@
       (effects (font (size 1.27 1.27)) (justify left) hide)
     )
-    (property "Footprint" "Diode_SMD:D_SMA" (id 2) (at 170.815 46.355 90)
+    (property "Footprint" "Diode_THT:D_DO-41_SOD81_P2.54mm_Vertical_AnodeUp" (id 2) (at 170.815 46.355 90)
       (effects (font (size 1.27 1.27)) hide)
     )
@@
       (effects (font (size 1.27 1.27)) (justify left) hide)
     )
-    (property "Footprint" "Diode_SMD:D_SMA" (id 2) (at 130.81 42.545 90)
+    (property "Footprint" "Diode_THT:D_DO-41_SOD81_P2.54mm_Vertical_AnodeUp" (id 2) (at 130.81 42.545 90)
       (effects (font (size 1.27 1.27)) hide)
     )
@@
       (effects (font (size 1.27 1.27)) (justify left) hide)
     )
-    (property "Footprint" "Diode_SMD:D_SMA" (id 2) (at 160.655 38.735 90)
+    (property "Footprint" "Diode_THT:D_DO-41_SOD81_P2.54mm_Vertical_AnodeUp" (id 2) (at 160.655 38.735 90)
       (effects (font (size 1.27 1.27)) hide)
     )
@@
       (effects (font (size 1.27 1.27)) (justify left) hide)
     )
-    (property "Footprint" "Diode_SMD:D_SMA" (id 2) (at 165.735 42.545 90)
+    (property "Footprint" "Diode_THT:D_DO-41_SOD81_P2.54mm_Vertical_AnodeUp" (id 2) (at 165.735 42.545 90)
       (effects (font (size 1.27 1.27)) hide)
     )
@@
       (effects (font (size 1.27 1.27)) (justify left) hide)
     )
-    (property "Footprint" "Diode_SMD:D_SMA" (id 2) (at 135.89 46.355 90)
+    (property "Footprint" "Diode_THT:D_DO-41_SOD81_P2.54mm_Vertical_AnodeUp" (id 2) (at 135.89 46.355 90)
       (effects (font (size 1.27 1.27)) hide)
     )
@@
       (effects (font (size 1.27 1.27)) (justify left) hide)
     )
-    (property "Footprint" "Diode_SMD:D_SMA" (id 2) (at 125.73 38.735 90)
+    (property "Footprint" "Diode_THT:D_DO-41_SOD81_P2.54mm_Vertical_AnodeUp" (id 2) (at 125.73 38.735 90)
       (effects (font (size 1.27 1.27)) hide)
     )
@@
       (effects (font (size 1.27 1.27)) (justify left) hide)
     )
-    (property "Footprint" "Diode_SMD:D_SMA" (id 2) (at 155.575 34.925 90)
+    (property "Footprint" "Diode_THT:D_DO-41_SOD81_P2.54mm_Vertical_AnodeUp" (id 2) (at 155.575 34.925 90)
       (effects (font (size 1.27 1.27)) hide)
     )
@@
     )
     (path "/49c3db61-1043-403e-be57-cfa7c33467e6"
-      (reference "D2") (unit 1) (value "D_Small") (footprint "Diode_SMD:D_SMA")
+      (reference "D2") (unit 1) (value "D_Small") (footprint "Diode_THT:D_DO-41_SOD81_P2.54mm_Vertical_AnodeUp")
     )
     (path "/d5c57804-d4f1-441c-9336-dca39c2d6ed2"
@@
     )
     (path "/eb517cd7-6c6a-407e-94e4-9054daa45237"
-      (reference "D4") (unit 1) (value "D_Small") (footprint "Diode_SMD:D_SMA")
+      (reference "D4") (unit 1) (value "D_Small") (footprint "Diode_THT:D_DO-41_SOD81_P2.54mm_Vertical_AnodeUp")
     )
     (path "/8755c255-6b28-4909-9018-df776153b310"
@@
     )
     (path "/59a6193f-d073-4986-a006-f1f8447058ee"
-      (reference "D6") (unit 1) (value "D_Small") (footprint "Diode_SMD:D_SMA")
+      (reference "D6") (unit 1) (value "D_Small") (footprint "Diode_THT:D_DO-41_SOD81_P2.54mm_Vertical_AnodeUp")
     )
     (path "/2a79166c-6333-47d2-91d4-96129d1e6405"
@@
     )
     (path "/ce524cfc-4482-4f00-9fcb-ef8673e48a7a"
-      (reference "D8") (unit 1) (value "D_Small") (footprint "Diode_SMD:D_SMA")
+      (reference "D8") (unit 1) (value "D_Small") (footprint "Diode_THT:D_DO-41_SOD81_P2.54mm_Vertical_AnodeUp")
     )
     (path "/fd27f067-6f2c-4456-9579-de12a6c2f4e8"
@@
     )
     (path "/ec35e1dc-1b31-441e-ba9d-09a62f23042c"
-      (reference "D10") (unit 1) (value "D_Small") (footprint "Diode_SMD:D_SMA")
+      (reference "D10") (unit 1) (value "D_Small") (footprint "Diode_THT:D_DO-41_SOD81_P2.54mm_Vertical_AnodeUp")
     )
     (path "/270cecef-3be6-4c4a-a31d-ac220064c9c1"
@@
     )
     (path "/77c22556-98ca-4ffb-9d51-06a9698a3659"
-      (reference "D12") (unit 1) (value "D_Small") (footprint "Diode_SMD:D_SMA")
+      (reference "D12") (unit 1) (value "D_Small") (footprint "Diode_THT:D_DO-41_SOD81_P2.54mm_Vertical_AnodeUp")
     )
     (path "/ec881cd0-a082-4b99-8e4a-dd013d1d4f3d"
@@
     )
     (path "/966c473e-b0a5-4933-98d3-bb1e9e88a242"
-      (reference "D14") (unit 1) (value "D_Small") (footprint "Diode_SMD:D_SMA")
+      (reference "D14") (unit 1) (value "D_Small") (footprint "Diode_THT:D_DO-41_SOD81_P2.54mm_Vertical_AnodeUp")
     )
     (path "/537a9b92-68e3-4e21-b593-4ea57da46157"
@@
     )
     (path "/5725a608-2b64-431b-8170-c5c55d69b366"
-      (reference "D16") (unit 1) (value "D_Small") (footprint "Diode_SMD:D_SMA")
+      (reference "D16") (unit 1) (value "D_Small") (footprint "Diode_THT:D_DO-41_SOD81_P2.54mm_Vertical_AnodeUp")
     )
     (path "/b26fd2b8-4112-417c-8697-2c75192f2809"

Commit message: Reworked the solenoid board
Parts:
- removed D10, D12, D14, D16, D2, D4, D6, D8: D_Small, Diode_THT:D_DO-41_SOD81_P2.54mm_Vertical_AnodeUp, symbol Device:D_Small
- added D10, D11, D12, D9: MMBZxx, Package_TO_SOT_SMD:SOT-23, symbol Diode:MMBZxx
- renumbered D3 to D2, D5 to D3, D7 to D4, D9 to D5, D11 to D6, D13 to D7, D15 to D8
Connections:
- net GND: now also D10.3 (A), D11.3 (A), D12.3 (A), D9.3 (A)
- net POW IN A: now also D9.1 (K)
- net POW IN B: now also D9.2 (K)
- net POW IN C: now also D10.1 (K)
- net POW IN D: now also D10.2 (K)
- net POW IN E: now also D11.1 (K)
- net POW IN F: now also D11.2 (K)
- net POW IN G: now also D12.1 (K)
- net POW IN H: now also D12.2 (K)
Other:
- moved on the sheet: J1, J3
