File: RFD900 Interface/RFD900 Interface.kicad_sch (KiCad schematic)
At the start: 1 part

Commit message: added all the things for can
Parts:
- added C?: 1uF, Capacitor_SMD:C_0402_1005Metric, symbol Device:C
- added C? (x2): .1uF, Capacitor_SMD:C_0402_1005Metric, symbol Device:C
- added C?: 4u7, Capacitor_SMD:C_0402_1005Metric, symbol Device:C
- added C? (x2): 20pF, Capacitor_SMD:C_0402_1005Metric, symbol Device:C
- added C?: 10uF, Capacitor_SMD:C_0603_1608Metric, symbol Device:C
- added C?: 10nF, Capacitor_SMD:C_0402_1005Metric, symbol Device:C
- added C?: 4.7nF, Capacitor_SMD:C_0402_1005Metric, symbol Device:C
- added J? (x2): Bat, Connector_PinHeader_1.00mm:PinHeader_1x02_P1.00mm_Vertical, symbol Connector:Conn_01x02_Female
- added J?: DEBUG, Connector_PinHeader_1.00mm:PinHeader_1x02_P1.00mm_Vertical, symbol Connector:Conn_01x04_Female
- added J?: CAN Header, Connector_PinHeader_1.00mm:PinHeader_1x04_P1.00mm_Vertical, symbol Connector:Conn_01x04_Female
- added R?: 10k, Resistor_SMD:R_0402_1005Metric, symbol Device:R
- added R? (x2): 60 ohm, Resistor_SMD:R_0805_2012Metric, symbol Device:R
- added SW?: SW_SPST, Jumper:SolderJumper-2_P1.3mm_Open_RoundedPad1.0x1.5mm, symbol Switch:SW_SPST
- added SW?: SW_SPDT, Jumper:SolderJumper-3_P1.3mm_Open_RoundedPad1.0x1.5mm_NumberLabels, symbol Switch:SW_SPDT
- added U?: LD1117S33TR_SOT223, Package_TO_SOT_SMD:SOT-223-3_TabPin2, symbol Regulator_Linear:LD1117S33TR_SOT223
- added U?: SN65HVD230, Package_SO:SOIC-8_3.9x4.9mm_P1.27mm, symbol Interface_CAN_LIN:SN65HVD230
- added U?: STM32F042G4Ux, Package_DFN_QFN:QFN-28_4x4mm_P0.5mm, symbol MCU_ST_STM32F0:STM32F042G4Ux
- added X?: ECS-2520MV-xxx-xx, Oscillator:Oscillator_SMD_ECS_2520MV-xxx-xx-4Pin_2.5x2.0mm, symbol Oscillator:ECS-2520MV-xxx-xx
Connections:
- new net: R?.2, SW?.2 (B)
- new net: R?.1, SW?.1 (A)
- new net: C?.1, R?.1, R?.2
- new net +3.3V: C?.1, C?.1, C?.1, C?.1, C?.1, J?.1 (Pin_1), SW?.3 (C), U?.17 (VDD), U?.18 (VDDIO2), U?.2 (VO), U?.3 (VCC), U?.5 (VDDA)
- new net 12V+: C?.1, J?.2 (Pin_2), J?.2 (Pin_2), U?.3 (VI)
- new net BOOT0: R?.1, U?.4 (NRST)
- new net CAN_H: J?.3 (Pin_3), J?.4 (Pin_4), SW?.2 (B), U?.7 (CANH)
- new net CAN_L: J?.1 (Pin_1), J?.2 (Pin_2), R?.2, U?.6 (CANL)
- new net CAN_RX: U?.1 (PB8), U?.4 (R)
- new net CAN_TX: U?.1 (D), U?.20 (PA10/PA12)
- new net GND: C?.2, C?.2, C?.2, C?.2, C?.2, C?.2, C?.2, C?.2, C?.2, J?.1 (Pin_1), J?.1 (Pin_1), J?.4 (Pin_4), SW?.1 (A), U?.1 (GND), U?.16 (VSSA), U?.2 (GND), U?.8 (Rs), X?.2 (GND), X?.4 (VDD)
- new net RCC_OSC_IN: C?.1, U?.2 (PF0), X?.1 (Tri-State)
- new net RCC_OSC_OUT: C?.1, U?.3 (PF1), X?.3 (OUT)
- new net SYS_SWCLK: J?.3 (Pin_3), U?.22 (PA14)
- new net SYS_SWDIO: J?.2 (Pin_2), U?.21 (PA13)
- new net USART1_RX: U?.28 (PB7)
- new net USART1_TX: U?.27 (PB6)
Other:
- note added: "Debug"
- note added: "Decoupling Caps"
- note added: "Microcontroller"
- note added: "Oscillator"
- note added: "Output: 3.3V 800ma Input: 15V max"
- note added: "Power Supply"
- note added: "Run/Debug"
- note added: "STM32"
- note added: "Transciever (CAN)"
- moved on the sheet: J?

Commit message: AGS Board Work
Other:
- moved on the sheet: C?, J?, R?, SW?, U?

Commit message: some changes
Parts:
- J?: footprint (none) -> Connector_PinHeader_2.54mm:PinHeader_2x08_P2.54mm_Horizontal
Changed lines of the file:
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@@
       (effects (font (size 1.27 1.27)) (justify left) hide)
     )
-    (property "Footprint" "" (id 2) (at 257.175 46.99 0)
+    (property "Footprint" "Connector_PinHeader_2.54mm:PinHeader_2x08_P2.54mm_Horizontal" (id 2) (at 257.175 46.99 0)
       (effects (font (size 1.27 1.27)) hide)
     )
@@
     )
     (path "/475f8da9-d37c-4d78-9b1e-987b8b87d7f1"
-      (reference "J?") (unit 1) (value "Conn_02x08_Odd_Even") (footprint "")
+      (reference "J?") (unit 1) (value "Conn_02x08_Odd_Even") (footprint "Connector_PinHeader_2.54mm:PinHeader_2x08_P2.54mm_Horizontal")
     )
     (path "/db7f65d0-b56b-4155-a900-b3cbec3e04b8"

Commit message: RFD900 Work
Made the whole board
Parts:
- removed J?: Bat, Connector_PinHeader_1.00mm:PinHeader_1x02_P1.00mm_Vertical, symbol Connector:Conn_01x02_Female
- added C1: .1uF, Capacitor_SMD:C_0402_1005Metric, symbol Device:C
- added C3: 10uF, Capacitor_SMD:C_0603_1608Metric, symbol Device:C
- added U2: LD1117S50TR_SOT223, Package_TO_SOT_SMD:SOT-223-3_TabPin2, symbol Regulator_Linear:LD1117S50TR_SOT223
- J1: renamed from J?; footprint Connector_PinHeader_1.00mm:PinHeader_1x02_P1.00mm_Vertical -> Connector_PinHeader_2.54mm:PinHeader_1x04_P2.54mm_Vertical; symbol Connector:Conn_01x02_Female -> Connector:Conn_01x04_Male
- J2: renamed from J?; footprint Connector_PinHeader_1.00mm:PinHeader_1x02_P1.00mm_Vertical -> Connector_PinHeader_2.54mm:PinHeader_1x04_P2.54mm_Vertical; symbol Connector:Conn_01x04_Female -> Connector:Conn_01x04_Male
- J3: renamed from J?; footprint Connector_PinHeader_1.00mm:PinHeader_1x04_P1.00mm_Vertical -> Connector_PinHeader_2.54mm:PinHeader_1x04_P2.54mm_Vertical
- J4: renamed from J?; footprint Connector_PinHeader_2.54mm:PinHeader_2x08_P2.54mm_Horizontal -> Connector_PinSocket_2.54mm:PinSocket_2x08_P2.54mm_Horizontal
- gave numbers to parts that had none: 18
Connections:
- net 12V+: now also J1.1 (Pin_1), C1.1, U2.3 (VI)
- net GND: now also J1.3 (Pin_3), J1.4 (Pin_4), J4.1 (Pin_1), J4.16 (Pin_16), J4.2 (Pin_2), C1.2, C3.2, U2.1 (GND); no longer J1.1 (Pin_1)
- net SYS_SWCLK: now also J2.2 (Pin_2); no longer J2.3 (Pin_3)
- net SYS_SWDIO: now also J2.3 (Pin_3); no longer J2.2 (Pin_2)
- net USART1_RX: now also J4.7 (Pin_7)
- net USART1_TX: now also J4.9 (Pin_9)
- net GPIO4: now reaches J4.10 (Pin_10)
- net RTS: now reaches J4.11 (Pin_11)
- net GPIO3: now reaches J4.12 (Pin_12)
- net GPIO0: now reaches J4.13 (Pin_13)
- net GPIO2: now reaches J4.14 (Pin_14)
- net GPIO1: now reaches J4.15 (Pin_15)
- net CTS: now reaches J4.3 (Pin_3)
- net +5V: now reaches J4.4 (Pin_4)
- net +5V: now also C3.1, U2.2 (VO)
- net VUSB: now reaches J4.5 (Pin_5)
- net VUSB: now also J4.6 (Pin_6)
- net GPIO5: now reaches J4.8 (Pin_8)
Other:
- note added: "Output: 3.3V 800ma Output: 5V 800ma Input: 15V max"
- note removed: "Output: 3.3V 800ma Input: 15V max"
- moved on the sheet: C2, C4, J4, U3
