File: RFD900 Interface/RFD900 Interface.kicad_pcb (KiCad board)
At the start: 2 copper layers, 25.4 x 34.3 mm, 25 parts, among them J1 Bat, J2 DEBUG, J3 CAN Header, J4 Conn_02x08_Odd_Even, SW1 SW_SPST, SW2 SW_SPDT, U1 SN65HVD230, U2 LD1117S50TR_SOT223, U3 LD1117S33TR_SOT223, U4 STM32F042G4Ux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

Commit message: Some misc work
Routing:
- net GND: track 11.6 -> 14.1 mm
