File: Power Supply Board Ground Systems V1.1/Power Supply Board Ground Systems V1.1.kicad_sch (KiCad schematic)
At the start: 32 parts, among them J1 POWER, J2 POWER OUT, SW1 SW_SPDT, SW2 SW_SPDT, SW3 SW_SPDT, SW4 SW_SPDT, SW5 SW_SPDT, SW6 SW_SPDT, SW7 SW_SPDT, SW8 SW_SPDT

Commit message: Changed all the things to 5mm pitch
yuck big board be like
Parts:
- J1: footprint TerminalBlock_Phoenix:TerminalBlock_Phoenix_MPT-0,5-2-2.54_1x02_P2.54mm_Horizontal -> TerminalBlock_Phoenix:TerminalBlock_Phoenix_PT-1,5-2-5.0-H_1x02_P5.00mm_Horizontal
- J2: footprint TerminalBlock_Phoenix:TerminalBlock_Phoenix_MPT-0,5-8-2.54_1x08_P2.54mm_Horizontal -> TerminalBlock_Phoenix:TerminalBlock_Phoenix_PT-1,5-8-5.0-H_1x08_P5.00mm_Horizontal

Commit message: Revions and new board
Parts:
- removed J1: POWER, TerminalBlock_Phoenix:TerminalBlock_Phoenix_PT-1,5-2-5.0-H_1x02_P5.00mm_Horizontal, symbol Connector:Screw_Terminal_01x02
- removed J2: POWER OUT, TerminalBlock_Phoenix:TerminalBlock_Phoenix_PT-1,5-8-5.0-H_1x08_P5.00mm_Horizontal, symbol Connector:Screw_Terminal_01x08
- added J3: TBLH10V-350-02BK, RHDR4W80P550X350_2X2_770X850X1420P, symbol TBLH10V-350-02BK:TBLH10V-350-02BK
- added J4: TBLH10V-350-08BK, RHDR16W80P550X350_2X8_2870X850X1420P, symbol TBLH10V-350-08BK:TBLH10V-350-08BK
Connections:
- net GND: now also J3.3, J3.4
- net OUT1: now also J4.1, J4.2
- net OUT2: now also J4.3, J4.4
- net OUT3: now also J4.5, J4.6
- net OUT4: now also J4.7, J4.8
- net OUT5: now also J4.10, J4.9
- net OUT6: now also J4.11, J4.12
- net OUT7: now also J4.13, J4.14
- net OUT8: now also J4.15, J4.16
- net POW IN: now also J3.1, J3.2
