File: DeploymentBoardV2.0/DeploymentBoardV2.0.kicad_pcb (KiCad board)
At the start: 4 copper layers, 20.3 x 38.1 mm, 50 parts, among them IC1 MCP2557FDT-H_MNY, IC2 AP2205-33W5-7, J1 Conn_01x04_Socket, J2 Conn_01x04_Socket, J3 Conn_01x04_Socket, J6 PYRO CHANNELS, Q1 SSM6N58NU,LF, SW1 SW_SPDT, SW2 SW_SPST, U1 STM32G473CBTx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

Commit message: Finished Board
Name: OH CHUTE!
Parts:
- added G***: LOGO, LOGO, F.Cu at (38.3, 42.0)
- D1, D2, D3, D4: footprint Capacitor_SMD:C_0402_1005Metric -> LED_SMD:LED_0402_1005Metric
- moved H4 49.3 mm to (27.9, 54.6)
- moved H3 33.3 mm to (43.2, 54.6), turned to 45 degrees
- moved D1 2.76 mm to (31.9, 52.4), turned to 180 degrees
- moved R8 2.76 mm to (30.0, 52.4)
- moved J1 2.69 mm to (39.7, 54.4)
- moved C9 2.50 mm to (35.4, 37.2), turned to 180 degrees
- moved R6 0.98 mm to (29.1, 34.6)
- moved C5 0.66 mm to (35.7, 46.4)
- moved IC2 0.62 mm to (39.0, 36.6)
- moved C14 0.62 mm to (39.6, 34.0)
- moved J2 0.62 mm to (43.8, 43.4)
- moved C10 0.56 mm to (30.6, 41.5)
- moved C11 0.52 mm to (33.9, 49.6)
- moved C12 0.52 mm to (42.2, 48.5)
- moved R2 0.52 mm to (40.6, 46.2)
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Connections:
- C11 pad 1: PWR IN -> BATT+
- IC1 pad 3: PWR IN -> BATT+
- J1 pad 3: GND -> +3.3V
- J1 pad 4: +3.3V -> GND
- U1 pad 32: unconnected-(U1-PA10-Pad32) -> TXD
- U1 pad 42: TXD -> unconnected-(U1-PB5-Pad42)
Routing:
- net BATT+: track 3.91 -> 19.0 mm
- net GND: track 23.5 -> 33.9 mm, vias 20 -> 29
- net CAN_FD_H: track 0.00 -> 8.98 mm, vias 0 -> 1
- net CAN_FD_L: track 0.00 -> 8.79 mm
- net SYS_SWDIO: track 0.00 -> 8.01 mm
- net SYS_SWCLK: track 0.00 -> 7.17 mm
- net +3.3V: track 13.0 -> 19.6 mm, vias 5 -> 9
- net FDCAN_RX: track 0.00 -> 5.07 mm, vias 0 -> 1
- net TXD: track 0.00 -> 4.39 mm, vias 0 -> 1
- net FDCAN_TX: track 0.00 -> 3.20 mm, vias 0 -> 1
- net Net-(C12-Pad2): track 0.00 -> 3.12 mm
- net Net-(SW2-B): track 0.00 -> 2.91 mm, vias 0 -> 1
- net LED_1: track 0.00 -> 1.87 mm, vias 0 -> 1
- net Net-(D1-A): track 0.00 -> 0.98 mm
- net Net-(D2-A): track 0.00 -> 0.95 mm
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- added copper zone on F.Cu, net GND
Other:
- board size 20.3 x 38.1 mm -> 20.3 x 31.8 mm
- board text added: "-BATT+"
- board text added: "3.3"
- board text added: "ALEX AARHUS"
- board text added: "APOGEE"
- board text added: "CAN TERM RES"
- board text added: "CAN_H"
- board text added: "CAN_L"
- board text added: "CLK"
- board text added: "DIO"
- board text added: "GND"
- board text added: "OHHH CHUTE!"
- board text added: "SDSURP 2023"
- board text added: "SWITCH"

Commit message: GERBS!
Changed lines of the file:
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@@
       (plot_on_all_layers_selection 0x0000000_00000000)
       (disableapertmacros false)
-      (usegerberextensions false)
-      (usegerberattributes true)
-      (usegerberadvancedattributes true)
-      (creategerberjobfile true)
+      (usegerberextensions true)
+      (usegerberattributes false)
+      (usegerberadvancedattributes false)
+      (creategerberjobfile false)
       (dashed_line_dash_ratio 12.000000)
       (dashed_line_gap_ratio 3.000000)
@@
       (psa4output false)
       (plotreference true)
-      (plotvalue true)
+      (plotvalue false)
       (plotinvisibletext false)
       (sketchpadsonfab false)
-      (subtractmaskfromsilk false)
+      (subtractmaskfromsilk true)
       (outputformat 1)
       (mirror false)
-      (drillshape 1)
+      (drillshape 0)
       (scaleselection 1)
-      (outputdirectory "")
+      (outputdirectory "Gerbs/")
     )
   )
@@
     (fp_line (start 1 0.625) (end -1 0.625)
       (stroke (width 0.1) (type solid)) (layer "F.Fab"))
-    (pad "1" smd roundrect (at -0.9125 0 270) (size 1.025 1.4) (layers "F.Cu" "F.Paste" "F.Mask") (roundrect_rratio 0.243902)
+    (pad "1" smd roundrect (at -0.9125 0 270) (size 1.025 1.4) (layers "F.Cu" "F.Paste" "F.Mask") (roundrect_rratio 0.243902439)
       (net 33 "Net-(SW2-B)") (pintype "passive"))
-    (pad "2" smd roundrect (at 0.9125 0 270) (size 1.025 1.4) (layers "F.Cu" "F.Paste" "F.Mask") (roundrect_rratio 0.243902)
+    (pad "2" smd roundrect (at 0.9125 0 270) (size 1.025 1.4) (layers "F.Cu" "F.Paste" "F.Mask") (roundrect_rratio 0.243902439)
       (net 6 "Net-(C12-Pad2)") (pintype "passive"))
     (model "${KICAD6_3DMODEL_DIR}/Resistor_SMD.3dshapes/R_0805_2012Metric.wrl"
@@
     (fp_line (start 1 0.625) (end -1 0.625)
       (stroke (width 0.1) (type solid)) (layer "F.Fab"))
-    (pad "1" smd roundrect (at -0.9125 0 270) (size 1.025 1.4) (layers "F.Cu" "F.Paste" "F.Mask") (roundrect_rratio 0.243902)
+    (pad "1" smd roundrect (at -0.9125 0 270) (size 1.025 1.4) (layers "F.Cu" "F.Paste" "F.Mask") (roundrect_rratio 0.243902439)
       (net 6 "Net-(C12-Pad2)") (pintype "passive"))
-    (pad "2" smd roundrect (at 0.9125 0 270) (size 1.025 1.4) (layers "F.Cu" "F.Paste" "F.Mask") (roundrect_rratio 0.243902)
+    (pad "2" smd roundrect (at 0.9125 0 270) (size 1.025 1.4) (layers "F.Cu" "F.Paste" "F.Mask") (roundrect_rratio 0.243902439)
       (net 13 "CAN_FD_L") (pintype "passive"))
     (model "${KICAD6_3DMODEL_DIR}/Resistor_SMD.3dshapes/R_0805_2012Metric.wrl"
