File: VoltageDivPCB/VoltageDivPCB.kicad_sch (KiCad schematic)
At the start: 6 parts, among them J1 Conn_01x04

Commit message: Lab jack work
Parts:
- removed H1: MountingHole_Pad, MountingHole:MountingHole_2.1mm, symbol Mechanical:MountingHole
- removed J1: Conn_01x04, Connector_PinHeader_2.54mm:PinHeader_1x04_P2.54mm_Vertical, symbol Connector_Generic:Conn_01x04
- added J1: FWS-04-02-T-S-RA, FWS0402TSRA, symbol FWS-04-02-T-S-RA:FWS-04-02-T-S-RA
- added J2: Screw_Terminal_01x04, TerminalBlock_Phoenix:TerminalBlock_Phoenix_PT-1,5-4-3.5-H_1x04_P3.50mm_Horizontal, symbol Connector:Screw_Terminal_01x04
Connections:
- net GND: now also J1.2, J2.4 (Pin_4)
- net V In: now also J2.1 (Pin_1), J2.2 (Pin_2)
- net V Out: now also J1.3, J2.3 (Pin_3)
- no-connect marks 0 -> 2
Other:
- moved on the sheet: R1, R2, R3, R4
