File: AnalogStandPCBify1_PowerDistribution/AnalogStandPCBify1_PowerDistribution.kicad_sch (KiCad schematic)
At the start: 0 parts

Commit message: Analog stand stuffs
Parts:
- added BT1: 24V+, symbol Device:Battery
- added D1, D2, D3, D4: D, symbol Device:D
- added L1, L2, L3, L4: L, symbol Device:L
- added SW1, SW2, SW3, SW4: SOL_SW, symbol Switch:SW_SPST
Connections:
- new net: BT1.1 (+), SW1.1 (A), SW2.1 (A), SW3.1 (A), SW4.1 (A)
- new net: D4.1 (K), L4.1, SW4.2 (B)
- new net: D2.1 (K), L2.1, SW2.2 (B)
- new net: D1.1 (K), L1.1, SW1.2 (B)
- new net: D3.1 (K), L3.1, SW3.2 (B)
- new net GND: BT1.2 (-), D1.2 (A), D2.2 (A), D3.2 (A), D4.2 (A), L1.2, L2.2, L3.2, L4.2

Commit message: Train work
Parts:
- BT1: footprint (none) -> Connector_Wire:SolderWire-1.5sqmm_1x02_P6mm_D1.7mm_OD3mm_Relief
- D1, D2, D3, D4: footprint (none) -> Diode_THT:D_A-405_P7.62mm_Horizontal
- L1, L2, L3, L4: footprint (none) -> Connector_Wire:SolderWire-1sqmm_1x02_P5.4mm_D1.4mm_OD2.7mm_Relief
- SW1, SW2, SW3, SW4: footprint (none) -> Connector_Wire:SolderWire-1.5sqmm_1x02_P7.8mm_D1.7mm_OD3.9mm_Relief
Changed lines of the file:
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@@
       (effects (font (size 1.27 1.27)) (justify left))
     )
-    (property "Footprint" "" (at 59.69 67.691 90)
+    (property "Footprint" "Connector_Wire:SolderWire-1.5sqmm_1x02_P6mm_D1.7mm_OD3mm_Relief" (at 59.69 67.691 90)
       (effects (font (size 1.27 1.27)) hide)
     )
@@
       (effects (font (size 1.27 1.27)) (justify left))
     )
-    (property "Footprint" "" (at 107.315 99.695 0)
+    (property "Footprint" "Connector_Wire:SolderWire-1sqmm_1x02_P5.4mm_D1.4mm_OD2.7mm_Relief" (at 107.315 99.695 0)
       (effects (font (size 1.27 1.27)) hide)
     )
@@
       (effects (font (size 1.27 1.27)) (justify left))
     )
-    (property "Footprint" "" (at 98.425 63.5 0)
+    (property "Footprint" "Diode_THT:D_A-405_P7.62mm_Horizontal" (at 98.425 63.5 0)
       (effects (font (size 1.27 1.27)) hide)
     )
@@
       (effects (font (size 1.27 1.27)) (justify left))
     )
-    (property "Footprint" "" (at 98.425 45.085 0)
+    (property "Footprint" "Diode_THT:D_A-405_P7.62mm_Horizontal" (at 98.425 45.085 0)
       (effects (font (size 1.27 1.27)) hide)
     )
@@
       (effects (font (size 1.27 1.27)))
     )
-    (property "Footprint" "" (at 88.9 94.615 0)
+    (property "Footprint" "Connector_Wire:SolderWire-1.5sqmm_1x02_P7.8mm_D1.7mm_OD3.9mm_Relief" (at 88.9 94.615 0)
       (effects (font (size 1.27 1.27)) hide)
     )
@@
       (effects (font (size 1.27 1.27)) (justify left))
     )
-    (property "Footprint" "" (at 107.315 45.085 0)
+    (property "Footprint" "Connector_Wire:SolderWire-1sqmm_1x02_P5.4mm_D1.4mm_OD2.7mm_Relief" (at 107.315 45.085 0)
       (effects (font (size 1.27 1.27)) hide)
     )
@@
       (effects (font (size 1.27 1.27)) (justify left))
     )
-    (property "Footprint" "" (at 98.425 81.28 0)
+    (property "Footprint" "Diode_THT:D_A-405_P7.62mm_Horizontal" (at 98.425 81.28 0)
       (effects (font (size 1.27 1.27)) hide)
     )
@@
       (effects (font (size 1.27 1.27)) (justify left))
     )
-    (property "Footprint" "" (at 107.315 81.28 0)
+    (property "Footprint" "Connector_Wire:SolderWire-1sqmm_1x02_P5.4mm_D1.4mm_OD2.7mm_Relief" (at 107.315 81.28 0)
       (effects (font (size 1.27 1.27)) hide)
     )
@@
       (effects (font (size 1.27 1.27)) (justify left))
     )
-    (property "Footprint" "" (at 107.315 63.5 0)
+    (property "Footprint" "Connector_Wire:SolderWire-1sqmm_1x02_P5.4mm_D1.4mm_OD2.7mm_Relief" (at 107.315 63.5 0)
       (effects (font (size 1.27 1.27)) hide)
     )
@@
       (effects (font (size 1.27 1.27)) (justify left))
     )
-    (property "Footprint" "" (at 98.425 99.695 0)
+    (property "Footprint" "Diode_THT:D_A-405_P7.62mm_Horizontal" (at 98.425 99.695 0)
       (effects (font (size 1.27 1.27)) hide)
     )
@@
       (effects (font (size 1.27 1.27)))
     )
-    (property "Footprint" "" (at 89.535 58.42 0)
+    (property "Footprint" "Connector_Wire:SolderWire-1.5sqmm_1x02_P7.8mm_D1.7mm_OD3.9mm_Relief" (at 89.535 58.42 0)
       (effects (font (size 1.27 1.27)) hide)
     )
@@
       (effects (font (size 1.27 1.27)))
     )
-    (property "Footprint" "" (at 89.535 76.2 0)
+    (property "Footprint" "Connector_Wire:SolderWire-1.5sqmm_1x02_P7.8mm_D1.7mm_OD3.9mm_Relief" (at 89.535 76.2 0)
       (effects (font (size 1.27 1.27)) hide)
     )
@@
       (effects (font (size 1.27 1.27)))
     )
-    (property "Footprint" "" (at 89.535 40.005 0)
-      (effects (font (size 1.27 1.27)) hide)
-    )
+    (property "Footprint" "Connector_Wire:SolderWire-1.5sqmm_1x02_P7.8mm_D1.7mm_OD3.9mm_Relief" (at 89.535 40.005 0)
+      (effects (font (size 1.27 1.27)) hide)
+    )

Commit message: Push
Parts:
- BT1: footprint Connector_Wire:SolderWire-1.5sqmm_1x02_P6mm_D1.7mm_OD3mm_Relief -> Connector_Wire:SolderWire-1.5sqmm_1x02_P7.8mm_D1.7mm_OD3.9mm_Relief
Connections:
- net 24V+: now reaches BT1.1 (+), SW1.1 (A), SW2.1 (A), SW3.1 (A), SW4.1 (A)
Changed lines of the file:
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@@
     (stroke (width 0) (type default))
+  )
+  (label "24V+" (at 59.69 40.005 0) (fields_autoplaced)
+    (effects (font (size 1.27 1.27)) (justify left bottom))
   )
   (symbol (lib_id "power:GND") (at 98.425 106.045 0) (unit 1)
@@
       (effects (font (size 1.27 1.27)) (justify left))
     )
-    (property "Footprint" "Connector_Wire:SolderWire-1.5sqmm_1x02_P6mm_D1.7mm_OD3mm_Relief" (at 59.69 67.691 90)
+    (property "Footprint" "Connector_Wire:SolderWire-1.5sqmm_1x02_P7.8mm_D1.7mm_OD3.9mm_Relief" (at 59.69 67.691 90)
       (effects (font (size 1.27 1.27)) hide)
     )

Commit message: A
Changed lines of the file:
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@@
   (junction (at 77.47 40.005) (diameter 0) (color 0 0 0 0)
   )
+  (junction (at 98.425 50.8) (diameter 0) (color 0 0 0 0)
+  )
   (junction (at 98.425 68.58) (diameter 0) (color 0 0 0 0)
   )
-  (junction (at 98.425 50.165) (diameter 0) (color 0 0 0 0)
-  )
   (junction (at 98.425 104.775) (diameter 0) (color 0 0 0 0)
   )
@@
     (stroke (width 0) (type default))
   )
+  (wire (pts (xy 98.425 50.8) (xy 98.425 48.895))
+    (stroke (width 0) (type default))
+  )
   (wire (pts (xy 98.425 67.31) (xy 98.425 68.58))
     (stroke (width 0) (type default))
   )
-  (wire (pts (xy 98.425 48.895) (xy 98.425 50.165))
-    (stroke (width 0) (type default))
-  )
   (wire (pts (xy 93.98 94.615) (xy 98.425 94.615))
     (stroke (width 0) (type default))
@@
     (stroke (width 0) (type default))
   )
+  (wire (pts (xy 107.315 48.895) (xy 107.315 50.8))
+    (stroke (width 0) (type default))
+  )
   (wire (pts (xy 107.315 85.09) (xy 107.315 86.36))
     (stroke (width 0) (type default))
@@
     (stroke (width 0) (type default))
   )
+  (wire (pts (xy 98.425 52.07) (xy 98.425 50.8))
+    (stroke (width 0) (type default))
+  )
   (wire (pts (xy 107.315 86.36) (xy 98.425 86.36))
     (stroke (width 0) (type default))
@@
     (stroke (width 0) (type default))
   )
-  (wire (pts (xy 107.315 48.895) (xy 107.315 50.165))
-    (stroke (width 0) (type default))
-  )
   (wire (pts (xy 107.315 68.58) (xy 98.425 68.58))
     (stroke (width 0) (type default))
@@
     (stroke (width 0) (type default))
   )
+  (wire (pts (xy 107.315 50.8) (xy 98.425 50.8))
+    (stroke (width 0) (type default))
+  )
   (wire (pts (xy 107.315 104.775) (xy 98.425 104.775))
     (stroke (width 0) (type default))
   )
-  (wire (pts (xy 98.425 51.435) (xy 98.425 50.165))
-    (stroke (width 0) (type default))
-  )
   (wire (pts (xy 94.615 58.42) (xy 98.425 58.42))
     (stroke (width 0) (type default))
@@
   )
   (wire (pts (xy 98.425 76.2) (xy 107.315 76.2))
-    (stroke (width 0) (type default))
-  )
-  (wire (pts (xy 107.315 50.165) (xy 98.425 50.165))
     (stroke (width 0) (type default))
   )
@@
     )
   )
-  (symbol (lib_id "power:GND") (at 98.425 51.435 0) (unit 1)
-    (in_bom yes) (on_board yes) (dnp no) (fields_autoplaced)
-    (property "Reference" "#PWR02" (at 98.425 57.785 0)
-      (effects (font (size 1.27 1.27)) hide)
-    )
-    (property "Value" "GND" (at 98.425 55.88 0)
-      (effects (font (size 1.27 1.27)))
-    )
-    (property "Footprint" "" (at 98.425 51.435 0)
-      (effects (font (size 1.27 1.27)) hide)
-    )
-    (property "Datasheet" "" (at 98.425 51.435 0)
-      (effects (font (size 1.27 1.27)) hide)
-    )
+  (symbol (lib_id "power:GND") (at 98.425 52.07 0) (unit 1)
+    (in_bom yes) (on_board yes) (dnp no) (fields_autoplaced)
+    (property "Reference" "#PWR02" (at 98.425 58.42 0)
+      (effects (font (size 1.27 1.27)) hide)
+    )
+    (property "Value" "GND" (at 98.425 56.515 0)
+      (effects (font (size 1.27 1.27)))
+    )
+    (property "Footprint" "" (at 98.425 52.07 0)
+      (effects (font (size 1.27 1.27)) hide)
+    )
+    (property "Datasheet" "" (at 98.425 52.07 0)
+      (effects (font (size 1.27 1.27)) hide)
+    )
