File: EthBreakoutBoard/EthBreakoutBoard.kicad_sch (KiCad schematic)
At the start: 2 parts, among them J1 1091946, J2 TBLH10V-350-09BK

Commit message: Push
Parts:
- removed J1: 1091946, 1091946:PHOENIX_1091946, symbol 1091946:1091946
- removed J2: TBLH10V-350-09BK, RHDR18W80P550X350_2X9_3220X850X1420P, symbol TBLH10V-350-09BK:TBLH10V-350-09BK
- added H1, H2: MountingHole, MountingHole:MountingHole_3.2mm_M3, symbol Mechanical:MountingHole
- added J1: TBLH10V-350-08BK, TBLH10V-350-08BK:RHDR16W80P550X350_2X8_2870X850X1420P, symbol TBLH10V-350-08BK:TBLH10V-350-08BK
- added J2: MTJ-889X1, MTJ-889X1:CONN_MTJ-889X1_ADM, symbol MTJ-889X1:MTJ-889X1
Connections:
- net Pin 1: now also J1.1, J1.2, J2.1
- net Pin 2: now also J1.3, J1.4, J2.2
- net Pin 3: now also J1.5, J1.6, J2.3
- net Pin 4: now also J1.7, J1.8, J2.4
- net Pin 5: now also J1.10, J1.9, J2.5
- net Pin 6: now also J1.11, J1.12, J2.6
- net Pin 7: now also J1.13, J1.14, J2.7
- net Pin 8: now also J1.15, J1.16, J2.8

Commit message: Ahhhhh
Changed lines of the file:
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@@
+    )
+  )
+  (symbol (lib_id "LOGO:LOGO") (at 161.29 43.18 0) (unit 1)
+    (in_bom yes) (on_board yes) (dnp no) (fields_autoplaced)
+    (property "Reference" "#G1" (at 161.29 42.7597 0)
+      (effects (font (size 1.27 1.27)) hide)
+    )
+    (property "Value" "LOGO" (at 161.29 43.6003 0)
+      (effects (font (size 1.27 1.27)) hide)
+    )
+    (property "Footprint" "LOGO:RP_Logo" (at 161.29 43.18 0)
+      (effects (font (size 1.27 1.27)) hide)
+    )
+    (property "Datasheet" "" (at 161.29 43.18 0)
+      (effects (font (size 1.27 1.27)) hide)
+    )
+    (instances
+      (project "EthBreakoutBoard"
+        (path "/5faa7872-a78c-419d-982c-2091ae072687"
+          (reference "#G1") (unit 1)
+        )
+      )
     )
   )
