File: PT Board Ground Systems V1.2/PT Board Ground Systems V1.2.kicad_pcb (KiCad board)
At the start: 2 copper layers, 82.6 x 25.4 mm, 11 parts, among them J1 TBLH10V-350-02BK, J2 TBLH10V-350-08BK, J3 TBLH10V-350-08BK, J4 TBLH10V-350-08BK, J5 TBLH10V-350-08BK

Commit message: A
Other:
- board text added: "Aarhus Wuz Here"
Changed lines of the file:
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@@
     (fp_line (start 26.6 1.4) (end -2.1 1.4)
       (stroke (width 0.1) (type solid)) (layer "F.Fab"))
-    (pad "1" thru_hole oval (at 0 0 180) (size 2.025 2.025) (drill 1.35) (layers "*.Cu" "*.Mask")
+    (pad "1" thru_hole circle (at 0 0 180) (size 2.025 2.025) (drill 1.35) (layers "*.Cu" "*.Mask")
       (net 2 "GND") (pinfunction "1") (pintype "passive"))
     (pad "2" thru_hole circle (at 0 -5.5 180) (size 2.025 2.025) (drill 1.35) (layers "*.Cu" "*.Mask")
@@
   (gr_rect (start 25.4 25.4) (end 107.95 50.8)
     (stroke (width 0.1) (type solid)) (fill none) (layer "Edge.Cuts"))
+  (gr_text "Aarhus Wuz Here" (at 75.692 38.862) (layer "B.SilkS")
+    (effects (font (size 1.5 1.5) (thickness 0.3) bold) (justify left bottom mirror))
+  )
   (gr_text "PWR" (at 60.017713 50.038) (layer "F.SilkS")
     (effects (font (size 1.5 1.5) (thickness 0.3) bold) (justify left bottom))
@@
     (polygon
       (pts
-        (xy 26.67 38.1)
-        (xy 96.012 38.1)
-        (xy 96.012 40.894)
-        (xy 97.79 42.672)
-        (xy 100.838 42.672)
+        (xy 26.162 37.592)
+        (xy 96.012 37.592)
+        (xy 96.012 39.624)
+        (xy 97.79 41.402)
+        (xy 100.838 41.402)
         (xy 100.838 44.45)
-        (xy 97.028 47.752)
-        (xy 36.83 47.498)
+        (xy 97.028 48.26)
+        (xy 36.83 48.006)
         (xy 36.83 45.212)
         (xy 33.02 41.656)
-        (xy 26.67 41.656)
+        (xy 26.162 41.656)
       )
     )
@@
     (connect_pads (clearance 0.508))
     (min_thickness 0.254) (filled_areas_thickness no)
-    (fill yes (thermal_gap 0.508) (thermal_bridge_width 0.508))
+    (fill yes (thermal_gap 0.508) (thermal_bridge_width 0.635))
     (polygon
       (pts

Commit message: Boards
Parts:
- added J6: TBLH10V-350-02BK, TBLH10V-350-02BK:RHDR4W80P550X350_2X2_770X850X1420P, F.Cu at (109.5, 39.6)
- moved J4 0.27 mm to (63.1, 40.5)
- moved J5 0.27 mm to (93.0, 40.5)
- moved J2 0.27 mm to (93.0, 29.8)
- moved J3 0.27 mm to (63.1, 29.9)
- moved D1 0.27 mm to (99.0, 32.8)
- moved R1 0.27 mm to (99.0, 38.4)
Other:
- board size 82.6 x 25.4 mm -> 86.4 x 25.4 mm
- board text removed: "IN"
Changed lines of the file:
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@@
   (net 3 "POWER IN")
   (footprint "TBLH10V-350-08BK:RHDR16W80P550X350_2X8_2870X850X1420P" (layer "F.Cu")
-    (at 63.388 29.84 180)
+    (at 63.12 29.85 180)
     (descr "TBLH10V-350-08BK height 14.2")
     (tags "Connector")
@@
   )
   (footprint "TBLH10V-350-08BK:RHDR16W80P550X350_2X8_2870X850X1420P" (layer "F.Cu")
-    (at 93.278 29.83 180)
+    (at 93.01 29.84 180)
     (descr "TBLH10V-350-08BK height 14.2")
     (tags "Connector")
@@
   )
   (footprint "TBLH10V-350-08BK:RHDR16W80P550X350_2X8_2870X850X1420P" (layer "F.Cu")
-    (at 93.278 40.474 180)
+    (at 93.01 40.484 180)
     (descr "TBLH10V-350-08BK height 14.2")
     (tags "Connector")
@@
     )
   )
+  (footprint "TBLH10V-350-02BK:RHDR4W80P550X350_2X2_770X850X1420P" (layer "F.Cu")
+    (at 109.492 39.606 90)
+    (descr "TBLH10V-350-02BK")
+    (tags "Connector")
+    (property "Height" "14.2")
+    (property "Manufacturer_Name" "CUI Devices")
+    (property "Manufacturer_Part_Number" "TBLH10V-350-02BK")
+    (property "Mouser Part Number" "490-TBLH10V-350-02BK")
+    (property "Mouser Price/Stock" "https://www.mouser.co.uk/ProductDetail/CUI-Devices/TBLH10V-350-02BK?qs=UXgszm6BlbHhb3E%252BatV8QQ%3D%3D")
+    (property "Sheetfile" "PT Board Ground Systems V1.2.kicad_sch")
+    (property "Sheetname" "")
+    (property "ki_description" "Conn Terminal Block 2 POS 3.5mm Solder ST Thru-Hole 10A/Contact")
+    (attr through_hole)
+    (fp_text reference "J6" (at 0 0 90) (layer "F.SilkS")
+        (effects (font (size 1.27 1.27) (thickness 0.254)))
+    )
+    (fp_text value "TBLH10V-350-02BK" (at 0 0 90) (layer "F.SilkS") hide
+        (effects (font (size 1.27 1.27) (thickness 0.254)))
+    )
+    (fp_text user "${REFERENCE}" (at 0 0 90) (layer "F.Fab")
+        (effects (font (size 1.27 1.27) (thickness 0.254)))
+    )
+    (fp_line (start -2.1 -7.1) (end -2.1 0)
+      (stroke (width 0.2) (type solid)) (layer "F.SilkS"))
+    (fp_line (start 0 1.4) (end 5.6 1.4)
+      (stroke (width 0.2) (type solid)) (layer "F.SilkS"))
+    (fp_line (start 5.6 -7.1) (end -2.1 -7.1)
+      (stroke (width 0.2) (type solid)) (layer "F.SilkS"))
+    (fp_line (start 5.6 1.4) (end 5.6 -7.1)
+      (stroke (width 0.2) (type solid)) (layer "F.SilkS"))
+    (fp_line (start -2.35 -7.35) (end 5.85 -7.35)
+      (stroke (width 0.05) (type solid)) (layer "F.CrtYd"))
+    (fp_line (start -2.35 1.65) (end -2.35 -7.35)
+      (stroke (width 0.05) (type solid)) (layer "F.CrtYd"))
+    (fp_line (start 5.85 -7.35) (end 5.85 1.65)
+      (stroke (width 0.05) (type solid)) (layer "F.CrtYd"))
+    (fp_line (start 5.85 1.65) (end -2.35 1.65)
+      (stroke (width 0.05) (type solid)) (layer "F.CrtYd"))
+    (fp_line (start -2.1 -7.1) (end 5.6 -7.1)
+      (stroke (width 0.1) (type solid)) (layer "F.Fab"))
+    (fp_line (start -2.1 1.4) (end -2.1 -7.1)
+      (stroke (width 0.1) (type solid)) (layer "F.Fab"))
+    (fp_line (start 5.6 -7.1) (end 5.6 1.4)
+      (stroke (width 0.1) (type solid)) (layer "F.Fab"))
+    (fp_line (start 5.6 1.4) (end -2.1 1.4)
+      (stroke (width 0.1) (type solid)) (layer "F.Fab"))
+    (pad "1" thru_hole circle (at 0 0 90) (size 2.025 2.025) (drill 1.35) (layers "*.Cu" "*.Mask")
+      (net 3 "POWER IN") (pinfunction "1") (pintype "passive"))
+    (pad "2" thru_hole circle (at 0 -5.5 90) (size 2.025 2.025) (drill 1.35) (layers "*.Cu" "*.Mask")
+      (net 3 "POWER IN") (pinfunction "2") (pintype "passive"))
+    (pad "3" thru_hole rect (at 3.5 0 90) (size 2.025 2.025) (drill 1.35) (layers "*.Cu" "*.Mask")
+      (net 2 "GND") (pinfunction "3") (pintype "passive"))
+    (pad "4" thru_hole rect (at 3.5 -5.5 90) (size 2.025 2.025) (drill 1.35) (layers "*.Cu" "*.Mask")
+      (net 2 "GND") (pinfunction "4") (pintype "passive"))
+    (model "TBLH10V-350-02BK.stp"
+      (offset (xyz 0 0 0))
+      (scale (xyz 1 1 1))
+      (rotate (xyz 0 0 0))
+    )
+  )
   (footprint "Resistor_THT:R_Axial_DIN0204_L3.6mm_D1.6mm_P5.08mm_Horizontal" (layer "F.Cu")
-    (at 99.314 38.354 -90)
+    (at 99.046 38.364 -90)
     (descr "Resistor, Axial_DIN0204 series, Axial, Horizontal, pin pitch=5.08mm, 0.167W, length*diameter=3.6*1.6mm^2, http://cdn-reichelt.de/documents/datenblatt/B400/1_4W%23YAG.pdf")
     (tags "Resistor Axial_DIN0204 series Axial Horizontal pin pitch 5.08mm 0.167W length 3.6mm diameter 1.6mm")
@@
     (property "ki_keywords" "R resistor")
     (attr through_hole)
-    (fp_text reference "R1" (at 2.54 -2.032 90) (layer "F.SilkS")
+    (fp_text reference "R1" (at 2.576 -0.086 90) (layer "F.SilkS")
         (effects (font (size 1 1) (thickness 0.15)))
     )
@@
   )
   (footprint "LED_THT:LED_D3.0mm" (layer "F.Cu")
-    (at 99.314 32.761 -90)
+    (at 99.046 32.771 -90)
     (descr "LED, diameter 3.0mm, 2 pins")
     (tags "LED diameter 3.0mm 2 pins")
@@
     (property "ki_keywords" "LED diode")
     (attr through_hole)
-    (fp_text reference "D1" (at 1.275 -3.302 90) (layer "F.SilkS")
+    (fp_text reference "D1" (at -2.411 -0.056 90) (layer "F.SilkS")
         (effects (font (size 1 1) (thickness 0.15)))
     )
@@
   )
   (footprint "TBLH10V-350-08BK:RHDR16W80P550X350_2X8_2870X850X1420P" (layer "F.Cu")
-    (at 63.388 40.474 180)
+    (at 63.12 40.484 180)
     (descr "TBLH10V-350-08BK height 14.2")
     (tags "Connector")
@@
       (net 2 "GND") (pinfunction "1") (pintype "input"))
   )
-  (gr_rect (start 25.4 25.4) (end 107.95 50.8)
+  (gr_rect (start 25.4 25.4) (end 111.76 50.8)
     (stroke (width 0.1) (type solid)) (fill none) (layer "Edge.Cuts"))
   (gr_text "Aarhus Wuz Here" (at 75.692 38.862) (layer "B.SilkS")
@@
     (effects (font (size 1.5 1.5) (thickness 0.3) bold) (justify left bottom))
   )
-  (gr_text "PWR" (at 55.536 56.134) (layer "F.SilkS")
-    (effects (font (size 2 2) (thickness 0.25)))
-  )
-  (gr_text "IN" (at 76.794 56.134) (layer "F.SilkS")
-    (effects (font (size 3 3) (thickness 0.3)))
-  )
   (gr_text "GND" (at 32.766 25.146 270) (layer "F.SilkS")
     (effects (font (size 2.5 2.5) (thickness 0.3) bold) (justify left bottom))
   )
-  (gr_text "GND" (at 70.104 56.134) (layer "F.SilkS")
-    (effects (font (size 2 2) (thickness 0.25)))
+  (gr_text "GND" (at 110.892 34.006 90) (layer "F.SilkS")
+    (effects (font (size 2.5 2.5) (thickness 0.3) bold) (justify left bottom))
   )
   (gr_text "GND" (at 67.672856 27.94) (layer "F.SilkS")
@@
     (effects (font (size 1.5 1.5) (thickness 0.3) bold) (justify left bottom))
   )
-  (gr_text "IN" (at 49.276 56.134) (layer "F.SilkS")
-    (effects (font (size 3 3) (thickness 0.3)))
-  )
   (gr_text "GND" (at 75.25657 27.94) (layer "F.SilkS")
     (effects (font (size 1.5 1.5) (thickness 0.3) bold) (justify left bottom))
+  )
+  (gr_text "PWR" (at 110.91 41.73 90) (layer "F.SilkS")
+    (effects (font (size 2.5 2.5) (thickness 0.3) bold) (justify right bottom))
   )
   (segment (start 99.314 38.354) (end 99.314 35.301) (width 0.5) (layer "F.Cu") (net 1))
@@
     (polygon
       (pts
-        (xy 26.162 37.592)
-        (xy 96.012 37.592)
-        (xy 96.012 39.624)
-        (xy 97.79 41.402)
-        (xy 100.838 41.402)
-        (xy 100.838 44.45)
+        (xy 26.122 37.832)
+        (xy 111.23 37.73)
+        (xy 111.36 41.62)
+        (xy 103 41.64)
+        (xy 97.04 46.99)
         (xy 97.028 48.26)
         (xy 36.83 48.006)
-        (xy 36.83 45.212)
-        (xy 33.02 41.656)
+        (xy 36.9 45.202)
+        (xy 33.09 41.646)
         (xy 26.162 41.656)
       )
@@
     (polygon
       (pts
-        (xy 112.776 57.404)
+        (xy 116.866 58.654)
         (xy 19.558 57.912)
         (xy 18.034 19.05)
-        (xy 111.296598 18.49914)
+        (xy 115.386598 19.74914)
       )
     )
