File: AnalogBox/AnalogBox/AnalogBox/AnalogBox.kicad_sch (KiCad schematic)
At the start: 12 parts, among them J1 MTJ-889X1, J11 TBLH10V-350-08BK, J2 TBLH10V-350-08BK, J3 TBLH10V-350-08BK, J4 TBLH10V-350-02BK, J5 MTJ-889X1, J6 TBLH10V-350-08BK, J8 MTJ-889X1

Commit message: Piss bot
Parts:
- added D1: LED, LED_THT:LED_D3.0mm, symbol Device:LED
- added R1: R, Resistor_THT:R_Axial_DIN0207_L6.3mm_D2.5mm_P7.62mm_Horizontal, symbol Device:R
- J11, J2, J3, J6: footprint RHDR16W80P550X350_2X8_2870X850X1420P -> TBLH10V-350-08BK:RHDR16W80P550X350_2X8_2870X850X1420P
- J4: footprint RHDR4W80P550X350_2X2_770X850X1420P -> TBLH10V-350-02BK:RHDR4W80P550X350_2X2_770X850X1420P
Connections:
- net Abort In: now also R1.1
- net GND: now also D1.1 (K)
- new net: D1.2 (A), R1.2
Changed lines of the file:
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@@
+    (stroke (width 0) (type default))
+  )
+  (wire (pts (xy 52.705 113.03) (xy 52.705 114.3))
     (stroke (width 0) (type default))
   )
@@
     (stroke (width 0) (type default))
   )
+  (wire (pts (xy 32.385 113.03) (xy 34.29 113.03))
+    (stroke (width 0) (type default))
+  )
   (wire (pts (xy 179.705 55.88) (xy 182.245 55.88))
     (stroke (width 0) (type default))
@@
     (stroke (width 0) (type default))
   )
+  (wire (pts (xy 51.435 113.03) (xy 52.705 113.03))
+    (stroke (width 0) (type default))
+  )
   (wire (pts (xy 179.705 24.13) (xy 182.245 24.13))
     (stroke (width 0) (type default))
@@
     (stroke (width 0) (type default))
   )
+  (wire (pts (xy 43.815 113.03) (xy 41.91 113.03))
+    (stroke (width 0) (type default))
+  )
   (wire (pts (xy 36.195 67.31) (xy 36.195 69.85))
     (stroke (width 0) (type default))
@@
     )
   )
+  (global_label "Abort In" (shape input) (at 32.385 113.03 180) (fields_autoplaced)
+    (effects (font (size 1.27 1.27)) (justify right))
+    (property "Intersheetrefs" "${INTERSHEET_REFS}" (at 21.7799 113.03 0)
+      (effects (font (size 1.27 1.27)) (justify right) hide)
+    )
+  )
   (global_label "Switch7" (shape input) (at 123.825 38.1 0) (fields_autoplaced)
     (effects (font (size 1.27 1.27)) (justify left))
@@
       (effects (font (size 1.27 1.27)))
     )
-    (property "Footprint" "RHDR16W80P550X350_2X8_2870X850X1420P" (at 117.475 117.78 0)
+    (property "Footprint" "TBLH10V-350-08BK:RHDR16W80P550X350_2X8_2870X850X1420P" (at 117.475 117.78 0)
       (effects (font (size 1.27 1.27)) (justify left top) hide)
     )
@@
       (effects (font (size 1.27 1.27)))
     )
-    (property "Footprint" "RHDR16W80P550X350_2X8_2870X850X1420P" (at 57.15 118.415 0)
+    (property "Footprint" "TBLH10V-350-08BK:RHDR16W80P550X350_2X8_2870X850X1420P" (at 57.15 118.415 0)
       (effects (font (size 1.27 1.27)) (justify left top) hide)
     )
@@
     )
   )
+  (symbol (lib_id "Device:R") (at 38.1 113.03 90) (unit 1)
+    (in_bom yes) (on_board yes) (dnp no) (fields_autoplaced)
+    (property "Reference" "R1" (at 38.1 106.68 90)
+      (effects (font (size 1.27 1.27)))
+    )
+    (property "Value" "R" (at 38.1 109.22 90)
+      (effects (font (size 1.27 1.27)))
+    )
+    (property "Footprint" "Resistor_THT:R_Axial_DIN0207_L6.3mm_D2.5mm_P7.62mm_Horizontal" (at 38.1 114.808 90)
+      (effects (font (size 1.27 1.27)) hide)
+    )
+    (property "Datasheet" "~" (at 38.1 113.03 0)
+      (effects (font (size 1.27 1.27)) hide)
+    )
+    (pin "1")
+    (pin "2")
+    (instances
+      (project "AnalogBox"
+        (path "/f8e0a2f8-bdad-44b3-86dd-b2cc512c9ab6"
+          (reference "R1") (unit 1)
+        )
+      )
+    )
+  )
   (symbol (lib_id "power:GND") (at 18.415 189.23 0) (unit 1)
     (in_bom yes) (on_board yes) (dnp no) (fields_autoplaced)
@@
         (path "/f8e0a2f8-bdad-44b3-86dd-b2cc512c9ab6"
           (reference "H1") (unit 1)
+        )
+      )
+    )
+  )
+  (symbol (lib_id "power:GND") (at 52.705 114.3 0) (unit 1)
+    (in_bom yes) (on_board yes) (dnp no) (fields_autoplaced)
+    (property "Reference" "#PWR016" (at 52.705 120.65 0)
+      (effects (font (size 1.27 1.27)) hide)
+    )
+    (property "Value" "GND" (at 52.705 119.38 0)
+      (effects (font (size 1.27 1.27)))
+    )
+    (property "Footprint" "" (at 52.705 114.3 0)
+      (effects (font (size 1.27 1.27)) hide)
+    )
+    (property "Datasheet" "" (at 52.705 114.3 0)
+      (effects (font (size 1.27 1.27)) hide)
+    )
+    (pin "1")
+    (instances
+      (project "AnalogBox"
+        (path "/f8e0a2f8-bdad-44b3-86dd-b2cc512c9ab6"
+          (reference "#PWR016") (unit 1)
         )
       )
@@
       (effects (font (size 1.27 1.27)))
     )
-    (property "Footprint" "RHDR4W80P550X350_2X2_770X850X1420P" (at 55.245 185.09 0)
+    (property "Footprint" "TBLH10V-350-02BK:RHDR4W80P550X350_2X2_770X850X1420P" (at 55.245 185.09 0)
       (effects (font (size 1.27 1.27)) (justify left top) hide)
     )
@@
     )
   )
+  (symbol (lib_id "Device:LED") (at 47.625 113.03 180) (unit 1)
+    (in_bom yes) (on_board yes) (dnp no) (fields_autoplaced)
+    (property "Reference" "D1" (at 49.2125 105.41 0)
+      (effects (font (size 1.27 1.27)))
+    )
+    (property "Value" "LED" (at 49.2125 107.95 0)
+      (effects (font (size 1.27 1.27)))
+    )
+    (property "Footprint" "LED_THT:LED_D3.0mm" (at 47.625 113.03 0)
+      (effects (font (size 1.27 1.27)) hide)
+    )
+    (property "Datasheet" "~" (at 47.625 113.03 0)
+      (effects (font (size 1.27 1.27)) hide)
+    )
+    (pin "1")
+    (pin "2")
+    (instances
+      (project "AnalogBox"
+        (path "/f8e0a2f8-bdad-44b3-86dd-b2cc512c9ab6"
+          (reference "D1") (unit 1)
+        )
+      )
+    )
+  )
   (symbol (lib_id "power:GND") (at 178.435 38.1 0) (unit 1)
     (in_bom yes) (on_board yes) (dnp no) (fields_autoplaced)
@@
       (effects (font (size 1.27 1.27)))
     )
-    (property "Footprint" "RHDR16W80P550X350_2X8_2870X850X1420P" (at 117.475 153.34 0)
+    (property "Footprint" "TBLH10V-350-08BK:RHDR16W80P550X350_2X8_2870X850X1420P" (at 117.475 153.34 0)
       (effects (font (size 1.27 1.27)) (justify left top) hide)
     )
@@
       (effects (font (size 1.27 1.27)))
     )
-    (property "Footprint" "RHDR16W80P550X350_2X8_2870X850X1420P" (at 57.15 149.53 0)
-      (effects (font (size 1.27 1.27)) (justify left top) hide)
-    )
+    (property "Footprint" "TBLH10V-350-08BK:RHDR16W80P550X350_2X8_2870X850X1420P" (at 57.15 149.53 0)
+      (effects (font (size 1.27 1.27)) (justify left top) hide)
+    )
