File: Personal OBC V2.0/Personal OBC V2.0.kicad_pcb (KiCad board)
At the start: 2 copper layers, 7.5 x 2 mm, 44 parts, among them J1 Screw_Terminal_01x02, J2 Screw_Terminal_01x04, J3 USB_B_Mini, J4 SWD Pins, Q1 SI7232DN-T1-GE3, U1 STM32F042G6Ux, U2 MS560702BA03-50, U3 AP2210N-3.3TRG1, U4 W25X40CLUXIG_TR, U5 LM293QT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

Commit message: Bruhg
Parts:
- added H1: MountingHole_Pad, MountingHole:MountingHole_3.2mm_M3_DIN965_Pad_TopOnly, F.Cu at (83.7, 22.2)
- added H2: MountingHole_Pad, MountingHole:MountingHole_3.2mm_M3_DIN965_Pad_TopOnly, F.Cu at (83.7, 29.3)
- moved BZ1 106.6 mm to (31.8, 48.9), turned to -90 degrees
- moved J4 91.4 mm to (27.0, 35.7)
- moved BT1 81.1 mm to (31.8, 32.3), turned to 0 degrees
- moved J1 69.5 mm to (34.1, 36.4), turned to -90 degrees
- moved J3 53.0 mm to (32.1, 74.4)
- moved J2 42.9 mm to (86.9, 42.9), turned to -90 degrees
- moved U1 8.87 mm to (57.7, 65.9)
- moved U2 5.08 mm to (43.0, 60.7)
- moved Q1 0.13 mm to (44.5, 49.0)
Other:
- board size 7.5 x 2 mm -> 12.7 x 50.8 mm

Commit message: AAAAAAAAA
Parts:
- moved J2 50.3 mm to (36.7, 39.8)
- moved U3 44.9 mm to (27.4, 39.6)
- moved U2 35.7 mm to (66.7, 34.0), turned to 180 degrees
- moved L1 35.4 mm to (93.7, 17.9), turned to -90 degrees
- moved D1 33.7 mm to (26.5, 34.5), turned to -90 degrees
- moved U1 28.8 mm to (60.6, 37.2), turned to -45 degrees
- moved PS1 27.7 mm to (90.1, 18.1)
- moved U4 19.1 mm to (55.5, 41.1), turned to -45 degrees
- moved Y1 16.8 mm to (59.6, 31.1), turned to 180 degrees
- moved J4 12.7 mm to (36.7, 27.5)
- moved J1 11.2 mm to (26.6, 28.1)
- moved C12 6.32 mm to (58.1, 34.1), turned to 135 degrees
- moved BZ1 5.96 mm to (26.5, 46.2)
Routing:
- added copper zone on In1.Cu, net +3.3V
- added copper zone on In2.Cu, net GND
Other:
- copper layers 2 -> 4

Commit message: Personal OBC Layout
Parts:
- removed PS1: MCP1642B-50I_MC, MCP1642B-50I_MC:SON50P300X200X100-9N-D
- added U6: MCP1642B-50I/MS, MCP1642B_50I_MS:MSOP8_MCP1642B-50I&slash_MS_MCH-L, B.Cu at (38.8, 36.1)
- BTr: renamed from BT1; footprint Connector_JST:JST_PH_S2B-PH-K_1x02_P2.00mm_Horizontal -> Connector_JST:JST_PH_B2B-PH-K_1x02_P2.00mm_Vertical
- C13, C14: footprint Capacitor_SMD:C_0603_1608Metric -> Capacitor_SMD:C_0603_1608Metric_Pad1.08x0.95mm_HandSolder; moved to B.Cu
- C6, C7: footprint Capacitor_SMD:C_0402_1005Metric -> Capacitor_SMD:C_0402_1005Metric_Pad0.74x0.62mm_HandSolder; moved to B.Cu
- D1, U3: moved to B.Cu
- J1: footprint TerminalBlock_TE-Connectivity:TerminalBlock_TE_282834-2_1x02_P2.54mm_Horizontal -> Conn_Screw_SMD:2_Pin_Conn
- J2: value Screw_Terminal_01x04 -> Screw_Terminal_01x08; footprint TerminalBlock_TE-Connectivity:TerminalBlock_TE_282834-8_1x08_P2.54mm_Horizontal -> Conn_Screw_SMD:8_Pin_Conn
- J4: footprint Connector_PinHeader_2.54mm:PinHeader_1x04_P2.54mm_Vertical -> Conn_Screw_SMD:4_Pin_Conn
- L1: footprint Inductor_SMD:L_1008_2520Metric -> Inductor_SMD:L_1008_2520Metric_Pad1.43x2.20mm_HandSolder; moved to B.Cu
- moved L1 62.2 mm to (34.4, 36.8)
- moved H1 56.8 mm to (29.2, 38.1)
- moved H2 50.9 mm to (41.9, 58.4)
- moved C13 42.3 mm to (36.9, 33.6)
- moved U2 38.8 mm to (32.2, 51.8), turned to 0 degrees
- moved C14 38.4 mm to (39.9, 38.6), turned to 180 degrees
- moved C6 37.5 mm to (27.7, 33.2), turned to 90 degrees
- moved U5 36.6 mm to (37.1, 31.4)
- moved C5 33.3 mm to (32.2, 48.4)
- moved C7 31.9 mm to (33.1, 33.3), turned to 90 degrees
- moved C11 30.0 mm to (41.5, 49.8), turned to 180 degrees
- moved C12 28.3 mm to (32.4, 45.7), turned to 0 degrees
- moved J3 25.4 mm to (44.3, 52.1), turned to -90 degrees
- moved R3 25.3 mm to (32.0, 33.1)
- moved U1 25.0 mm to (36.1, 42.8), turned to 90 degrees
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Connections:
- L1 pad 2: Net-(PS1-SW) -> /Pin_8_L1
- U1 pad 14: PT_0_IN -> PT_1_IN
- U1 pad 15: PT_1_IN -> PT_0_IN
Routing:
- net V_LIPO: track 0.00 -> 32.3 mm
- net PWR: track 0.00 -> 7.73 mm
- net GND: track 0.00 -> 4.16 mm, vias 0 -> 9
- net +3.3V: track 0.00 -> 1.44 mm, vias 0 -> 3
- added copper zone on B.Cu, net +3.3V
- added copper zone on B.Cu, net +5V
- added copper zone on B.Cu, net /Pin_8_L1
- added copper zone on B.Cu, net /V_LDO_IN
- added copper zone on B.Cu, net GND
- added copper zone on B.Cu, net V_LIPO
Other:
- board size 12.7 x 50.8 mm -> 20.3 x 38.1 mm
- board text added: "+"
- board text added: "-"

Commit message: AAAAaaaa
Parts:
- moved R3 1.54 mm to (30.6, 33.8), turned to -90 degrees
Changed lines of the file:
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@@
   )
   (footprint "Resistor_SMD:R_0402_1005Metric" (layer "F.Cu")
-    (at 31.98 33.15)
+    (at 30.57 33.76 -90)
     (descr "Resistor SMD 0402 (1005 Metric), square (rectangular) end terminal, IPC_7351 nominal, (Body size source: IPC-SM-782 page 72, https://www.pcb-3d.com/wordpress/wp-content/uploads/ipc-sm-782a_amendment_1_and_2.pdf), generated with kicad-footprint-generator")
     (tags "resistor")
@@
     (property "ki_keywords" "R res resistor")
     (attr smd)
-    (fp_text reference "R3" (at 0 -1.17) (layer "F.SilkS")
+    (fp_text reference "R3" (at 0 -1.17 90) (layer "F.SilkS")
         (effects (font (size 1 1) (thickness 0.15)))
     )
-    (fp_text value "10k" (at 0 1.17) (layer "F.Fab")
+    (fp_text value "10k" (at 0 1.17 90) (layer "F.Fab")
         (effects (font (size 1 1) (thickness 0.15)))
     )
-    (fp_text user "${REFERENCE}" (at 0 0) (layer "F.Fab")
+    (fp_text user "${REFERENCE}" (at 0 0 90) (layer "F.Fab")
         (effects (font (size 0.26 0.26) (thickness 0.04)))
     )
@@
     (fp_line (start 0.525 0.27) (end -0.525 0.27)
       (stroke (width 0.1) (type solid)) (layer "F.Fab"))
-    (pad "1" smd roundrect (at -0.51 0) (size 0.54 0.64) (layers "F.Cu" "F.Paste" "F.Mask") (roundrect_rratio 0.25)
+    (pad "1" smd roundrect (at -0.51 0 270) (size 0.54 0.64) (layers "F.Cu" "F.Paste" "F.Mask") (roundrect_rratio 0.25)
       (net 5 "/V_LDO_IN") (pintype "passive"))
-    (pad "2" smd roundrect (at 0.51 0) (size 0.54 0.64) (layers "F.Cu" "F.Paste" "F.Mask") (roundrect_rratio 0.25)
+    (pad "2" smd roundrect (at 0.51 0 270) (size 0.54 0.64) (layers "F.Cu" "F.Paste" "F.Mask") (roundrect_rratio 0.25)
       (net 30 "CMP_LDO_IN_A") (pintype "passive"))
     (model "${KICAD6_3DMODEL_DIR}/Resistor_SMD.3dshapes/R_0402_1005Metric.wrl"
