File: ACS Arduino Board/ACS Arduino Board.kicad_pcb (KiCad board)
At the start: 2 copper layers, 16 parts, among them J1 TBLH10V-350-08BK, J2 TBLH10V-350-02BK, J3 TBLH10V-350-08BK, J4 TBLH10V-350-02BK, J5 MTJ-889X1

Commit message: Piss
Parts:
- removed R1: R, Resistor_THT:R_Axial_DIN0204_L3.6mm_D1.6mm_P5.08mm_Horizontal
- added D1: D, Diode_THT:D_A-405_P7.62mm_Horizontal, F.Cu at (101.3, 79.8)
- added J6: TBLH10V-350-08BK, TBLH10V-350-08BK:RHDR16W80P550X350_2X8_2870X850X1420P, F.Cu at (82.3, 38.8)
- added J7: TBLH10V-350-02BK, TBLH10V-350-02BK:RHDR4W80P550X350_2X2_770X850X1420P, F.Cu at (69.1, 80.7)
- added K1: CPC1706Y, RelayCPC:CPC1706Y, F.Cu at (46.1, 66.8)
- added K2: CPC1706Y, RelayCPC:CPC1706Y, F.Cu at (49.5, 67.5)
- added K3: CPC1706Y, RelayCPC:CPC1706Y, F.Cu at (81.4, 73.3)
- added K4: CPC1706Y, RelayCPC:CPC1706Y, F.Cu at (68.0, 64.2)
- added K5: CPC1706Y, RelayCPC:CPC1706Y, F.Cu at (68.0, 68.8)
- added R6: R, Resistor_THT:R_Axial_DIN0204_L3.6mm_D1.6mm_P5.08mm_Horizontal, F.Cu at (90.9, 79.8)
- added R7: R, Resistor_THT:R_Axial_DIN0204_L3.6mm_D1.6mm_P5.08mm_Horizontal, F.Cu at (83.6, 79.8)
- added R8: R, Resistor_THT:R_Axial_DIN0204_L3.6mm_D1.6mm_P5.08mm_Horizontal, F.Cu at (76.2, 79.8)
- added R9: R, Resistor_THT:R_Axial_DIN0204_L3.6mm_D1.6mm_P5.08mm_Horizontal, F.Cu at (63.0, 61.7)
- added RV1: R_Potentiometer, Connector_PinSocket_2.54mm:PinSocket_1x03_P2.54mm_Vertical, F.Cu at (117.3, 32.5)
- J3: value TBLH10V-350-08BK -> TBLH10V-350-02BK; footprint TBLH10V-350-08BK:RHDR16W80P550X350_2X8_2870X850X1420P -> TBLH10V-350-02BK:RHDR4W80P550X350_2X2_770X850X1420P
- moved J4 92.0 mm to (27.5, 74.4), turned to -90 degrees
- moved R2 85.3 mm to (38.2, 64.2)
- moved J2 80.7 mm to (38.3, 38.8)
- moved H1 79.3 mm to (31.8, 38.1)
- moved H4 78.9 mm to (32.0, 63.5)
- moved J1 59.3 mm to (49.5, 38.8)
- moved R4 39.2 mm to (93.7, 67.3), turned to 90 degrees
- moved R3 38.9 mm to (90.9, 67.3), turned to 90 degrees
- moved R5 36.4 mm to (104.6, 66.8), turned to 90 degrees
- moved J3 34.3 mm to (53.1, 75.0), turned to 180 degrees
- moved A2 19.4 mm to (77.8, 58.4), turned to 90 degrees
- moved J5 15.5 mm to (106.9, 75.2)
- moved H2 11.9 mm to (114.3, 38.1)
- moved H3 7.67 mm to (114.3, 63.5)
- moved A1 2.34 mm to (68.4, 43.2), turned to -90 degrees
Connections:
- net OxVent Out renamed Ox Vent Out
- A1 pad 27: Cycle Power -> Arduino Power
- A1 pad 29: GND -> Cycle GND
- A1 pad 4: GND -> Cycle GND
- A2 pad 29: GND -> Terminal GND
- A2 pad 4: GND -> Terminal GND
- H1 pad 1: GND -> unconnected-(H1-Pad1)
- H2 pad 1: GND -> unconnected-(H2-Pad1)
- H3 pad 1: GND -> unconnected-(H3-Pad1)
- H4 pad 1: GND -> unconnected-(H4-Pad1)
- J1 pad 10: Cycle Power -> Arduino Power
- J1 pad 11: Arm Key -> Cycle GND
- J1 pad 12: Arm Key -> Cycle GND
- J1 pad 13: Arm Key -> Cycle GND
- J1 pad 14: Arm Key -> Cycle GND
- J1 pad 15: Terminal Power -> 5V GND
- J1 pad 16: Terminal Power -> 5V GND
- J1 pad 7: Arduino Power -> Terminal Power
- J1 pad 8: Arduino Power -> Terminal Power
- J1 pad 9: Cycle Power -> Arduino Power
- J2 pad 1: GND -> 5V GND
- J2 pad 2: GND -> 5V GND
- J4 pad 1: GND -> 24V GND
- J4 pad 2: GND -> 24V GND
- J5 pad 1: unconnected-(J5-Pad1) -> Ignitor
- J5 pad 2: unconnected-(J5-Pad2) -> 24V GND
- J5 pad 5: unconnected-(J5-Pad5) -> Net-(D1-K)
Routing:
- net +5V: track 0.00 -> 149.3 mm
- net 5V GND: track 0.00 -> 145.3 mm
- net 24V GND: track 0.00 -> 95.3 mm
- net Cycle GND: track 0.00 -> 89.4 mm
- net +24V: track 0.00 -> 83.8 mm
- net Arduino Power: track 0.00 -> 82.1 mm
- net Terminal GND: track 0.00 -> 79.4 mm
- net Break Wire: track 0.00 -> 61.7 mm
- net Terminal Power: track 0.00 -> 32.8 mm
- net Net-(A1-D6): track 0.00 -> 22.7 mm
- net Net-(A1-D7): track 0.00 -> 22.0 mm
- net Main Fuel Out: track 0.00 -> 21.5 mm
- net Ignitor: track 0.00 -> 20.4 mm
- net Net-(A2-D3): track 0.00 -> 19.5 mm
- net LCD/SDA: track 0.00 -> 18.5 mm
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Other:
- board outline added: 95.2 x 58.4 mm
- board text added: "24V+"
- board text added: "5V+"
- board text added: "ARD |PWR|"
- board text added: "BURN TIME"
- board text added: "C. COM"
- board text added: "C. LED"
- board text added: "C. LED GND"
- board text added: "C. N_O"
- board text added: "F VENT"
- board text added: "GND"
- board text added: "LCD/SCL"
- board text added: "LCD/SDA"
- board text added: "MFV"
- board text added: "MOV"
- board text added: "O VENT"
- board text added: "T. COM"
- board text added: "T. LED"
- board text added: "T. LED GND"
- board text added: "T. N_O"
- board text added: "TERM |PWR|"

Commit message: EEEEE
Parts:
- D1: value D -> 1N5819
- R2, R3, R4, R5, R9: value R -> 2.2k; footprint Resistor_THT:R_Axial_DIN0204_L3.6mm_D1.6mm_P5.08mm_Horizontal -> Resistor_THT:R_Axial_DIN0207_L6.3mm_D2.5mm_P7.62mm_Horizontal
- R6: value R -> 470; footprint Resistor_THT:R_Axial_DIN0204_L3.6mm_D1.6mm_P5.08mm_Horizontal -> Resistor_THT:R_Axial_DIN0207_L6.3mm_D2.5mm_P7.62mm_Horizontal
- R7: value R -> 5.1k; footprint Resistor_THT:R_Axial_DIN0204_L3.6mm_D1.6mm_P5.08mm_Horizontal -> Resistor_THT:R_Axial_DIN0207_L6.3mm_D2.5mm_P7.62mm_Horizontal
- R8: value R -> 1M; footprint Resistor_THT:R_Axial_DIN0204_L3.6mm_D1.6mm_P5.08mm_Horizontal -> Resistor_THT:R_Axial_DIN0207_L6.3mm_D2.5mm_P7.62mm_Horizontal
- moved R6 12.7 mm to (103.6, 80.1)
- moved D1 8.07 mm to (93.3, 80.1)
- moved J7 4.33 mm to (64.8, 80.6)
- moved R7 3.26 mm to (84.1, 76.5), turned to 180 degrees
- moved R2 2.35 mm to (36.7, 62.4)
- moved R5 2.27 mm to (104.8, 69.1)
- moved R4 1.86 mm to (95.0, 68.7)
- moved R3 1.58 mm to (91.5, 68.8)
- moved J5 1.32 mm to (108.2, 75.2)
- moved R8 0.83 mm to (75.4, 80.1)
Connections:
- A1 pad 27: Arduino Power -> unconnected-(A1-+5V-Pad27)
- A1 pad 30: unconnected-(A1-VIN-Pad30) -> Arduino Power
- A2 pad 27: Terminal Power -> +5V
- A2 pad 30: unconnected-(A2-VIN-Pad30) -> Terminal Power
- D1 pad 2: Net-(D1-A) -> Break Wire
- J1 pad 1: +5V -> +9V
- J1 pad 15: 5V GND -> GND
- J1 pad 16: 5V GND -> GND
- J1 pad 2: +5V -> +9V
- J2 pad 1: 5V GND -> GND
- J2 pad 2: 5V GND -> GND
- J2 pad 3: +5V -> +9V
- J2 pad 4: +5V -> +9V
- J4 pad 1: 24V GND -> GND
- J4 pad 2: 24V GND -> GND
- J5 pad 2: 24V GND -> GND
- J5 pad 5: Net-(D1-K) -> Net-(J5-Pad5)
- J6 pad 7: 5V GND -> GND
- J6 pad 8: 5V GND -> GND
- R6 pad 1: Net-(D1-A) -> Net-(J5-Pad5)
- R6 pad 2: Break Wire -> Net-(D1-K)
- R8 pad 1: 5V GND -> GND
- RV1 pad 3: 5V GND -> Terminal GND
Routing:
- net GND: track 0.00 -> 272.2 mm
- net 5V GND: track 145.3 -> 0.00 mm
- net 24V GND: track 95.3 -> 0.00 mm
- net +5V: track 149.3 -> 79.5 mm
- net +9V: track 0.00 -> 18.7 mm
- net Terminal GND: track 79.4 -> 97.8 mm
- net Net-(J5-Pad5): track 0.00 -> 11.7 mm
- net Net-(D1-K): track 12.5 -> 2.68 mm
- net Terminal Power: track 32.8 -> 25.2 mm
- net Net-(K4-Pad2): track 8.04 -> 14.9 mm
- net Arduino Power: track 82.1 -> 85.3 mm
- net Net-(K5-Pad2): track 10.2 -> 13.1 mm
- net Net-(D1-A): track 2.79 -> 0.00 mm
- net Break Wire: track 61.7 -> 64.5 mm
- net Main Fuel Out: track 21.5 -> 24.0 mm
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Other:
- board text added: "VIN"

Commit message: Piss bot
Other:
- board text added: "Cycle"
- board text added: "Terminal"
Changed lines of the file:
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@@
       (plot_on_all_layers_selection 0x0000000_00000000)
       (disableapertmacros false)
-      (usegerberextensions false)
-      (usegerberattributes true)
-      (usegerberadvancedattributes true)
-      (creategerberjobfile true)
+      (usegerberextensions true)
+      (usegerberattributes false)
+      (usegerberadvancedattributes false)
+      (creategerberjobfile false)
       (dashed_line_dash_ratio 12.000000)
       (dashed_line_gap_ratio 3.000000)
@@
       (psa4output false)
       (plotreference true)
-      (plotvalue true)
+      (plotvalue false)
       (plotinvisibletext false)
       (sketchpadsonfab false)
-      (subtractmaskfromsilk false)
+      (subtractmaskfromsilk true)
       (outputformat 1)
       (mirror false)
-      (drillshape 1)
+      (drillshape 0)
       (scaleselection 1)
-      (outputdirectory "")
+      (outputdirectory "Gerbs/")
     )
   )
@@
     (effects (font (size 1 1) (thickness 0.15)) (justify left bottom))
   )
+  (gr_text "Cycle " (at 44.95 53.22) (layer "F.SilkS")
+    (effects (font (size 3 3) (thickness 0.5) bold) (justify left bottom))
+  )
   (gr_text "GND" (at 35.306 77.47) (layer "F.SilkS")
     (effects (font (size 2 2) (thickness 0.4) bold) (justify left bottom))
@@
     (effects (font (size 1.5 1.5) (thickness 0.25) bold) (justify left bottom))
   )
+  (gr_text "Terminal" (at 87.17 52.86) (layer "F.SilkS")
+    (effects (font (size 3 3) (thickness 0.5) bold) (justify left bottom))
+  )
   (gr_text "TERM\n|PWR|" (at 58.28 30.59) (layer "F.SilkS")

Commit message: ACS board changes
Parts:
- moved J4 1.07 mm to (28.6, 74.4)
Connections:
- J5 pad 2: GND -> Terminal GND
- R8 pad 1: GND -> Terminal GND
Routing:
- net GND: track 272.2 -> 137.7 mm
- net Terminal GND: track 97.8 -> 125.8 mm
- net +24V: track 83.1 -> 82.1 mm
Other:
- outline, holes or cut-outs redrawn
