File: LAF Board Proto V1.0/LAF Board Proto V1.0.kicad_pcb (KiCad board)
At the start: 4 copper layers, 57.1 x 50.8 mm, 95 parts, among them J1 PWR_IN, J2 USB_C_Receptacle_USB2.0, J3 RS485 Out, J4 PT_IN, J5 GPIO_OUT, J6 CAN_TERMINAL, Q1 MBT2222ADW1T1, SW1 RESET, SW2 SW_SPST, U1 ESP32-PICO-MINI-02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

Commit message: LAF board works
Parts:
- added G***: LOGO, LOGO, B.Cu at (46.3, 45.5)
- moved G*** 6.91 mm to (37.5, 54.7)
Other:
- board text added: "NAME:"
- board text added: "SERIAL:"

Commit message: ACS board changes
Parts:
- moved G*** 11.0 mm to (46.4, 48.2)
- moved G*** 10.0 mm to (40.5, 53.8)
Changed lines of the file:
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@@
       (plot_on_all_layers_selection 0x0000000_00000000)
       (disableapertmacros false)
-      (usegerberextensions false)
-      (usegerberattributes true)
-      (usegerberadvancedattributes true)
-      (creategerberjobfile true)
+      (usegerberextensions true)
+      (usegerberattributes false)
+      (usegerberadvancedattributes false)
+      (creategerberjobfile false)
       (dashed_line_dash_ratio 12.000000)
       (dashed_line_gap_ratio 3.000000)
@@
       (psa4output false)
       (plotreference true)
-      (plotvalue true)
+      (plotvalue false)
       (plotinvisibletext false)
       (sketchpadsonfab false)
-      (subtractmaskfromsilk false)
+      (subtractmaskfromsilk true)
       (outputformat 1)
       (mirror false)
-      (drillshape 1)
+      (drillshape 0)
       (scaleselection 1)
-      (outputdirectory "")
+      (outputdirectory "Gerbs/")
     )
   )
@@
     (fp_line (start 1.6 1.25) (end -1.6 1.25)
       (stroke (width 0.1) (type solid)) (layer "F.Fab"))
-    (pad "1" smd roundrect (at -1.475 0 270) (size 1.15 2.7) (layers "F.Cu" "F.Paste" "F.Mask") (roundrect_rratio 0.217391)
+    (pad "1" smd roundrect (at -1.475 0 270) (size 1.15 2.7) (layers "F.Cu" "F.Paste" "F.Mask") (roundrect_rratio 0.2173913043)
       (net 2 "GND") (pintype "passive"))
-    (pad "2" smd roundrect (at 1.475 0 270) (size 1.15 2.7) (layers "F.Cu" "F.Paste" "F.Mask") (roundrect_rratio 0.217391)
+    (pad "2" smd roundrect (at 1.475 0 270) (size 1.15 2.7) (layers "F.Cu" "F.Paste" "F.Mask") (roundrect_rratio 0.2173913043)
       (net 12 "Net-(U7-REFCAP)") (pintype "passive"))
     (model "${KICAD6_3DMODEL_DIR}/Capacitor_SMD.3dshapes/C_1210_3225Metric.wrl"
@@
     (fp_line (start 1 0.625) (end -1 0.625)
       (stroke (width 0.1) (type solid)) (layer "F.Fab"))
-    (pad "1" smd roundrect (at -0.9125 0 270) (size 1.025 1.4) (layers "F.Cu" "F.Paste" "F.Mask") (roundrect_rratio 0.243902)
+    (pad "1" smd roundrect (at -0.9125 0 270) (size 1.025 1.4) (layers "F.Cu" "F.Paste" "F.Mask") (roundrect_rratio 0.243902439)
       (net 41 "Net-(SW2-B)") (pintype "passive"))
-    (pad "2" smd roundrect (at 0.9125 0 270) (size 1.025 1.4) (layers "F.Cu" "F.Paste" "F.Mask") (roundrect_rratio 0.243902)
+    (pad "2" smd roundrect (at 0.9125 0 270) (size 1.025 1.4) (layers "F.Cu" "F.Paste" "F.Mask") (roundrect_rratio 0.243902439)
       (net 11 "Net-(C18-Pad2)") (pintype "passive"))
     (model "${KICAD6_3DMODEL_DIR}/Resistor_SMD.3dshapes/R_0805_2012Metric.wrl"
@@
     (fp_line (start 1 0.625) (end -1 0.625)
       (stroke (width 0.1) (type solid)) (layer "F.Fab"))
-    (pad "1" smd roundrect (at -0.9125 0 90) (size 1.025 1.4) (layers "F.Cu" "F.Paste" "F.Mask") (roundrect_rratio 0.243902)
+    (pad "1" smd roundrect (at -0.9125 0 90) (size 1.025 1.4) (layers "F.Cu" "F.Paste" "F.Mask") (roundrect_rratio 0.243902439)
       (net 26 "B") (pintype "passive"))
-    (pad "2" smd roundrect (at 0.9125 0 90) (size 1.025 1.4) (layers "F.Cu" "F.Paste" "F.Mask") (roundrect_rratio 0.243902)
+    (pad "2" smd roundrect (at 0.9125 0 90) (size 1.025 1.4) (layers "F.Cu" "F.Paste" "F.Mask") (roundrect_rratio 0.243902439)
       (net 27 "A") (pintype "passive"))
     (model "${KICAD6_3DMODEL_DIR}/Resistor_SMD.3dshapes/R_0805_2012Metric.wrl"
@@
     (fp_line (start 2 2) (end -2 2)
       (stroke (width 0.1) (type solid)) (layer "F.Fab"))
-    (pad "" smd roundrect (at -0.675 -0.675) (size 1.09 1.09) (layers "F.Paste") (roundrect_rratio 0.229358))
-    (pad "" smd roundrect (at -0.675 0.675) (size 1.09 1.09) (layers "F.Paste") (roundrect_rratio 0.229358))
-    (pad "" smd roundrect (at 0.675 -0.675) (size 1.09 1.09) (layers "F.Paste") (roundrect_rratio 0.229358))
-    (pad "" smd roundrect (at 0.675 0.675) (size 1.09 1.09) (layers "F.Paste") (roundrect_rratio 0.229358))
+    (pad "" smd roundrect (at -0.675 -0.675) (size 1.09 1.09) (layers "F.Paste") (roundrect_rratio 0.2293577982))
+    (pad "" smd roundrect (at -0.675 0.675) (size 1.09 1.09) (layers "F.Paste") (roundrect_rratio 0.2293577982))
+    (pad "" smd roundrect (at 0.675 -0.675) (size 1.09 1.09) (layers "F.Paste") (roundrect_rratio 0.2293577982))
+    (pad "" smd roundrect (at 0.675 0.675) (size 1.09 1.09) (layers "F.Paste") (roundrect_rratio 0.2293577982))
     (pad "1" smd roundrect (at -1.9625 -1.25) (size 0.825 0.25) (layers "F.Cu" "F.Paste" "F.Mask") (roundrect_rratio 0.25)
       (net 64 "unconnected-(U3-~{RI}{slash}CLK-Pad1)") (pinfunction "~{RI}/CLK") (pintype "bidirectional+no_connect"))
@@
     (fp_line (start 1 0.625) (end -1 0.625)
       (stroke (width 0.1) (type solid)) (layer "F.Fab"))
-    (pad "1" smd roundrect (at -0.9125 0 90) (size 1.025 1.4) (layers "F.Cu" "F.Paste" "F.Mask") (roundrect_rratio 0.243902)
+    (pad "1" smd roundrect (at -0.9125 0 90) (size 1.025 1.4) (layers "F.Cu" "F.Paste" "F.Mask") (roundrect_rratio 0.243902439)
       (net 11 "Net-(C18-Pad2)") (pintype "passive"))
-    (pad "2" smd roundrect (at 0.9125 0 90) (size 1.025 1.4) (layers "F.Cu" "F.Paste" "F.Mask") (roundrect_rratio 0.243902)
+    (pad "2" smd roundrect (at 0.9125 0 90) (size 1.025 1.4) (layers "F.Cu" "F.Paste" "F.Mask") (roundrect_rratio 0.243902439)
       (net 34 "CAN_L") (pintype "passive"))
     (model "${KICAD6_3DMODEL_DIR}/Resistor_SMD.3dshapes/R_0805_2012Metric.wrl"
@@
   )
   (footprint "LOGO" (layer "B.Cu")
-    (at 46.26 45.54 180)
+    (at 40.47 53.75 180)
     (attr board_only exclude_from_pos_files exclude_from_bom)
     (fp_text reference "G***" (at 0 0) (layer "B.SilkS") hide
@@
   )
   (footprint "LOGO:RP_Logo" (layer "B.Cu")
-    (at 37.5 54.71 180)
+    (at 46.39 48.17 180)
     (attr board_only exclude_from_pos_files exclude_from_bom)
     (fp_text reference "G***" (at 0 0) (layer "B.SilkS") hide
@@
         (effects (font (size 1 1) (thickness 0.15)) (justify mirror))
     )
-    (fp_line (start -1.8 -3.4) (end -1.3 -3.4)
-      (stroke (width 0.12) (type solid)) (layer "B.SilkS"))
-    (fp_line (start -1.8 -2.66) (end -1.8 -3.4)
-      (stroke (width 0.12) (type solid)) (layer "B.SilkS"))
     (fp_line (start -1.56 -3.16) (end 9.18 -3.16)
       (stroke (width 0.12) (type solid)) (layer "B.SilkS"))
@@
         (effects (font (size 1 1) (thickness 0.15)) (justify mirror))
     )
-    (fp_line (start -1.8 -3.4) (end -1.3 -3.4)
-      (stroke (width 0.12) (type solid)) (layer "B.SilkS"))
-    (fp_line (start -1.8 -2.66) (end -1.8 -3.4)
-      (stroke (width 0.12) (type solid)) (layer "B.SilkS"))
     (fp_line (start -1.56 -3.16) (end 6.64 -3.16)
       (stroke (width 0.12) (type solid)) (layer "B.SilkS"))
@@
         (effects (font (size 1 1) (thickness 0.15)) (justify mirror))
     )
-    (fp_line (start -1.8 -3.4) (end -1.3 -3.4)
-      (stroke (width 0.12) (type solid)) (layer "B.SilkS"))
-    (fp_line (start -1.8 -2.66) (end -1.8 -3.4)
-      (stroke (width 0.12) (type solid)) (layer "B.SilkS"))
     (fp_line (start -1.56 -3.16) (end 19.341 -3.16)
       (stroke (width 0.12) (type solid)) (layer "B.SilkS"))
@@
     (effects (font (size 2 2) (thickness 0.4) bold) (justify left bottom mirror))
   )
-  (gr_text "TXD1" (at 46.42 58.54) (layer "B.SilkS")
+  (gr_text "TXD1" (at 42.78 60.27) (layer "B.SilkS")
     (effects (font (size 1 1) (thickness 0.15)) (justify left bottom mirror))
   )
@@
     (effects (font (size 1 1) (thickness 0.15)) (justify left bottom mirror))
   )
-  (gr_text "CAN_RX" (at 56.81 54.9) (layer "B.SilkS")
+  (gr_text "CAN_RX" (at 60.32 54.69) (layer "B.SilkS")
     (effects (font (size 1 1) (thickness 0.15)) (justify left bottom mirror))
   )
@@
   (via (at 56.54 38.38) (size 1) (drill 0.5) (layers "F.Cu" "B.Cu") (net 2))
   (via (at 44.1 41.49) (size 0.7) (drill 0.3) (layers "F.Cu" "B.Cu") (net 2))
-  (via (at 44.11 48.16) (size 0.7) (drill 0.3) (layers "F.Cu" "B.Cu") (free) (net 2))
+  (via (at 42.32 48.48) (size 0.7) (drill 0.3) (layers "F.Cu" "B.Cu") (free) (net 2))
   (via (at 65.54 52.55) (size 0.7) (drill 0.3) (layers "F.Cu" "B.Cu") (net 2))
   (via (at 76.4 63.32) (size 0.7) (drill 0.3) (layers "F.Cu" "B.Cu") (net 2))
@@
   (via (at 35.46 52.47) (size 0.7) (drill 0.3) (layers "F.Cu" "B.Cu") (net 2))
   (via (at 40.47 62.99) (size 1) (drill 0.5) (layers "F.Cu" "B.Cu") (net 2))
-  (via (at 44.12 47.4) (size 0.7) (drill 0.3) (layers "F.Cu" "B.Cu") (free) (net 2))
+  (via (at 43.07 48.5) (size 0.7) (drill 0.3) (layers "F.Cu" "B.Cu") (free) (net 2))
   (via (at 59.4855 38.08) (size 1) (drill 0.5) (layers "F.Cu" "B.Cu") (net 2))
   (via (at 53.035001 46.390318) (size 1) (drill 0.5) (layers "F.Cu" "B.Cu") (net 2))
@@
       (pts
         (xy 38.87 46.89)
-        (xy 44.54 46.89)
-        (xy 44.52 48.57)
-        (xy 38.88 48.59)
+        (xy 43.67 46.94)
+        (xy 43.66 48.9)
+        (xy 38.89 48.87)
       )
     )

Commit message: EEEErrrr
Parts:
- D1: value LED -> GREEN
- D2, D3, D4, D5: value LED -> RED
- D6: value LED -> BLUE
- R13, R20: value R -> 5
- R14: value R -> 100k
- R15: value R -> 35.2k
- R16, R19: value R -> 150
- R17: value R -> 65
- R18: value R -> 530
Changed lines of the file:
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@@
     (property "ki_keywords" "inductor choke coil reactor magnetic")
     (attr smd)
-    (fp_text reference "L1" (at -2.34 -0.59 -180) (layer "F.SilkS")
+    (fp_text reference "L1" (at -2.34 -0.59) (layer "F.SilkS")
         (effects (font (size 1 1) (thickness 0.15)))
     )
-    (fp_text value "3.3uH" (at 0 2.05 -90) (layer "F.Fab")
+    (fp_text value "3.3uH" (at 0 2.05 90) (layer "F.Fab")
         (effects (font (size 1 1) (thickness 0.15)))
     )
-    (fp_text user "${REFERENCE}" (at 0 0 -90) (layer "F.Fab")
+    (fp_text user "${REFERENCE}" (at 0 0 90) (layer "F.Fab")
         (effects (font (size 0.62 0.62) (thickness 0.09)))
     )
@@
         (effects (font (size 1 1) (thickness 0.15)))
     )
-    (fp_text value "R" (at 0 1.17 90) (layer "F.Fab")
+    (fp_text value "65" (at 0 1.17 90) (layer "F.Fab")
         (effects (font (size 1 1) (thickness 0.15)))
     )
@@
         (effects (font (size 1 1) (thickness 0.15)))
     )
-    (fp_text value "R" (at 0 1.17 90) (layer "F.Fab")
+    (fp_text value "530" (at 0 1.17 90) (layer "F.Fab")
         (effects (font (size 1 1) (thickness 0.15)))
     )
@@
         (effects (font (size 1 1) (thickness 0.15)))
     )
-    (fp_text value "LED" (at 0 1.43 90) (layer "F.Fab")
+    (fp_text value "RED" (at 0 1.43 90) (layer "F.Fab")
         (effects (font (size 1 1) (thickness 0.15)))
     )
@@
         (effects (font (size 1 1) (thickness 0.15)))
     )
-    (fp_text value "R" (at 0 1.17 90) (layer "F.Fab")
+    (fp_text value "100k" (at 0 1.17 90) (layer "F.Fab")
         (effects (font (size 1 1) (thickness 0.15)))
     )
@@
         (effects (font (size 1 1) (thickness 0.15)))
     )
-    (fp_text value "R" (at 0 1.17) (layer "F.Fab")
+    (fp_text value "5" (at 0 1.17) (layer "F.Fab")
         (effects (font (size 1 1) (thickness 0.15)))
     )
@@
         (effects (font (size 1 1) (thickness 0.15)))
     )
-    (fp_text value "LED" (at 0 1.43 90) (layer "F.Fab")
+    (fp_text value "RED" (at 0 1.43 90) (layer "F.Fab")
         (effects (font (size 1 1) (thickness 0.15)))
     )
@@
         (effects (font (size 1 1) (thickness 0.15)))
     )
-    (fp_text value "LED" (at 0 1.43 90) (layer "F.Fab")
+    (fp_text value "RED" (at 0 1.43 90) (layer "F.Fab")
         (effects (font (size 1 1) (thickness 0.15)))
     )
@@
         (effects (font (size 1 1) (thickness 0.15)))
     )
-    (fp_text value "LED" (at 0 1.43 -270) (layer "F.Fab")
+    (fp_text value "RED" (at 0 1.43 -270) (layer "F.Fab")
         (effects (font (size 1 1) (thickness 0.15)))
     )
@@
         (effects (font (size 1 1) (thickness 0.15)))
     )
-    (fp_text value "R" (at 0 1.17 90) (layer "F.Fab")
+    (fp_text value "150" (at 0 1.17 90) (layer "F.Fab")
         (effects (font (size 1 1) (thickness 0.15)))
     )
@@
         (effects (font (size 1 1) (thickness 0.15)))
     )
-    (fp_text value "R" (at 0 1.17 90) (layer "F.Fab")
+    (fp_text value "35.2k" (at 0 1.17 90) (layer "F.Fab")
         (effects (font (size 1 1) (thickness 0.15)))
     )
@@
         (effects (font (size 1 1) (thickness 0.15)))
     )
-    (fp_text value "R" (at 0 1.17 90) (layer "F.Fab")
+    (fp_text value "150" (at 0 1.17 90) (layer "F.Fab")
         (effects (font (size 1 1) (thickness 0.15)))
     )
@@
         (effects (font (size 1 1) (thickness 0.15)))
     )
-    (fp_text value "R" (at 0 1.17 90) (layer "F.Fab")
+    (fp_text value "5" (at 0 1.17 90) (layer "F.Fab")
         (effects (font (size 1 1) (thickness 0.15)))
     )
@@
         (effects (font (size 1 1) (thickness 0.15)))
     )
-    (fp_text value "LED" (at 0 1.43 90) (layer "F.Fab")
+    (fp_text value "BLUE" (at 0 1.43 90) (layer "F.Fab")
         (effects (font (size 1 1) (thickness 0.15)))
     )
@@
         (effects (font (size 1 1) (thickness 0.15)))
     )
-    (fp_text value "LED" (at 0 1.43) (layer "F.Fab")
+    (fp_text value "GREEN" (at 0 1.43) (layer "F.Fab")
         (effects (font (size 1 1) (thickness 0.15)))
     )
