File: Constellation Stack V2.0/Constellation Stack V2.0.kicad_sch (KiCad schematic)
At the start: 93 parts, among them J1 PWR_IN, J2 USB_C_Receptacle_USB2.0, J3 RS485 Out, J4 PT_IN, J5 GPIO_OUT, J6 CAN_TERMINAL, Q1 MBT2222ADW1T1, SW1 RESET, SW2 SW_SPST, U1 ESP32-PICO-MINI-02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

Commit message: Work today
Parts:
- removed C15: 10uF, Capacitor_SMD:C_0402_1005Metric, symbol Device:C
- removed C16: 100nF, Capacitor_SMD:C_0402_1005Metric, symbol Device:C
- removed C17: 22uF, Capacitor_SMD:C_0402_1005Metric, symbol Device:C
- removed L1: 3.3uH, Inductor_SMD:L_1008_2520Metric, symbol Device:L
- removed R7: 52.3k, Resistor_SMD:R_0402_1005Metric, symbol Device:R
- removed R9: 10k, Resistor_SMD:R_0402_1005Metric, symbol Device:R
- removed TP3: TestPoint, TestPoint:TestPoint_Loop_D1.80mm_Drill1.0mm_Beaded, symbol Connector:TestPoint
- removed U4: AP62150Z6-7, Package_TO_SOT_SMD:TSOT-23-6, symbol AP62150Z6-7:AP62150Z6-7
- removed U5: TCR2EF50_LMCT, TCR2EF50:SOT_EF50_LMCT_TOS, symbol TCR2EF50:TCR2EF50_LMCT
- removed U6: TLV1117LV33DCYR, TLV1117LV33DCYR:VREG_TLV1117LV33DCYR, symbol TLV1117LV33DCYR:TLV1117LV33DCYR
- added C5: 1uF, Capacitor_SMD:C_1210_3225Metric, symbol Device:C
- added SW3: GPIO_0, Jumper:SolderJumper-2_P1.3mm_Open_RoundedPad1.0x1.5mm, symbol PTS636 SM50J SMTR LFS:PTS636_SM50J_SMTR_LFS
- added U10: AZ1117-3.3, Package_TO_SOT_SMD:SOT-223-3_TabPin2, symbol Regulator_Linear:AZ1117-3.3
- added U4: AP2210N-5.0TRG1, AP2210N-5.0TRG1_DIO, symbol AP2210N_5_0TRG1:AP2210N-5.0TRG1
- C1: value 1uF -> 10uF; footprint Capacitor_SMD:C_0603_1608Metric -> Capacitor_SMD:C_0402_1005Metric
- C10, C19, C20, C8: footprint Capacitor_SMD:C_0402_1005Metric -> Capacitor_SMD:C_0603_1608Metric
- C12: value 0.1uF -> 1uF
- C14: value 1uF -> 2.2uF; footprint Capacitor_SMD:C_0603_1608Metric -> Capacitor_SMD:C_0402_1005Metric
- C18, C9: footprint Capacitor_SMD:C_0402_1005Metric -> Capacitor_SMD:C_0805_2012Metric
- C2: value 1uF -> 22uF; footprint Capacitor_SMD:C_0805_2012Metric -> Capacitor_SMD:C_0603_1608Metric
- C21, C3: footprint Capacitor_SMD:C_0805_2012Metric -> Capacitor_SMD:C_0402_1005Metric
- C22, C23: footprint Capacitor_SMD:C_0603_1608Metric -> Capacitor_SMD:C_0402_1005Metric
- C24: footprint Capacitor_SMD:C_1210_3225Metric -> Capacitor_SMD:C_0402_1005Metric
- C7: footprint Capacitor_SMD:C_0603_1608Metric -> Capacitor_SMD:C_1210_3225Metric
- J2: footprint Connector_USB:USB_C_Receptacle_HCTL_HC-TYPE-C-16P-01A -> TerminalBlock_Phoenix:TerminalBlock_Phoenix_MPT-0,5-3-2.54_1x03_P2.54mm_Horizontal
- J3: footprint TerminalBlock_Phoenix:TerminalBlock_Phoenix_MPT-0,5-3-2.54_1x03_P2.54mm_Horizontal -> TerminalBlock_Phoenix:TerminalBlock_Phoenix_MPT-0,5-12-2.54_1x12_P2.54mm_Horizontal
- J4: footprint TerminalBlock_Phoenix:TerminalBlock_Phoenix_MPT-0,5-12-2.54_1x12_P2.54mm_Horizontal -> TerminalBlock_Phoenix:TerminalBlock_Phoenix_MPT-0,5-4-2.54_1x04_P2.54mm_Horizontal
- J6: footprint TerminalBlock_Phoenix:TerminalBlock_Phoenix_MPT-0,5-4-2.54_1x04_P2.54mm_Horizontal -> Connector_USB:USB_C_Receptacle_HCTL_HC-TYPE-C-16P-01A
- R1, R2, R8: footprint Resistor_SMD:R_0402_1005Metric -> Resistor_SMD:R_0805_2012Metric
- R10, R11, R12: footprint Resistor_SMD:R_0805_2012Metric -> Resistor_SMD:R_0402_1005Metric
- SW1: footprint PTS636 SM50J SMTR LFS:SW_PTS636_CNK -> Jumper:SolderJumper-2_P1.3mm_Open_RoundedPad1.0x1.5mm
- SW2: footprint Jumper:SolderJumper-2_P1.3mm_Open_RoundedPad1.0x1.5mm -> PTS636 SM50J SMTR LFS:SW_PTS636_CNK
- U1: footprint ESP32-PICO-MINI-02:MODULE_ESP32-PICO-MINI-02 -> TCR2EF50:SOT_EF50_LMCT_TOS
- U2: footprint TJA1050T:SOIC127P600X175-8N -> Package_SO:TSSOP-38_4.4x9.7mm_P0.5mm
- U3: footprint Package_DFN_QFN:QFN-24-1EP_4x4mm_P0.5mm_EP2.7x2.7mm -> TJA1050T:SOIC127P600X175-8N
- U7: footprint Package_SO:TSSOP-38_4.4x9.7mm_P0.5mm -> Package_TO_SOT_SMD:SOT-223-3_TabPin2
- U8: footprint MAX485CSA_T:21-0041-3-M_90-0096-8L_MXM -> ESP32-PICO-MINI-02:MODULE_ESP32-PICO-MINI-02
- U9: footprint W25Q16JVSSIQ:W25Q16JVSSIQ_WIN -> Package_DFN_QFN:QFN-24-1EP_4x4mm_P0.5mm_EP2.7x2.7mm
Connections:
- net +3.3V: now also U10.2 (VO)
- net +5V: now also U4.2 (VOUT)
- net BUCK_OUT: no longer C1.1, C12.1
- net GND: now also C5.2, SW3.1, U10.1 (GND), U4.1 (GND)
- net GPIO_0: now also C5.1, SW3.2
- net RESET: now also Q1.3 (C2); no longer Q1.4 (E2)
- net RTS: now also Q1.4 (E2); no longer Q1.3 (C2)
- net V IN: now also C1.1, C12.1, U10.3 (VI), U4.3 (VIN)
- no-connect marks 22 -> 21
Other:
- note added: "3.3V LDO Max In: 18V Out: 3.3V Max Amp Out: 1A"
- note added: "GPIO 0 BUTTON"
- note removed: "3.3V LDO Max In: 5.5v Out: 3.3v Max Amp Out: 1A"
- note removed: "5V OUT CONFIG"
- note removed: "Adj. Buck Converter Min/Max In: 4.2V/18V Min/Max Out: 0.8V/7V Max Amp Out: 1.5A"
- moved on the sheet: C1, C12, C14, C2, Q1B

Commit message: Ahhh
Parts:
- U1: footprint TCR2EF50:SOT_EF50_LMCT_TOS -> ESP32-PICO-MINI-02:MODULE_ESP32-PICO-MINI-02
- U2: footprint Package_SO:TSSOP-38_4.4x9.7mm_P0.5mm -> TJA1050T_CM_118:SOIC127P600X175-8N
- U4: footprint AP2210N-5.0TRG1_DIO -> AP2210N_5_0TRG1:AP2210N-5.0TRG1_DIO
Changed lines of the file:
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@@
 			)
 		)
-		(property "Footprint" "Package_SO:TSSOP-38_4.4x9.7mm_P0.5mm"
+		(property "Footprint" "TJA1050T_CM_118:SOIC127P600X175-8N"
 			(at 49.53 247.015 0)
 			(effects
@@
 			)
 		)
-		(property "Footprint" "AP2210N-5.0TRG1_DIO"
+		(property "Footprint" "AP2210N_5_0TRG1:AP2210N-5.0TRG1_DIO"
 			(at 103.886 25.908 0)
 			(effects
@@
 			)
 		)
-		(property "Footprint" "TCR2EF50:SOT_EF50_LMCT_TOS"
+		(property "Footprint" "ESP32-PICO-MINI-02:MODULE_ESP32-PICO-MINI-02"
 			(at 208.915 103.505 0)
 			(effects
@@
 			)
 		)
-		(property "Description" "\nBluetooth, WiFi 802.11b/g/n, Bluetooth v4.2 +EDR, Class 1, 2 and 3 Transceiver Module 2.412GHz ~ 2.484GHz PCB Trace Chassis Mount\n"
+		(property "Description" "Bluetooth, WiFi 802.11b/g/n, Bluetooth v4.2 +EDR, Class 1, 2 and 3 Transceiver Module 2.412GHz ~ 2.484GHz PCB Trace Chassis Mount"
 			(at 208.915 103.505 0)
 			(effects

Commit message: pUSH
Parts:
- added TP3: TestPoint, TestPoint:TestPoint_Loop_D1.80mm_Drill1.0mm_Beaded, symbol Connector:TestPoint
- U7: footprint Package_TO_SOT_SMD:SOT-223-3_TabPin2 -> Package_SO:TSSOP-32_4.4x6.5mm_P0.4mm
- U8: footprint ESP32-PICO-MINI-02:MODULE_ESP32-PICO-MINI-02 -> Package_SO:SOIC-8_3.9x4.9mm_P1.27mm
Changed lines of the file:
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@@
 			)
 		)
-		(property "Footprint" "Package_TO_SOT_SMD:SOT-223-3_TabPin2"
+		(property "Footprint" "Package_SO:TSSOP-32_4.4x6.5mm_P0.4mm"
 			(at 44.45 188.595 0)
 			(effects
@@
 			)
 		)
-		(property "Footprint" "ESP32-PICO-MINI-02:MODULE_ESP32-PICO-MINI-02"
+		(property "Footprint" "Package_SO:SOIC-8_3.9x4.9mm_P1.27mm"
 			(at 113.03 240.665 0)
 			(effects
@@
 					(italic yes)
 				)
-				(hide yes)
 			)
 		)
@@
 					(unit 1)
 				)
+			)
+		)
+	)
+	(symbol
+		(lib_id "Connector:TestPoint")
+		(at 19.05 102.235 0)
+		(mirror x)
+		(unit 1)
+		(exclude_from_sim no)
+		(in_bom yes)
+		(on_board yes)
+		(dnp no)
+		(property "Reference" "TP3"
+			(at 19.05 106.68 90)
+			(effects
+				(font
+					(size 1.27 1.27)
+				)
+				(justify left)
+			)
+		)
+		(property "Value" "TestPoint"
+			(at 20.955 104.267 0)
+			(effects
+				(font
+					(size 1.27 1.27)
+				)
+				(justify left)
+				(hide yes)
+			)
+		)
+		(property "Footprint" "TestPoint:TestPoint_Loop_D1.80mm_Drill1.0mm_Beaded"
+			(at 24.13 102.235 0)
+			(effects
+				(font
+					(size 1.27 1.27)
+				)
+				(hide yes)
+			)
+		)
+		(property "Datasheet" "~"
+			(at 24.13 102.235 0)
+			(effects
+				(font
+					(size 1.27 1.27)
+				)
+				(hide yes)
+			)
+		)
+		(property "Description" ""
+			(at 19.05 102.235 0)
+			(effects
+				(font
+					(size 1.27 1.27)
+				)
+				(hide yes)
+			)
+		)
+		(pin "1"
+		)
+		(instances
+			(project "Constellation Stack V2.0"
+				(path "/06ddcaa0-ac6e-44b3-adb2-f0cfced90a77"
+					(reference "TP3")
+					(unit 1)
+				)

Commit message: eEE errr
Parts:
- J2: footprint TerminalBlock_Phoenix:TerminalBlock_Phoenix_MPT-0,5-3-2.54_1x03_P2.54mm_Horizontal -> Connector_USB:USB_C_Receptacle_HCTL_HC-TYPE-C-16P-01A
- J3: footprint TerminalBlock_Phoenix:TerminalBlock_Phoenix_MPT-0,5-12-2.54_1x12_P2.54mm_Horizontal -> TerminalBlock_Phoenix:TerminalBlock_Phoenix_MPT-0,5-3-2.54_1x03_P2.54mm_Horizontal
- J4: footprint TerminalBlock_Phoenix:TerminalBlock_Phoenix_MPT-0,5-4-2.54_1x04_P2.54mm_Horizontal -> TerminalBlock_Phoenix:TerminalBlock_Phoenix_MPT-0,5-12-2.54_1x12_P2.54mm_Horizontal
- J6: footprint Connector_USB:USB_C_Receptacle_HCTL_HC-TYPE-C-16P-01A -> TerminalBlock_TE-Connectivity:TerminalBlock_TE_282834-4_1x04_P2.54mm_Horizontal
- U2: footprint TJA1050T_CM_118:SOIC127P600X175-8N -> Package_SO:SOIC-8_3.9x4.9mm_P1.27mm
- U3: footprint TJA1050T:SOIC127P600X175-8N -> Package_DFN_QFN:QFN-24-1EP_4x4mm_P0.5mm_EP2.7x2.7mm
- U9: footprint Package_DFN_QFN:QFN-24-1EP_4x4mm_P0.5mm_EP2.7x2.7mm -> Package_SO:SOIC-8W_5.3x5.3mm_P1.27mm
Changed lines of the file:
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@@
 			)
 		)
-		(property "Footprint" "Package_DFN_QFN:QFN-24-1EP_4x4mm_P0.5mm_EP2.7x2.7mm"
+		(property "Footprint" "Package_SO:SOIC-8W_5.3x5.3mm_P1.27mm"
 			(at 113.665 193.675 0)
 			(effects
@@
 			)
 		)
-		(property "Footprint" "TerminalBlock_Phoenix:TerminalBlock_Phoenix_MPT-0,5-3-2.54_1x03_P2.54mm_Horizontal"
+		(property "Footprint" "Connector_USB:USB_C_Receptacle_HCTL_HC-TYPE-C-16P-01A"
 			(at 392.43 102.235 0)
 			(effects
@@
 			)
 		)
-		(property "Footprint" "TJA1050T_CM_118:SOIC127P600X175-8N"
+		(property "Footprint" "Package_SO:SOIC-8_3.9x4.9mm_P1.27mm"
 			(at 49.53 247.015 0)
 			(effects
@@
 					(italic yes)
 				)
+				(hide yes)
 			)
 		)
@@
 			)
 		)
-		(property "Footprint" "TerminalBlock_Phoenix:TerminalBlock_Phoenix_MPT-0,5-12-2.54_1x12_P2.54mm_Horizontal"
+		(property "Footprint" "TerminalBlock_Phoenix:TerminalBlock_Phoenix_MPT-0,5-3-2.54_1x03_P2.54mm_Horizontal"
 			(at 175.26 245.745 0)
 			(effects
@@
 			)
 		)
-		(property "Footprint" "Connector_USB:USB_C_Receptacle_HCTL_HC-TYPE-C-16P-01A"
+		(property "Footprint" "TerminalBlock_TE-Connectivity:TerminalBlock_TE_282834-4_1x04_P2.54mm_Horizontal"
 			(at 265.43 227.965 0)
 			(effects
@@
 			)
 		)
-		(property "Footprint" "TerminalBlock_Phoenix:TerminalBlock_Phoenix_MPT-0,5-4-2.54_1x04_P2.54mm_Horizontal"
+		(property "Footprint" "TerminalBlock_Phoenix:TerminalBlock_Phoenix_MPT-0,5-12-2.54_1x12_P2.54mm_Horizontal"
 			(at 228.6 201.93 0)
 			(effects
@@
 			)
 		)
-		(property "Footprint" "TJA1050T:SOIC127P600X175-8N"
+		(property "Footprint" "Package_DFN_QFN:QFN-24-1EP_4x4mm_P0.5mm_EP2.7x2.7mm"
 			(at 427.99 219.075 0)
 			(effects

Commit message: Constella boards
Parts:
- removed D5: RED, LED_SMD:LED_0603_1608Metric, symbol Device:LED
- removed R19: 150, Resistor_SMD:R_0402_1005Metric, symbol Device:R
- removed TP20: TestPoint, TestPoint:TestPoint_Loop_D1.80mm_Drill1.0mm_Beaded, symbol Connector:TestPoint
- C1: footprint Capacitor_SMD:C_0402_1005Metric -> (none)
- C10: renamed from C5; footprint Capacitor_SMD:C_1210_3225Metric -> (none)
- C11: renamed from C22; footprint Capacitor_SMD:C_0402_1005Metric -> (none)
- C12: renamed from C23; footprint Capacitor_SMD:C_0402_1005Metric -> (none)
- C13: renamed from C11; footprint Capacitor_SMD:C_0402_1005Metric -> (none)
- C14: renamed from C9; footprint Capacitor_SMD:C_0805_2012Metric -> (none)
- C15: renamed from C21; footprint Capacitor_SMD:C_0402_1005Metric -> (none)
- C16: renamed from C20; footprint Capacitor_SMD:C_0603_1608Metric -> (none)
- C17: renamed from C24; footprint Capacitor_SMD:C_0402_1005Metric -> (none)
- C18: renamed from C25; footprint Capacitor_SMD:C_0603_1608Metric -> (none)
- C19: renamed from C26; footprint Capacitor_SMD:C_0603_1608Metric -> (none)
- C2, C8: footprint Capacitor_SMD:C_0603_1608Metric -> (none)
- C20: renamed from C13; footprint Capacitor_SMD:C_0402_1005Metric -> (none)
- C21: renamed from C18; footprint Capacitor_SMD:C_0805_2012Metric -> (none)
- C22: renamed from C19; footprint Capacitor_SMD:C_0603_1608Metric -> (none)
- C3: renamed from C12; footprint Capacitor_SMD:C_0603_1608Metric -> (none)
- C4: renamed from C14; footprint Capacitor_SMD:C_0402_1005Metric -> (none)
- C5: renamed from C3; footprint Capacitor_SMD:C_0402_1005Metric -> (none)
- C6: renamed from C4; footprint Capacitor_SMD:C_0603_1608Metric -> (none)
- C7: footprint Capacitor_SMD:C_1210_3225Metric -> (none)
- C9: renamed from C10; footprint Capacitor_SMD:C_0603_1608Metric -> (none)
- R1: renamed from R14; footprint Resistor_SMD:R_0402_1005Metric -> (none)
- R10: renamed from R3; footprint Resistor_SMD:R_0402_1005Metric -> (none)
- R11: renamed from R2; footprint Resistor_SMD:R_0805_2012Metric -> (none)
- R12: renamed from R6; footprint Resistor_SMD:R_0402_1005Metric -> (none)
- R13: renamed from R8; footprint Resistor_SMD:R_0805_2012Metric -> (none)
- R14: renamed from R12; footprint Resistor_SMD:R_0402_1005Metric -> (none)
- R15: renamed from R10; footprint Resistor_SMD:R_0402_1005Metric -> (none)
- R16: renamed from R11; footprint Resistor_SMD:R_0402_1005Metric -> (none)
- R17: renamed from R13; footprint Resistor_SMD:R_0402_1005Metric -> (none)
- R2: renamed from R18; footprint Resistor_SMD:R_0402_1005Metric -> (none)
- R3: renamed from R15; footprint Resistor_SMD:R_0402_1005Metric -> (none)
- R4: renamed from R16; footprint Resistor_SMD:R_0402_1005Metric -> (none)
- R5: renamed from R17; footprint Resistor_SMD:R_0402_1005Metric -> (none)
- R6: renamed from R4; footprint Resistor_SMD:R_0402_1005Metric -> (none)
- R7: renamed from R20; footprint Resistor_SMD:R_0402_1005Metric -> (none)
- R8: renamed from R1; footprint Resistor_SMD:R_0805_2012Metric -> (none)
- R9: renamed from R5; footprint Resistor_SMD:R_0402_1005Metric -> (none)
- SW1, SW3: footprint Jumper:SolderJumper-2_P1.3mm_Open_RoundedPad1.0x1.5mm -> PTS636SM50JSMTR LFS:SW_PTS636_CNK
- SW2: footprint PTS636 SM50J SMTR LFS:SW_PTS636_CNK -> Jumper:SolderJumper-2_P1.3mm_Open_RoundedPad1.0x1.5mm
- TP1, TP10, TP11, TP12, TP13, TP14, TP15, TP16, TP17, TP18, TP19, TP2, TP3, TP4, TP5, TP6, TP7, TP8, TP9: footprint TestPoint:TestPoint_Loop_D1.80mm_Drill1.0mm_Beaded -> (none)
- renumbered D6 to D5
Connections:
- net +3.3V: now also TP4.1; no longer TP5.1
- net +5V: now also TP3.1; no longer TP4.1
- net 485_CONTROL: now also TP13.1; no longer TP14.1
- net A: now also TP14.1; no longer TP15.1
- net ADC_CS: now also TP8.1; no longer TP9.1
- net ADC_RST: now also TP10.1; no longer TP11.1
- net B: now also TP15.1; no longer TP16.1
- net CAN_H: now also TP18.1; no longer TP19.1
- net CAN_L: now also TP19.1
- net CAN_RX: now also TP17.1; no longer TP18.1
- net CAN_TX: now also TP16.1; no longer TP17.1
- net CLK: now also TP5.1; no longer TP6.1
- net FLASH_CS: now also TP9.1; no longer TP10.1
- net MISO: now also TP7.1; no longer TP8.1
- net MOSI: now also TP6.1; no longer TP7.1
- net RXD1: now also TP11.1; no longer TP12.1
- net TXD1: now also TP12.1; no longer TP13.1
Other:
- moved on the sheet: C1, C2, C3, C4, TP1, TP10, TP11, TP12, TP13, TP14, TP15, TP16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

Commit message: Push
Parts:
- TP1, TP10, TP11, TP12, TP13, TP14, TP15, TP16, TP17, TP18, TP19, TP2, TP3, TP4, TP5, TP6, TP7, TP8, TP9: footprint (none) -> TestPoint:TestPoint_Loop_D2.60mm_Drill1.6mm_Beaded
Changed lines of the file:
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@@
 			)
 		)
-		(property "Footprint" ""
+		(property "Footprint" "TestPoint:TestPoint_Loop_D2.60mm_Drill1.6mm_Beaded"
 			(at 66.04 108.585 0)
 			(effects
@@
 			)
 		)
-		(property "Footprint" ""
+		(property "Footprint" "TestPoint:TestPoint_Loop_D2.60mm_Drill1.6mm_Beaded"
 			(at 22.86 108.585 0)
 			(effects
@@
 			)
 		)
-		(property "Footprint" ""
+		(property "Footprint" "TestPoint:TestPoint_Loop_D2.60mm_Drill1.6mm_Beaded"
 			(at 29.21 102.235 0)
 			(effects
@@
 			)
 		)
-		(property "Footprint" ""
+		(property "Footprint" "TestPoint:TestPoint_Loop_D2.60mm_Drill1.6mm_Beaded"
 			(at 43.18 108.585 0)
 			(effects
@@
 			)
 		)
-		(property "Footprint" ""
+		(property "Footprint" "TestPoint:TestPoint_Loop_D2.60mm_Drill1.6mm_Beaded"
 			(at 54.61 108.585 0)
 			(effects
@@
 			)
 		)
-		(property "Footprint" ""
+		(property "Footprint" "TestPoint:TestPoint_Loop_D2.60mm_Drill1.6mm_Beaded"
 			(at 40.64 108.585 0)
 			(effects
@@
 			)
 		)
-		(property "Footprint" ""
+		(property "Footprint" "TestPoint:TestPoint_Loop_D2.60mm_Drill1.6mm_Beaded"
 			(at 38.1 108.585 0)
 			(effects
@@
 			)
 		)
-		(property "Footprint" ""
+		(property "Footprint" "TestPoint:TestPoint_Loop_D2.60mm_Drill1.6mm_Beaded"
 			(at 68.58 108.585 0)
 			(effects
@@
 			)
 		)
-		(property "Footprint" ""
+		(property "Footprint" "TestPoint:TestPoint_Loop_D2.60mm_Drill1.6mm_Beaded"
 			(at 45.72 108.585 0)
 			(effects
@@
 			)
 		)
-		(property "Footprint" ""
+		(property "Footprint" "TestPoint:TestPoint_Loop_D2.60mm_Drill1.6mm_Beaded"
 			(at 63.5 108.585 0)
 			(effects
@@
 			)
 		)
-		(property "Footprint" ""
+		(property "Footprint" "TestPoint:TestPoint_Loop_D2.60mm_Drill1.6mm_Beaded"
 			(at 57.15 108.585 0)
 			(effects
@@
 			)
 		)
-		(property "Footprint" ""
+		(property "Footprint" "TestPoint:TestPoint_Loop_D2.60mm_Drill1.6mm_Beaded"
 			(at 59.69 108.585 0)
 			(effects
@@
 			)
 		)
-		(property "Footprint" ""
+		(property "Footprint" "TestPoint:TestPoint_Loop_D2.60mm_Drill1.6mm_Beaded"
 			(at 26.67 102.235 0)
 			(effects
@@
 			)
 		)
-		(property "Footprint" ""
+		(property "Footprint" "TestPoint:TestPoint_Loop_D2.60mm_Drill1.6mm_Beaded"
 			(at 21.59 108.585 0)
 			(effects
@@
 			)
 		)
-		(property "Footprint" ""
+		(property "Footprint" "TestPoint:TestPoint_Loop_D2.60mm_Drill1.6mm_Beaded"
 			(at 52.07 108.585 0)
 			(effects
@@
 			)
 		)
-		(property "Footprint" ""
+		(property "Footprint" "TestPoint:TestPoint_Loop_D2.60mm_Drill1.6mm_Beaded"
 			(at 24.13 108.585 0)
 			(effects
@@
 			)
 		)
-		(property "Footprint" ""
+		(property "Footprint" "TestPoint:TestPoint_Loop_D2.60mm_Drill1.6mm_Beaded"
 			(at 71.12 108.585 0)
 			(effects
@@
 			)
 		)
-		(property "Footprint" ""
+		(property "Footprint" "TestPoint:TestPoint_Loop_D2.60mm_Drill1.6mm_Beaded"
 			(at 35.56 108.585 0)
 			(effects
@@
 			)
 		)
-		(property "Footprint" ""
+		(property "Footprint" "TestPoint:TestPoint_Loop_D2.60mm_Drill1.6mm_Beaded"
 			(at 49.53 108.585 0)
 			(effects

Commit message: Stella boards
Parts:
- C1: footprint (none) -> Capacitor_SMD:C_0603_1608Metric
- C2: footprint (none) -> Capacitor_SMD:C_0402_1005Metric
Other:
- note added: "PIN OUTS"
- note removed: "SCREW TERMINAL OUTS"
Changed lines of the file:
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@@
 		)
 	)
-	(text "SCREW TERMINAL OUTS"
+	(text "PIN OUTS"
 		(exclude_from_sim no)
 		(at 221.615 178.435 0)
@@
 			)
 		)
-		(property "Footprint" ""
+		(property "Footprint" "Capacitor_SMD:C_0603_1608Metric"
 			(at 60.6552 31.115 0)
 			(effects
@@
 			)
 		)
-		(property "Footprint" ""
+		(property "Footprint" "Capacitor_SMD:C_0402_1005Metric"
 			(at 80.9752 31.115 0)
 			(effects
