File: Constellation Stack V2.0/Constellation Stack V2.0.kicad_pcb (KiCad board)
At the start: 4 copper layers, 57.1 x 50.8 mm, 96 parts, among them J1 PWR_IN, J2 USB_C_Receptacle_USB2.0, J3 RS485 Out, J4 PT_IN, J5 GPIO_OUT, J6 CAN_TERMINAL, Q1 MBT2222ADW1T1, SW1 RESET, SW2 SW_SPST, U1 ESP32-PICO-MINI-02, U2 TJA1050T_CM_118, U3 CP2102N-Axx-xQFN24, U4 AP62150Z6-7, U5 TCR2EF50_LMCT, U6 TLV1117LV33DCYR, U7 ADS8684, U8 MAX485CSA+T, U9 W25Q16JVSSIQ

Commit message: Work today
Parts:
- removed C15: 10uF, Capacitor_SMD:C_0402_1005Metric
- removed C16: 100nF, Capacitor_SMD:C_0402_1005Metric
- removed C17: 22uF, Capacitor_SMD:C_0402_1005Metric
- removed D5: RED, LED_SMD:LED_0603_1608Metric
- removed L1: 3.3uH, Inductor_SMD:L_1008_2520Metric
- removed R19: 150, Resistor_SMD:R_0402_1005Metric
- removed R7: 52.3k, Resistor_SMD:R_0402_1005Metric
- removed R9: 10k, Resistor_SMD:R_0402_1005Metric
- removed TP3: TestPoint, TestPoint:TestPoint_Loop_D1.80mm_Drill1.0mm_Beaded
- removed U4: AP62150Z6-7, Package_TO_SOT_SMD:TSOT-23-6
Routing:
- net BUCK_OUT: track 14.6 -> 4.26 mm, vias 1 -> 0
- net /SW: track 4.44 -> 0.00 mm
- net GND: track 67.5 -> 65.7 mm, vias 56 -> 53
- net Net-(D5-A): track 1.28 -> 0.00 mm
- removed copper zone on F.Cu, net /BST
- removed copper zone on F.Cu, net /FB
- removed copper zone on F.Cu, net /SW
- removed copper zone on F.Cu, net BUCK_OUT
- removed copper zone on F.Cu, net V IN
Other:
- board text removed: "BUCK LED"

Commit message: Ahahahaha
Parts:
- removed the C12 at (44.1, 39.9)
- removed TP20: TestPoint, TestPoint:TestPoint_Loop_D1.80mm_Drill1.0mm_Beaded
- removed U5: TCR2EF50_LMCT, TCR2EF50:SOT_EF50_LMCT_TOS
- removed U6: TLV1117LV33DCYR, TLV1117LV33DCYR:VREG_TLV1117LV33DCYR
- added C10: 1uF, Capacitor_SMD:C_0603_1608Metric, F.Cu at (17.0, 17.6)
- added C3: 1uF, Capacitor_SMD:C_0805_2012Metric, F.Cu at (40.8, 32.9)
- added SW3: GPIO_0, pt36:SW_PTS636_CNK, F.Cu at (10.6, 17.5)
- added TP3: TestPoint, TestPoint:TestPoint_Loop_D2.60mm_Drill1.6mm_Beaded, B.Cu at (40.9, 41.9)
- added U10: AZ1117-3.3, Package_TO_SOT_SMD:SOT-223-3_TabPin2, F.Cu at (35.2, 39.5)
- added U4: AP2210N-5.0TRG1, AP2210N_5_0TRG1:AP2210N-5.0TRG1_DIO, F.Cu at (40.9, 36.1)
- C1: value 1uF -> 10uF; footprint Capacitor_SMD:C_0603_1608Metric -> Capacitor_SMD:C_0805_2012Metric
- C13: renamed from C11; footprint Capacitor_SMD:C_0402_1005Metric -> Capacitor_SMD:C_0603_1608Metric
- C14: renamed from C9; footprint Capacitor_SMD:C_0402_1005Metric -> Capacitor_SMD:C_0603_1608Metric
- C16: renamed from C20; footprint Capacitor_SMD:C_0402_1005Metric -> Capacitor_SMD:C_0603_1608Metric
- C2: value 1uF -> 22uF; footprint Capacitor_SMD:C_0805_2012Metric -> Capacitor_SMD:C_0603_1608Metric
- C20: renamed from C13; footprint Capacitor_SMD:C_0402_1005Metric -> Capacitor_SMD:C_0603_1608Metric
- C21: renamed from C18; footprint Capacitor_SMD:C_0402_1005Metric -> Capacitor_SMD:C_0603_1608Metric
- C22: renamed from C19; footprint Capacitor_SMD:C_0402_1005Metric -> Capacitor_SMD:C_0603_1608Metric_Pad1.08x0.95mm_HandSolder
- C4: renamed from C14; value 1uF -> 2.2uF
- C8: footprint Capacitor_SMD:C_0402_1005Metric -> Capacitor_SMD:C_0603_1608Metric
- C9: renamed from C10; footprint Capacitor_SMD:C_0402_1005Metric -> Capacitor_SMD:C_0603_1608Metric
- J1, J6: footprint TerminalBlock_Phoenix:TerminalBlock_Phoenix_MPT-0,5-4-2.54_1x04_P2.54mm_Horizontal -> Connector_PinSocket_2.54mm:PinSocket_1x02_P2.54mm_Vertical; moved to F.Cu
- J3: footprint TerminalBlock_Phoenix:TerminalBlock_Phoenix_MPT-0,5-3-2.54_1x03_P2.54mm_Horizontal -> Connector_PinSocket_2.54mm:PinSocket_1x03_P2.54mm_Vertical; moved to F.Cu
- J4: footprint TerminalBlock_Phoenix:TerminalBlock_Phoenix_MPT-0,5-12-2.54_1x12_P2.54mm_Horizontal -> Connector_PinSocket_2.54mm:PinSocket_1x12_P2.54mm_Vertical; moved to F.Cu
- J5: footprint TerminalBlock_Phoenix:TerminalBlock_Phoenix_MPT-0,5-8-2.54_1x08_P2.54mm_Horizontal -> Connector_PinSocket_2.54mm:PinSocket_1x08_P2.54mm_Vertical; moved to F.Cu
- R1: renamed from R14; footprint Resistor_SMD:R_0402_1005Metric -> Resistor_SMD:R_0603_1608Metric
- R10: renamed from R3; footprint Resistor_SMD:R_0402_1005Metric -> Resistor_SMD:R_0603_1608Metric
- R11: renamed from R2; footprint Resistor_SMD:R_0402_1005Metric -> Resistor_SMD:R_0603_1608Metric
- R12: renamed from R6; footprint Resistor_SMD:R_0402_1005Metric -> Resistor_SMD:R_0603_1608Metric
- R13: renamed from R8; footprint Resistor_SMD:R_0402_1005Metric -> Resistor_SMD:R_0603_1608Metric
- R14: renamed from R12; footprint Resistor_SMD:R_0805_2012Metric -> Resistor_SMD:R_0603_1608Metric
- R17: renamed from R13; footprint Resistor_SMD:R_0402_1005Metric -> Resistor_SMD:R_0603_1608Metric
- R2: renamed from R18; footprint Resistor_SMD:R_0402_1005Metric -> Resistor_SMD:R_0603_1608Metric
- R3: renamed from R15; footprint Resistor_SMD:R_0402_1005Metric -> Resistor_SMD:R_0603_1608Metric
- R4: renamed from R16; footprint Resistor_SMD:R_0402_1005Metric -> Resistor_SMD:R_0603_1608Metric
- R5: renamed from R17; footprint Resistor_SMD:R_0402_1005Metric -> Resistor_SMD:R_0603_1608Metric
- R6: renamed from R4; footprint Resistor_SMD:R_0402_1005Metric -> Resistor_SMD:R_0603_1608Metric
- R7: renamed from R20; footprint Resistor_SMD:R_0402_1005Metric -> Resistor_SMD:R_0603_1608Metric
- R8: renamed from R1; footprint Resistor_SMD:R_0402_1005Metric -> Resistor_SMD:R_0603_1608Metric
- R9: renamed from R5; footprint Resistor_SMD:R_0402_1005Metric -> Resistor_SMD:R_0603_1608Metric
- SW1: footprint PTS636 SM50J SMTR LFS:SW_PTS636_CNK -> pt36:SW_PTS636_CNK
- TP1, TP10, TP11, TP12, TP13, TP14, TP15, TP16, TP17, TP18, TP19, TP2, TP4, TP5, TP6, TP7, TP8, TP9: footprint TestPoint:TestPoint_Loop_D1.80mm_Drill1.0mm_Beaded -> TestPoint:TestPoint_Loop_D2.60mm_Drill1.6mm_Beaded
- U2: footprint TJA1050T:SOIC127P600X175-8N -> Package_SO:SOIC-8_3.9x4.9mm_P1.27mm
- U8: footprint MAX485CSA_T:21-0041-3-M_90-0096-8L_MXM -> Package_SO:SOIC-8_3.9x4.9mm_P1.27mm
- U9: footprint W25Q16JVSSIQ:W25Q16JVSSIQ_WIN -> Package_SO:SOIC-8W_5.3x5.3mm_P1.27mm
- moved G*** 83.9 mm to (124.2, 58.4)
- moved G*** 82.1 mm to (144.6, 50.1)
- moved G*** 78.1 mm to (124.5, 49.0)
- moved TP5 59.9 mm to (89.8, 52.0)
- moved TP4 23.8 mm to (27.5, 45.5)
- moved TP10 19.9 mm to (85.2, 64.9)
- moved TP16 17.9 mm to (34.6, 85.0)
- moved TP14 15.7 mm to (31.4, 64.3)
- moved C1 14.3 mm to (32.9, 33.3), turned to 90 degrees
- moved C2 14.1 mm to (36.3, 34.1), turned to 0 degrees
- moved TP18 12.6 mm to (50.5, 67.3)
- moved TP9 11.3 mm to (62.2, 51.3)
- moved R9 10.3 mm to (38.8, 46.6), turned to 90 degrees
- moved C4 9.05 mm to (41.1, 39.1), turned to 180 degrees
- moved Q1 8.94 mm to (40.8, 45.9), turned to 90 degrees
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- renumbered C22 to C11, C23 to C12, C21 to C15, C24 to C17, C25 to C18, C26 to C19, C3 to C5, C4 to C6, D6 to D5, R10 to R15, R11 to R16
Connections:
- C1 pad 1: BUCK_OUT -> V IN
- Q1 pad 3: RTS -> RESET
- Q1 pad 4: RESET -> RTS
- TP10 pad 1: FLASH_CS -> ADC_RST
- TP11 pad 1: ADC_RST -> RXD1
- TP12 pad 1: RXD1 -> TXD1
- TP13 pad 1: TXD1 -> 485_CONTROL
- TP14 pad 1: 485_CONTROL -> A
- TP15 pad 1: A -> B
- TP16 pad 1: B -> CAN_TX
- TP17 pad 1: CAN_TX -> CAN_RX
- TP18 pad 1: CAN_RX -> CAN_H
- TP19 pad 1: CAN_H -> CAN_L
- TP4 pad 1: +5V -> +3.3V
- TP5 pad 1: +3.3V -> CLK
- TP6 pad 1: CLK -> MOSI
- TP7 pad 1: MOSI -> MISO
- TP8 pad 1: MISO -> ADC_CS
- TP9 pad 1: ADC_CS -> FLASH_CS
Routing:
- net V IN: track 76.7 -> 0.00 mm
- net V_BATT: track 68.6 -> 0.00 mm, vias 2 -> 0
- net GND: track 65.7 -> 0.00 mm, vias 53 -> 0
- net +5V: track 59.1 -> 0.00 mm, vias 4 -> 0
- net MOSI: track 46.1 -> 0.00 mm, vias 1 -> 0
- net MISO: track 45.9 -> 0.00 mm, vias 3 -> 0
- net CLK: track 45.1 -> 0.00 mm, vias 4 -> 0
- net 485_CONTROL: track 44.0 -> 0.00 mm, vias 1 -> 0
- net GPIO_OUT_5: track 34.2 -> 0.00 mm, vias 3 -> 0
- net TXD0: track 32.8 -> 0.00 mm, vias 2 -> 0
- net TXD1: track 32.1 -> 0.00 mm, vias 1 -> 0
- net GPIO_OUT_4: track 31.9 -> 0.00 mm, vias 3 -> 0
- net RXD0: track 31.4 -> 0.00 mm
- net RXD1: track 31.2 -> 0.00 mm, vias 1 -> 0
- net GPIO_OUT_3: track 30.5 -> 0.00 mm, vias 3 -> 0
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- removed copper zone on F.Cu, net +5V
Other:
- board size 57.1 x 50.8 mm -> 50.8 x 50.8 mm

Commit message: Constella V2.0 Work
Parts:
- TP1: footprint TestPoint:TestPoint_Loop_D2.60mm_Drill1.6mm_Beaded -> Connector_Pin:Pin_D1.0mm_L10.0mm_LooseFit
- TP10, TP11, TP12, TP13, TP14, TP15, TP16, TP17, TP18, TP19, TP5, TP6, TP7, TP8, TP9: footprint TestPoint:TestPoint_Loop_D2.60mm_Drill1.6mm_Beaded -> Connector_Pin:Pin_D1.3mm_L11.0mm_LooseFit
- TP2, TP3, TP4: footprint TestPoint:TestPoint_Loop_D2.60mm_Drill1.6mm_Beaded -> TestPoint:TestPoint_Pad_D2.0mm
- moved G*** 85.1 mm to (39.3, 54.0)
- moved G*** 77.6 mm to (67.4, 58.1)
- moved G*** 66.0 mm to (61.1, 67.6)
- moved SW3 57.4 mm to (57.2, 50.8)
- moved C10 56.9 mm to (62.1, 52.2), turned to -90 degrees
- moved TP16 36.2 mm to (55.1, 55.3)
- moved TP5 30.9 mm to (60.4, 61.7)
- moved TP10 29.6 mm to (104.3, 42.3)
- moved TP11 27.7 mm to (44.3, 65.8)
- moved R2 26.7 mm to (40.6, 31.0), turned to 0 degrees
- moved TP8 26.6 mm to (94.6, 43.5)
- moved D4 24.0 mm to (43.7, 31.0), turned to 180 degrees
- moved R5 22.9 mm to (56.4, 63.5)
- moved D3 22.9 mm to (56.4, 60.3)
- moved TP9 13.5 mm to (72.5, 60.1)
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Routing:
- net GND: track 0.00 -> 27.0 mm, vias 0 -> 25
- net FLASH_CS: track 0.00 -> 20.0 mm
- net MISO: track 0.00 -> 19.9 mm
- net V IN: track 0.00 -> 19.0 mm
- net CLK: track 0.00 -> 18.0 mm
- net VBUS: track 0.00 -> 17.5 mm
- net MOSI: track 0.00 -> 17.5 mm
- net CAN_L: track 0.00 -> 15.9 mm
- net AN_IN_0: track 0.00 -> 12.8 mm
- net 485_CONTROL: track 0.00 -> 12.7 mm
- net B: track 0.00 -> 11.0 mm
- net +5V: track 0.00 -> 9.38 mm
- net A: track 0.00 -> 9.21 mm
- net D+: track 0.00 -> 9.00 mm
- net D-: track 0.00 -> 8.98 mm
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- added copper zone on F.Cu, net V IN
Other:
- board text removed: "BUCK_OUT"

Commit message: Push
Parts:
- removed U1: ESP32-PICO-MINI-02, ESP32-PICO-MINI-02:MODULE_ESP32-PICO-MINI-02
- added U5: ESP32-PICO-MINI-02U-N8R2, ESP32-PICO-MINI-02U:MODULE_ESP32-PICO-MINI-02U-N8R2, F.Cu at (62.0, 61.5)
- J4: footprint Connector_PinSocket_2.54mm:PinSocket_1x12_P2.54mm_Vertical -> Connector_PinSocket_2.54mm:PinSocket_1x04_P2.54mm_Vertical
- J5: footprint Connector_PinSocket_2.54mm:PinSocket_1x08_P2.54mm_Vertical -> Connector_PinSocket_2.54mm:PinSocket_1x06_P2.54mm_Vertical
- moved C6 37.5 mm to (58.9, 71.3), turned to 180 degrees
- moved TP9 37.5 mm to (109.8, 56.6)
- moved TP6 36.0 mm to (104.1, 56.5)
- moved TP10 35.9 mm to (69.2, 35.0)
- moved J5 33.1 mm to (74.3, 41.9), turned to 0 degrees
- moved C5 32.8 mm to (60.6, 69.5), turned to 0 degrees
- moved D5 31.0 mm to (73.9, 64.2), turned to 180 degrees
- moved TP7 30.5 mm to (55.6, 42.6)
- moved TP8 30.0 mm to (65.3, 37.4)
- moved R7 27.4 mm to (70.9, 64.2), turned to 0 degrees
- moved G*** 26.9 mm to (90.5, 71.8)
- moved SW3 24.4 mm to (80.6, 57.8)
- moved C10 24.4 mm to (85.5, 59.2)
- moved C16 23.4 mm to (56.8, 45.9), turned to -90 degrees
- moved U9 21.7 mm to (62.4, 44.4), turned to 0 degrees
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Connections:
- J4 pad 1: GND -> AN_IN_3
- J4 pad 2: AN_IN_3 -> AN_IN_2
- J4 pad 3: V IN -> AN_IN_1
- J4 pad 4: GND -> AN_IN_0
- J5 pad 1: +3.3V -> GPIO_OUT_0
- J5 pad 2: GPIO_OUT_0 -> GPIO_OUT_1
- J5 pad 3: GPIO_OUT_1 -> GPIO_OUT_2
- J5 pad 4: GPIO_OUT_2 -> GPIO_OUT_3
- J5 pad 5: GPIO_OUT_3 -> GPIO_OUT_4
- J5 pad 6: GPIO_OUT_4 -> GPIO_OUT_5
Routing:
- net CAN_RX: track 0.00 -> 26.9 mm, vias 0 -> 1
- net RXD1: track 0.00 -> 24.9 mm, vias 0 -> 1
- net 485_CONTROL: track 12.7 -> 37.6 mm, vias 0 -> 2
- net TXD1: track 2.76 -> 27.2 mm, vias 0 -> 1
- net TXD0: track 0.00 -> 23.0 mm, vias 0 -> 2
- net GPIO_OUT_0: track 0.00 -> 22.2 mm
- net RXD0: track 0.00 -> 21.9 mm, vias 0 -> 2
- net CAN_TX: track 0.00 -> 21.5 mm, vias 0 -> 1
- net GPIO_OUT_1: track 0.00 -> 20.5 mm
- net GPIO_OUT_2: track 0.00 -> 18.9 mm
- net GPIO_OUT_3: track 0.00 -> 17.3 mm
- net GPIO_OUT_4: track 0.00 -> 15.8 mm
- net CAN_H: track 5.75 -> 21.4 mm, vias 0 -> 1
- net MOSI: track 17.5 -> 31.9 mm
- net GPIO_OUT_5: track 0.00 -> 14.2 mm
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- added copper zone on F.Cu, net GPIO_0
Other:
- board text removed: "+3.3"
- board text removed: "-"

Commit message: Aaaaa
Parts:
- moved U5 27.9 mm to (55.0, 88.5), turned to 180 degrees
- moved C6 21.1 mm to (64.8, 91.5), turned to -90 degrees
- moved C5 20.5 mm to (63.0, 89.9), turned to 90 degrees
Routing:
- net 485_CONTROL: track 37.6 -> 0.00 mm, vias 2 -> 0
- net MOSI: track 31.9 -> 0.00 mm
- net CLK: track 29.7 -> 0.00 mm, vias 2 -> 0
- net GND: track 28.9 -> 0.00 mm, vias 36 -> 0
- net TXD1: track 27.2 -> 0.00 mm, vias 1 -> 0
- net CAN_RX: track 26.9 -> 0.00 mm, vias 1 -> 0
- net MISO: track 26.2 -> 0.00 mm
- net RXD1: track 24.9 -> 0.00 mm, vias 1 -> 0
- net TXD0: track 23.0 -> 0.00 mm, vias 2 -> 0
- net GPIO_OUT_0: track 22.2 -> 0.00 mm
- net RXD0: track 21.9 -> 0.00 mm, vias 2 -> 0
- net CAN_TX: track 21.5 -> 0.00 mm, vias 1 -> 0
- net CAN_H: track 21.4 -> 0.00 mm, vias 1 -> 0
- net V IN: track 21.0 -> 0.00 mm, vias 1 -> 0
- net GPIO_OUT_1: track 20.5 -> 0.00 mm
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
Commit message: GERBS MADE
Parts:
- moved TP2 99.1 mm to (133.7, 15.5)
- moved TP1 80.9 mm to (97.2, 78.5)
- moved TP9 73.9 mm to (39.0, 77.9)
- moved TP13 70.4 mm to (112.2, 41.4)
- moved C20 67.9 mm to (115.2, 36.1)
- moved TP6 67.8 mm to (36.4, 61.0)
- moved TP4 59.7 mm to (85.4, 26.7), turned to 0 degrees
- moved D2 58.3 mm to (98.9, 53.9), turned to 180 degrees
- moved C4 55.0 mm to (94.8, 51.3), turned to 90 degrees
- moved R4 54.5 mm to (95.9, 53.9), turned to 0 degrees
- moved J3 53.1 mm to (62.0, 27.2), turned to 90 degrees
- moved J1 52.4 mm to (63.4, 74.4), turned to -90 degrees
- moved TP3 52.0 mm to (92.1, 51.1), turned to 90 degrees
- moved D4 51.2 mm to (81.3, 65.8), turned to -90 degrees
- moved D1 50.0 mm to (73.5, 36.6), turned to 180 degrees
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Routing:
- net 485_CONTROL: track 0.00 -> 49.7 mm, vias 0 -> 2
- net TXD1: track 0.00 -> 47.8 mm
- net RXD1: track 0.00 -> 41.7 mm, vias 0 -> 1
- net GND: track 0.00 -> 37.7 mm, vias 0 -> 30
- net MISO: track 0.00 -> 36.0 mm
- net TXD0: track 0.00 -> 36.0 mm, vias 0 -> 2
- net RXD0: track 0.00 -> 33.9 mm, vias 0 -> 2
- net ADC_RST: track 0.00 -> 31.8 mm, vias 0 -> 3
- net ADC_CS: track 0.00 -> 27.6 mm, vias 0 -> 3
- net CAN_TX: track 0.00 -> 27.5 mm
- net MOSI: track 0.00 -> 25.8 mm
- net CAN_RX: track 0.00 -> 25.7 mm, vias 0 -> 1
- net CLK: track 0.00 -> 22.4 mm, vias 0 -> 2
- net CAN_H: track 0.00 -> 21.4 mm, vias 0 -> 1
- net CAN_L: track 0.00 -> 19.6 mm
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Other:
- board text added: "CANBUS OUT"
- board text added: "GPIO_0"
- board text removed: "CAN BUS OUT"

Commit message: Ye haw looking 2.0
Parts:
- removed C1, C15, C5: 10uF, Capacitor_SMD:C_0805_2012Metric
- removed C10, C11, C12, C18, C20, C7: 1uF, Capacitor_SMD:C_0603_1608Metric
- removed C13, C14: 0.1uf, Capacitor_SMD:C_0603_1608Metric
- removed C16, C6: 0.1uF, Capacitor_SMD:C_0603_1608Metric
- removed C17: 22uF, Capacitor_SMD:C_1210_3225Metric
- removed C19: 10uF, Capacitor_SMD:C_0603_1608Metric
- removed C2: 22uF, Capacitor_SMD:C_0603_1608Metric
- removed C21: 47nf, Capacitor_SMD:C_0603_1608Metric
- removed C22: 0.1uF, Capacitor_SMD:C_0603_1608Metric_Pad1.08x0.95mm_HandSolder
- removed C3: 1uF, Capacitor_SMD:C_0805_2012Metric
- removed C4: 2.2uF, Capacitor_SMD:C_0603_1608Metric
- removed C8, C9: 4.7uf, Capacitor_SMD:C_0603_1608Metric
- removed D1: GREEN, LED_SMD:LED_0603_1608Metric
- removed D2, D3, D4: RED, LED_SMD:LED_0603_1608Metric
- removed D5: BLUE, LED_SMD:LED_0603_1608Metric
- removed the G*** at (97.0, 40.8)
- removed H1, H2, H3, H4: MountingHole_Pad, MountingHole:MountingHole_3.2mm_M3_DIN965_Pad
- removed J1: PWR_IN, Connector_PinSocket_2.54mm:PinSocket_1x02_P2.54mm_Vertical
- removed J2: USB_C_Receptacle_USB2.0, Connector_USB:USB_C_Receptacle_HCTL_HC-TYPE-C-16P-01A
- removed J3: RS485 Out, Connector_PinSocket_2.54mm:PinSocket_1x03_P2.54mm_Vertical
- removed J4: PT_IN, Connector_PinSocket_2.54mm:PinSocket_1x04_P2.54mm_Vertical
- removed J5: GPIO_OUT, Connector_PinSocket_2.54mm:PinSocket_1x06_P2.54mm_Vertical
- removed J6: CAN_TERMINAL, Connector_PinSocket_2.54mm:PinSocket_1x02_P2.54mm_Vertical
- removed Q1: MBT2222ADW1T1, Package_TO_SOT_SMD:SOT-363_SC-70-6
- removed R1: 100k, Resistor_SMD:R_0603_1608Metric
- removed R10, R11: 5.1k, Resistor_SMD:R_0603_1608Metric
- removed R12: 22.1k, Resistor_SMD:R_0603_1608Metric
- removed R13: 47.5k, Resistor_SMD:R_0603_1608Metric
- removed R14: 120, Resistor_SMD:R_0603_1608Metric
- removed R15, R16: 60, Resistor_SMD:R_0805_2012Metric
- removed R17, R7: 5, Resistor_SMD:R_0603_1608Metric
- removed R2: 530, Resistor_SMD:R_0603_1608Metric
- removed R3: 35.2k, Resistor_SMD:R_0603_1608Metric
- removed R4: 150, Resistor_SMD:R_0603_1608Metric
- removed R5: 65, Resistor_SMD:R_0603_1608Metric
- removed R6, R8, R9: 10k, Resistor_SMD:R_0603_1608Metric
- removed SW1: RESET, pt36:SW_PTS636_CNK
- removed SW2: SW_SPST, Jumper:SolderJumper-2_P1.3mm_Open_RoundedPad1.0x1.5mm
- removed SW3: GPIO_0, pt36:SW_PTS636_CNK
- removed TP1: TestPoint, Connector_Pin:Pin_D1.0mm_L10.0mm_LooseFit
- removed TP10, TP11, TP12, TP13, TP14, TP15, TP16, TP17, TP18, TP19, TP5, TP6, TP7, TP8, TP9: TestPoint, Connector_Pin:Pin_D1.3mm_L11.0mm_LooseFit
- removed TP2, TP3, TP4: TestPoint, TestPoint:TestPoint_Pad_D2.0mm
- removed U10: AZ1117-3.3, Package_TO_SOT_SMD:SOT-223-3_TabPin2
- removed U2: TJA1050T_CM_118, Package_SO:SOIC-8_3.9x4.9mm_P1.27mm
- removed U3: CP2102N-Axx-xQFN24, Package_DFN_QFN:QFN-24-1EP_4x4mm_P0.5mm_EP2.7x2.7mm
- removed U4: AP2210N-5.0TRG1, AP2210N_5_0TRG1:AP2210N-5.0TRG1_DIO
- removed U5: ESP32-PICO-MINI-02U-N8R2, ESP32-PICO-MINI-02U:MODULE_ESP32-PICO-MINI-02U-N8R2
- removed U7: ADS8684, Package_SO:TSSOP-38_4.4x9.7mm_P0.5mm
- removed U8: MAX485CSA+T, Package_SO:SOIC-8_3.9x4.9mm_P1.27mm
- removed U9: W25Q16JVSSIQ, Package_SO:SOIC-8W_5.3x5.3mm_P1.27mm
Routing:
- net 485_CONTROL: track 49.7 -> 0.00 mm, vias 2 -> 0
- net TXD1: track 47.8 -> 0.00 mm
- net RXD1: track 41.7 -> 0.00 mm, vias 1 -> 0
- net GND: track 37.7 -> 0.00 mm, vias 30 -> 0
- net MISO: track 36.0 -> 0.00 mm
- net TXD0: track 36.0 -> 0.00 mm, vias 2 -> 0
- net RXD0: track 33.9 -> 0.00 mm, vias 2 -> 0
- net ADC_RST: track 31.8 -> 0.00 mm, vias 3 -> 0
- net ADC_CS: track 27.6 -> 0.00 mm, vias 3 -> 0
- net CAN_TX: track 27.5 -> 0.00 mm
- net MOSI: track 25.8 -> 0.00 mm
- net CAN_RX: track 25.7 -> 0.00 mm, vias 1 -> 0
- net CLK: track 22.4 -> 0.00 mm, vias 2 -> 0
- net CAN_H: track 21.4 -> 0.00 mm, vias 1 -> 0
- net CAN_L: track 19.6 -> 0.00 mm
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- removed copper zone on F.Cu, net +3.3V
- removed copper zone on F.Cu, net GND
- removed copper zone on F.Cu, net GPIO_0
- removed copper zone on F.Cu, net RESET
- removed copper zone on F.Cu, net V IN
Other:
- board outline removed
- board text removed: "+"
- board text removed: "1"
- board text removed: "2"
- board text removed: "3"
- board text removed: "3.3 PWR"
- board text removed: "4"
- board text removed: "5"
- board text removed: "5V LED"
- board text removed: "6"
- board text removed: "A"
- board text removed: "B"
- board text removed: "CANBUS OUT"
- board text removed: "GPIOS OUT"
- board text removed: "GPIO_0"
- board text removed: "H"
- board text removed: "L"
- board text removed: "LED"
- board text removed: "PT PORTS IN"
- board text removed: "PWR IN"
- board text removed: "RESET"
- board text removed: "RS485 LED"
- board text removed: "RS485 OUT"
- board text removed: "USB C"
- board text removed: "V IN"
