File: Constellation Stack V2.0/Constellation Stack V2.0.kicad_pcb (KiCad board)
At the start: 4 copper layers, 2 parts

Commit message: 69 changes
Parts:
- added C1: 100nF, Capacitor_SMD:C_0603_1608Metric, F.Cu at (70.3, 40.2)
- added C10: 1uF, Capacitor_SMD:C_0603_1608Metric, F.Cu at (57.3, 58.4)
- added C11: 4.7uf, Capacitor_SMD:C_0603_1608Metric, F.Cu at (36.8, 48.1)
- added C12: 4.7uf, Capacitor_SMD:C_0603_1608Metric, F.Cu at (40.9, 47.0)
- added C13: 1uF, Capacitor_SMD:C_0603_1608Metric, F.Cu at (34.7, 67.1)
- added C14: 1uF, Capacitor_SMD:C_0603_1608Metric, F.Cu at (34.1, 57.8)
- added C15: 0.1uf, Capacitor_SMD:C_0603_1608Metric, F.Cu at (35.2, 48.1)
- added C16: 0.1uf, Capacitor_SMD:C_0603_1608Metric, F.Cu at (39.3, 47.0)
- added C17: 10uF, Capacitor_SMD:C_0805_2012Metric, F.Cu at (37.2, 68.1)
- added C18: 0.1uF, Capacitor_SMD:C_0603_1608Metric, F.Cu at (42.8, 73.1)
- added C19: 22uF, Capacitor_SMD:C_1210_3225Metric, F.Cu at (34.1, 53.7)
- added C2: 10uF, Capacitor_SMD:C_0805_2012Metric, F.Cu at (74.9, 37.6)
- added C20: 1uF, Capacitor_SMD:C_0603_1608Metric, F.Cu at (35.6, 56.1)
- added C21: 10uF, Capacitor_SMD:C_0603_1608Metric, F.Cu at (38.0, 56.9)
- added C22: 1uF, Capacitor_SMD:C_0603_1608Metric, F.Cu at (56.7, 47.4)
- added C23: 47nf, Capacitor_SMD:C_0603_1608Metric, F.Cu at (58.8, 36.3)
- added C24: 0.1uF, Capacitor_SMD:C_0603_1608Metric, F.Cu at (42.2, 42.1)
- added C3: 22uF, Capacitor_SMD:C_0603_1608Metric, F.Cu at (74.9, 41.1)
- added C4: 1uF, Capacitor_SMD:C_0603_1608Metric, F.Cu at (65.9, 47.1)
- added C5: 1uF, Capacitor_SMD:C_0805_2012Metric, F.Cu at (72.3, 47.1)
- added C6: 1uF, Capacitor_SMD:C_0805_2012Metric, F.Cu at (75.0, 51.5)
- added C7: 4.7uF, Capacitor_SMD:C_0603_1608Metric, F.Cu at (64.2, 55.3)
- added C8: 10uF, Capacitor_SMD:C_0805_2012Metric, F.Cu at (63.6, 79.8)
- added C9: 0.1uF, Capacitor_SMD:C_0603_1608Metric, F.Cu at (61.7, 79.6)
- added D1: RED, LED_SMD:LED_0603_1608Metric, F.Cu at (80.4, 33.4)
- added D2: RED, LED_SMD:LED_0603_1608Metric, F.Cu at (64.4, 39.3)
- added D3: RED, LED_SMD:LED_0603_1608Metric, F.Cu at (60.8, 41.7)
- added D4: RED, LED_SMD:LED_0603_1608Metric, F.Cu at (27.8, 33.4)
- added D5: BLUE, LED_SMD:LED_0603_1608Metric, F.Cu at (73.2, 70.1)
- added D6: GREEN, LED_SMD:LED_0603_1608Metric, F.Cu at (46.9, 27.7)
- added G***: LOGO, LOGO:RP_Logo, F.Cu at (72.3, 75.6)
- added H1: MountingHole_Pad, MountingHole:MountingHole_3.2mm_M3_DIN965_Pad, F.Cu at (29.2, 29.2)
- added H2: MountingHole_Pad, MountingHole:MountingHole_3.2mm_M3_DIN965_Pad, F.Cu at (78.7, 29.2)
- added H3: MountingHole_Pad, MountingHole:MountingHole_3.2mm_M3_DIN965_Pad, F.Cu at (29.2, 78.7)
- added H4: MountingHole_Pad, MountingHole:MountingHole_3.2mm_M3_DIN965_Pad, F.Cu at (78.7, 78.7)
- added J1: PWR, Connector_PinSocket_2.54mm:PinSocket_1x02_P2.54mm_Vertical, B.Cu at (69.8, 27.9)
- added J2: USB_C_Receptacle_USB2.0, Connector_USB:USB_C_Receptacle_HCTL_HC-TYPE-C-16P-01A, F.Cu at (29.2, 44.5)
- added J3: PT_IN, Connector_PinSocket_2.54mm:PinSocket_1x04_P2.54mm_Vertical, B.Cu at (27.9, 66.0)
- added J5: CAN_TERMINAL, Connector_PinSocket_2.54mm:PinSocket_1x02_P2.54mm_Vertical, B.Cu at (57.1, 27.9)
- added J7: RS485 Out, Connector_PinSocket_2.54mm:PinSocket_1x03_P2.54mm_Vertical, B.Cu at (38.1, 27.9)
- added J8: GPIO/ESP_ADC OUT, Connector_PinSocket_2.54mm:PinSocket_1x14_P2.54mm_Vertical, B.Cu at (80.0, 36.8)
- added L1: 3.3uH, Inductor_SMD:L_1008_2520Metric, F.Cu at (72.1, 42.5)
- added Q1: MBT2222ADW1T1, Package_TO_SOT_SMD:SOT-363_SC-70-6, F.Cu at (58.2, 55.0)
- added Q2: DMP3099L, Package_TO_SOT_SMD:SOT-23-3, F.Cu at (67.4, 32.3)
- added R1: 100k, Resistor_SMD:R_0603_1608Metric, F.Cu at (67.6, 35.2)
- added R10: 5, Resistor_SMD:R_0603_1608Metric, F.Cu at (70.2, 70.1)
- added R11: 10k, Resistor_SMD:R_0603_1608Metric, F.Cu at (54.3, 58.4)
- added R12: 10k, Resistor_SMD:R_0603_1608Metric, F.Cu at (55.8, 54.1)
- added R13: 5.1k, Resistor_SMD:R_0603_1608Metric, F.Cu at (36.0, 45.7)
- added R14: 5.1k, Resistor_SMD:R_0603_1608Metric, F.Cu at (35.2, 41.7)
- added R15: 22.1k, Resistor_SMD:R_0603_1608Metric, F.Cu at (38.8, 50.0)
- added R16: 47.5k, Resistor_SMD:R_0603_1608Metric, F.Cu at (38.0, 52.3)
- added R17: 120, Resistor_SMD:R_0805_2012Metric, F.Cu at (38.9, 35.0)
- added R18: 60, Resistor_SMD:R_0805_2012Metric, F.Cu at (57.1, 36.2)
- added R19: 60, Resistor_SMD:R_0805_2012Metric, F.Cu at (60.6, 36.2)
- added R2: 68k, Resistor_SMD:R_0603_1608Metric, F.Cu at (66.7, 36.8)
- added R20: 5, Resistor_SMD:R_0603_1608Metric, F.Cu at (46.9, 30.8)
- added R3: 750, Resistor_SMD:R_0603_1608Metric, F.Cu at (77.3, 33.4)
- added R4: 270, Resistor_SMD:R_0603_1608Metric, F.Cu at (64.4, 42.4)
- added R5: 10k, Resistor_SMD:R_0603_1608Metric, F.Cu at (69.0, 37.6)
- added R6: 24.3k, Resistor_SMD:R_0603_1608Metric, F.Cu at (64.6, 35.2)
- added R7: 150, Resistor_SMD:R_0603_1608Metric, F.Cu at (60.8, 44.8)
- added R8: 65, Resistor_SMD:R_0603_1608Metric, F.Cu at (30.8, 33.4)
- added R9: 10k, Resistor_SMD:R_0603_1608Metric, F.Cu at (60.7, 55.6)
- added SW1: RESET, PTS636SM50JSMTR LFS:SW_PTS636_CNK, F.Cu at (55.8, 63.2)
- added SW2: GPIO_0, PTS636SM50JSMTR LFS:SW_PTS636_CNK, F.Cu at (60.2, 63.2)
- added SW3: SW_SPST, Jumper:SolderJumper-2_P1.3mm_Open_RoundedPad1.0x1.5mm, B.Cu at (56.1, 35.3)
- added TP1: TestPoint, TestPoint:TestPoint_Loop_D2.60mm_Drill1.6mm_Beaded, B.Cu at (63.3, 47.8)
- added TP10: TestPoint, TestPoint:TestPoint_Loop_D2.60mm_Drill1.6mm_Beaded, B.Cu at (40.2, 79.5)
- added TP11: TestPoint, TestPoint:TestPoint_Loop_D2.60mm_Drill1.6mm_Beaded, B.Cu at (42.5, 56.1)
- added TP12: TestPoint, TestPoint:TestPoint_Loop_D2.60mm_Drill1.6mm_Beaded, B.Cu at (48.2, 46.7)
- added TP13: TestPoint, TestPoint:TestPoint_Loop_D2.60mm_Drill1.6mm_Beaded, B.Cu at (44.5, 44.6)
- added TP14: TestPoint, TestPoint:TestPoint_Loop_D2.60mm_Drill1.6mm_Beaded, B.Cu at (50.4, 41.2)
- added TP15: TestPoint, TestPoint:TestPoint_Loop_D2.60mm_Drill1.6mm_Beaded, B.Cu at (41.4, 31.9)
- added TP16: TestPoint, TestPoint:TestPoint_Loop_D2.60mm_Drill1.6mm_Beaded, B.Cu at (36.2, 31.9)
- added TP17: TestPoint, TestPoint:TestPoint_Loop_D2.60mm_Drill1.6mm_Beaded, B.Cu at (56.6, 50.4)
- added TP18: TestPoint, TestPoint:TestPoint_Loop_D2.60mm_Drill1.6mm_Beaded, B.Cu at (52.2, 50.3)
- added TP19: TestPoint, TestPoint:TestPoint_Loop_D2.60mm_Drill1.6mm_Beaded, B.Cu at (55.7, 31.7)
- added TP2: TestPoint, TestPoint:TestPoint_Loop_D2.60mm_Drill1.6mm_Beaded, B.Cu at (62.9, 28.0)
- added TP20: TestPoint, TestPoint:TestPoint_Loop_D2.60mm_Drill1.6mm_Beaded, B.Cu at (59.9, 31.7)
- added TP3: TestPoint, TestPoint:TestPoint_Loop_D2.60mm_Drill1.6mm_Beaded, B.Cu at (73.8, 27.9)
- added TP4: TestPoint, TestPoint:TestPoint_Loop_D2.60mm_Drill1.6mm_Beaded, B.Cu at (72.5, 32.7)
- added TP5: TestPoint, TestPoint:TestPoint_Loop_D2.60mm_Drill1.6mm_Beaded, B.Cu at (75.3, 45.1)
- added TP6: TestPoint, TestPoint:TestPoint_Loop_D2.60mm_Drill1.6mm_Beaded, B.Cu at (42.1, 67.8)
- added TP7: TestPoint, TestPoint:TestPoint_Loop_D2.60mm_Drill1.6mm_Beaded, B.Cu at (44.6, 77.6)
- added TP8: TestPoint, TestPoint:TestPoint_Loop_D2.60mm_Drill1.6mm_Beaded, B.Cu at (35.9, 79.5)
- added TP9: TestPoint, TestPoint:TestPoint_Loop_D2.60mm_Drill1.6mm_Beaded, B.Cu at (42.2, 62.5)
- added U1: AP62150Z6-7, Package_TO_SOT_SMD:TSOT-23-6, F.Cu at (71.8, 37.7)
- added U2: LDK320AM50R, Package_TO_SOT_SMD:SC-74A-5_1.55x2.9mm_P0.95mm, F.Cu at (69.0, 47.1)
- added U3: LDL1117S33R, Package_TO_SOT_SMD:SOT-223, F.Cu at (69.5, 53.1)
- added U4: ESP32-PICO-MINI-02U-N8R2, ESP32-PICO-MINI-02U:MODULE_ESP32-PICO-MINI-02U-N8R2, F.Cu at (54.0, 76.2)
- added U5: ADS8684, Package_SO:TSSOP-38_4.4x9.7mm_P0.5mm, F.Cu at (34.9, 62.4)
- added U6: CP2102N-Axx-xQFN24, Package_DFN_QFN:QFN-24-1EP_4x4mm_P0.5mm_EP2.7x2.7mm, F.Cu at (42.2, 51.2)
- added U7: W25Q16JVSSIQ, Package_SO:SOIC-8_5.275x5.275mm_P1.27mm, F.Cu at (37.3, 74.3)
- added U8: MAX485CSA+T, Package_SO:SOIC-8_3.9x4.9mm_P1.27mm, F.Cu at (44.4, 38.5)
- added U9: TJA1050T_CM_118, Package_SO:SOIC-8_3.9x4.9mm_P1.27mm, F.Cu at (56.9, 42.9)
Routing:
- net +5V: track 0.00 -> 97.1 mm, vias 0 -> 4
- net V_BATT: track 0.00 -> 73.2 mm, vias 0 -> 2
- net GND: track 0.00 -> 53.1 mm, vias 0 -> 60
- net GPIO_OUT_1: track 0.00 -> 49.4 mm
- net 485_CONTROL: track 0.00 -> 48.1 mm
- net GPIO_OUT_2: track 0.00 -> 46.3 mm
- net GPIO_OUT_3: track 0.00 -> 43.4 mm
- net TXD1: track 0.00 -> 41.4 mm
- net GPIO_OUT_4: track 0.00 -> 40.5 mm
- net GPIO_OUT_5: track 0.00 -> 37.7 mm
- net CAN_RX: track 0.00 -> 36.7 mm
- net ADC_RST: track 0.00 -> 36.1 mm, vias 0 -> 1
- net MISO: track 0.00 -> 36.1 mm
- net RXD1: track 0.00 -> 35.8 mm
- net GPIO_OUT_6: track 0.00 -> 34.6 mm
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- added copper zone on F.Cu, net +3.3V
- added copper zone on F.Cu, net BUCK_OUT
- added copper zone on F.Cu, net GND
- added copper zone on F.Cu, net PWR
- added copper zone on F.Cu, net V IN
Other:
- board outline added: 57.1 x 57.1 mm
