File: Constellation STAR ITC V1.0/Constellation STAR ITC V1.0.kicad_pcb (KiCad board)
At the start: 2 copper layers, 57.1 x 63.5 mm, 22 parts, among them IC1 TLV76033DBZR, J1 SIGNAL_OUT, J2 SIGNAL_OUT, J3 PWR IN, J4 PWR IN, J5 HALL_1, J6 PT_1

Commit message: GERBS MADE
Parts:
- D1: value RED -> GREEN
- R1: value R -> 470
- R2: value R -> 75
Changed lines of the file:
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@@
 			(plot_on_all_layers_selection 0x0000000_00000000)
 			(disableapertmacros no)
-			(usegerberextensions no)
-			(usegerberattributes yes)
-			(usegerberadvancedattributes yes)
-			(creategerberjobfile yes)
+			(usegerberextensions yes)
+			(usegerberattributes no)
+			(usegerberadvancedattributes no)
+			(creategerberjobfile no)
 			(dashed_line_dash_ratio 12.000000)
 			(dashed_line_gap_ratio 3.000000)
@@
 			(psa4output no)
 			(plotreference yes)
-			(plotvalue yes)
+			(plotvalue no)
 			(plotfptext yes)
 			(plotinvisibletext no)
 			(sketchpadsonfab no)
-			(subtractmaskfromsilk no)
+			(subtractmaskfromsilk yes)
 			(outputformat 1)
 			(mirror no)
-			(drillshape 1)
+			(drillshape 0)
 			(scaleselection 1)
-			(outputdirectory "")
+			(outputdirectory "Gerbs/")
 		)
 	)
@@
 			)
 		)
-		(property "Value" "R"
+		(property "Value" "470"
 			(at 0 1.65 90)
 			(layer "F.Fab")
@@
 			)
 		)
-		(property "Value" "R"
+		(property "Value" "75"
 			(at 0 1.65 0)
 			(layer "F.Fab")
@@
 			)
 		)
-		(property "Value" "RED"
+		(property "Value" "GREEN"
 			(at 0 1.65 90)
 			(layer "F.Fab")
