File: Constellation STAR LAF V1.0/Constellation STAR LAF V1.0.kicad_sch (KiCad schematic)
At the start: 15 parts, among them IC1 TLV76033DBZR, J1 SIGNAL_OUT, J2 PWR IN, J3 HALL_1, J4 HALL_2, J5 PT_1

Commit message: GERBS MADE
Parts:
- D1: value RED -> GREEN
- R1: value R -> 470
- R2: value R -> 75
Changed lines of the file:
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@@
 	(text "PWR BUS LED"
 		(exclude_from_sim no)
-		(at 197.612 67.31 0)
+		(at 197.866 55.118 0)
 		(effects
 			(font
@@
 	(text "3.3V LED"
 		(exclude_from_sim no)
-		(at 196.85 55.118 0)
+		(at 195.326 67.056 0)
 		(effects
 			(font
@@
 			)
 		)
-		(property "Value" "RED"
+		(property "Value" "GREEN"
 			(at 184.404 52.578 0)
 			(effects
@@
 			)
 		)
-		(property "Value" "R"
+		(property "Value" "75"
 			(at 170.18 65.278 90)
 			(effects
@@
 			)
 		)
-		(property "Value" "R"
+		(property "Value" "470"
 			(at 170.18 53.848 90)
 			(effects
