File: Constellation STAR UAF V1.0/Constellation STAR UAF V1.0.kicad_sch (KiCad schematic)
At the start: 17 parts, among them IC1 TLV76033DBZR, J1 SIGNAL_OUT, J2 SIGNAL_OUT, J3 PWR IN, J4 PWR IN, J5 HALL_1, J6 PT_1, J7 PT_2

Commit message: GERBS MADE
Parts:
- D1: value RED -> GREEN
- R1: value R -> 470
- R2: value R -> 75
Changed lines of the file:
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@@
 	(text "PWR BUS LED"
 		(exclude_from_sim no)
-		(at 197.612 67.31 0)
+		(at 197.612 55.118 0)
 		(effects
 			(font
@@
 	(text "3.3V LED"
 		(exclude_from_sim no)
-		(at 196.85 55.118 0)
+		(at 196.85 67.31 0)
 		(effects
 			(font
@@
 			)
 		)
-		(property "Value" "RED"
+		(property "Value" "GREEN"
 			(at 184.404 52.578 0)
 			(effects
@@
 			)
 		)
-		(property "Value" "R"
+		(property "Value" "75"
 			(at 170.18 65.278 90)
 			(effects
@@
 			)
 		)
-		(property "Value" "R"
+		(property "Value" "470"
 			(at 170.18 53.848 90)
 			(effects
