File: Constellation Stack V1.2/Constellation Stack V1.2.kicad_pcb (KiCad board)
At the start: 4 copper layers, 57.1 x 50.8 mm, 97 parts, among them J1 PWR_IN, J2 USB_C_Receptacle_USB2.0, J3 RS485 Out, J4 PT_IN, J5 GPIO_OUT, J6 CAN_TERMINAL, Q1 MBT2222ADW1T1, SW1 RESET, SW2 SW_SPST, SW3 GPIO_0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

Commit message: AAAAa
Parts:
- removed C5: 1uF, Capacitor_SMD:C_0603_1608Metric
- moved TP18 0.89 mm to (56.6, 57.3)
Connections:
- U2 pad 5: +5V -> unconnected-(U2-VREF-Pad5)
Routing:
- net GND: track 69.8 -> 68.3 mm, vias 58 -> 57
- net CAN_RX: track 24.7 -> 23.4 mm
- net +5V: track 59.1 -> 58.2 mm
