File: Constellation Stack V1.2/Constellation Stack V1.2.kicad_sch (KiCad schematic)
At the start: 95 parts, among them J1 PWR_IN, J2 USB_C_Receptacle_USB2.0, J3 RS485 Out, J4 PT_IN, J5 GPIO_OUT, J6 CAN_TERMINAL, Q1 MBT2222ADW1T1, SW1 RESET, SW2 SW_SPST, SW3 GPIO_0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

Commit message: Ahhhahahaha
Connections:
- net RXD0: now also U1.31 (TXD0); no longer U1.30 (RXD0)
- net TXD0: now also U1.30 (RXD0); no longer U1.31 (TXD0)
Other:
- note added: "Is reversed due to UART requirements"

Commit message: AAAAa
Parts:
- removed C5: 1uF, Capacitor_SMD:C_0603_1608Metric, symbol Device:C
- R7: value 52.3k -> 68k
Connections:
- net +5V: no longer U2.5 (VREF)
- no-connect marks 22 -> 23
Other:
- note added: "~6.25V OUT CONFIG"
- note removed: "5V OUT CONFIG"
