File: Constellation Saddle V1.0/Constellation Saddle V1.0.kicad_pcb (KiCad board)
At the start: 2 copper layers, 95.2 x 95.2 mm, 16 parts, among them J1 PWR, J10 2601-1102, J2 2601-1102, J3 PT_IN, J4 SIGNAL_OUT, J5 CAN_TERMINAL, J6 2601-1102, J7 RS485 Out, J8 GPIO/ESP_ADC OUT, J9 2601-1103

Commit message: Saddle
Parts:
- added J9: 2601-1103, 2601_1103:CONN3_2601-1103_WAG, F.Cu at (88.1, 56.6)
- added J9: 2601-1103, 2601_1103:CONN3_2601-1103_WAG, F.Cu at (88.1, 70.4)
- added LS1: SMT-1127-S-R, SMT-1127-S-R:XDCR_SMT-1127-S-R, F.Cu at (92.1, 39.1)
Connections:
- J3 pad 1: AN_IN_3 -> HE_TANK
- J3 pad 2: AN_IN_2 -> O_TANK
- J3 pad 3: AN_IN_1 -> F_TANK
- J3 pad 4: AN_IN_0 -> ENG_CHAMBER
- J8 pad 10: ESP_32_ADC_IN_5 -> ESP_32_ADC_IN_2
- J8 pad 11: ESP_32_ADC_IN_4 -> ESP_32_ADC_IN_3
- J8 pad 12: ESP_32_ADC_IN_3 -> ESP_32_ADC_IN_4
- J8 pad 13: ESP_32_ADC_IN_2 -> ESP_32_ADC_IN_5
- J8 pad 2: GPIO_OUT_1 -> MOV
- J8 pad 3: GPIO_OUT_2 -> MFV
- J8 pad 4: GPIO_OUT_3 -> F_VENT
- J8 pad 5: GPIO_OUT_4 -> O_VENT
- J8 pad 6: GPIO_OUT_5 -> BUZZER
Routing:
- net MOV: track 0.00 -> 113.3 mm, vias 0 -> 1
- net MFV: track 0.00 -> 108.7 mm, vias 0 -> 1
- net F_VENT: track 0.00 -> 96.5 mm, vias 0 -> 1
- net O_VENT: track 0.00 -> 92.4 mm, vias 0 -> 1
- net PWR: track 0.00 -> 70.6 mm
- net BUZZER: track 0.00 -> 16.4 mm
- net O_TANK: track 6.61 -> 12.9 mm
- net F_TANK: track 7.42 -> 13.6 mm
- net ENG_CHAMBER: track 14.9 -> 20.6 mm
- net HE_TANK: track 9.08 -> 14.8 mm
- net GND: track 0.00 -> 1.27 mm, vias 0 -> 1
Other:
- board text added: "CAN H"
- board text added: "CAN L"

Commit message: Kicad
Parts:
- removed the J9 at (88.1, 56.6)
- removed the J9 at (88.1, 70.4)
- added G***: LOGO, LOGO, F.Cu at (43.8, 77.3)
- added G***: LOGO, LOGO, F.Cu at (54.6, 86.2)
- added J11: TC_AMP_1, Connector_PinSocket_2.54mm:PinSocket_1x04_P2.54mm_Vertical, F.Cu at (96.5, 48.9)
- added J12: TC_AMP_2, Connector_PinSocket_2.54mm:PinSocket_1x04_P2.54mm_Vertical, F.Cu at (96.5, 66.7)
- added J13: TC_AMP_3, Connector_PinSocket_2.54mm:PinSocket_1x04_P2.54mm_Vertical, F.Cu at (66.7, 96.5)
- added J14: TC_AMP_4, Connector_PinSocket_2.54mm:PinSocket_1x04_P2.54mm_Vertical, F.Cu at (48.9, 96.5)
- moved G*** 14.5 mm to (62.7, 77.8)
- moved G*** 10.2 mm to (52.4, 76.4)
- moved LS1 3.27 mm to (88.8, 39.2)
- moved J4 0.18 mm to (20.8, 47.4)
Connections:
- J8 pad 10: ESP_32_ADC_IN_2 -> TC_2
- J8 pad 11: ESP_32_ADC_IN_3 -> TC_3
- J8 pad 12: ESP_32_ADC_IN_4 -> TC_4
- J8 pad 9: ESP_32_ADC_IN_1 -> TC_1
Routing:
- net +3.3V: track 0.00 -> 128.1 mm
- net TC_4: track 0.00 -> 48.1 mm
- net TC_3: track 0.00 -> 42.7 mm
- net TC_1: track 0.00 -> 20.5 mm
- net TC_2: track 0.00 -> 18.9 mm
- net CAN_L: track 0.00 -> 17.5 mm
- net CAN_H: track 0.00 -> 12.7 mm
- net A: track 0.00 -> 12.7 mm
- net B: track 0.00 -> 12.3 mm
- net BUZZER: track 16.4 -> 14.2 mm
- net MFV: track 108.7 -> 109.2 mm
Other:
- board text added: "+"
- board text added: "3.3V"
- board text added: "A"
- board text added: "AN_1"
- board text added: "AN_2"
- board text added: "AN_3"
- board text added: "AN_4"
- board text added: "B"
- board text added: "BLK"
- board text added: "BLU"
- board text added: "BRN"
- board text added: "CAN BUS"
- board text added: "GND"
- board text added: "GRN"
- board text added: "ORG"
- board text added: "PWR IN"
- board text added: "PWR OUT"
- board text added: "RED"
- board text added: "RS-485"
- board text added: "TO STAR BOARDS"
- board text added: "WHT"
- board text added: "YLW"
