File: Constellation Stack V3.0/Constellation Stack V3.0.kicad_sch (KiCad schematic)
At the start: 85 parts, among them J1 PWR, J2 PROG SOCKET, J3 PT_IN, J5 CAN_TERMINAL, J7 RS485 Out, J8 GPIO/ESP_ADC OUT, Q2 DMP3099L, SW1 RESET, SW2 GPIO_0, SW3 SW_SPST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

Commit message: 3.0 work
Connections:
- net +3.3V: now also U6.11 (VDDIO), U6.3 (VDD)
- net GND: now also U6.2 (NC), U6.4 (GNDA), U6.6 (GNDIO), U6.7 (PS)
- net VSPI_CLK: now also U6.8 (SCL/SCK)
- net VSPI_MISO: now also U6.10 (SDO2), U6.15 (SDO1)
- net VSPI_MOSI: now also U6.9 (SDA/SDI)
- net INT2_ACCEL: now reaches U6.1 (INT2)
- net INT3_GYRO: now reaches U6.12 (INT3)
- net INT4_GYRO: now reaches U6.13 (INT4)
- net ACCEL_CS: now reaches U6.14 (CSB1)
- net INT1_ACCEL: now reaches U6.16 (INT1)
- net GYRO_CS: now reaches U6.5 (CSB2)
Other:
- moved on the sheet: U6

Commit message: 3.0 stack
Parts:
- removed C22: 1uF, Capacitor_SMD:C_0603_1608Metric, symbol Device:C
- removed C23: 47nf, Capacitor_SMD:C_0603_1608Metric, symbol Device:C_Small
- removed J5: CAN_TERMINAL, Connector_PinSocket_2.54mm:PinSocket_1x02_P2.54mm_Vertical, symbol Connector:Conn_01x02_Socket
- removed R18, R19: 60, Resistor_SMD:R_0805_2012Metric, symbol Device:R_Small
- removed SW3: SW_SPST, Jumper:SolderJumper-2_P1.3mm_Open_RoundedPad1.0x1.5mm, symbol Switch:SW_SPST
- removed TP17, TP18, TP19, TP20: TestPoint, TestPoint:TestPoint_Loop_D2.60mm_Drill1.6mm_Beaded, symbol Connector:TestPoint
- removed U4: ESP32-PICO-MINI-02U-N8R2, ESP32-PICO-MINI-02U:MODULE_ESP32-PICO-MINI-02U-N8R2, symbol ESP32-PICO-MINI-02U:ESP32-PICO-MINI-02U-N8R2
- removed U9: TJA1050T_CM_118, Package_SO:SOIC-8_3.9x4.9mm_P1.27mm, symbol TJA1050T:TJA1050T_CM_118
- added C11, C12, C15, C16: 100nF, Capacitor_SMD:C_0603_1608Metric, symbol Device:C
- added U4: BMP390, BMP390:10LGA_2X2X0p75_BOS, symbol BMP390:BMP390
- SW1, SW2: footprint PTS636SM50JSMTR LFS:SW_PTS636_CNK -> pt36:SW_PTS636_CNK
- U6: footprint BMI088:PQFN50P450X300X100-16N -> bmi088:BMI088
Connections:
- net +3.3V: now also C11.1, C12.1, C15.1, C16.1, U4.1 (VDDIO), U4.10 (VDD)
- net GND: now also C11.2, C12.2, C15.2, C16.2, U4.3 (VSS), U4.8 (VSS), U4.9 (VSS)
- net RXD0: now also J2.2 (Pin_2); no longer J2.3 (Pin_3)
- net TXD0: now also J2.3 (Pin_3); no longer J2.2 (Pin_2)
- net VSPI_CLK: now also U4.2 (SCK)
- net VSPI_MISO: now also U4.5 (SDO)
- net VSPI_MOSI: now also U4.4 (SDI)
- net INT1_ACCEL: no longer names the net of U6.16 (INT1)
- net INT2_ACCEL: no longer names the net of U6.1 (INT2)
- net INT3_GYRO: no longer names the net of U6.12 (INT3)
- net INT4_GYRO: no longer names the net of U6.13 (INT4)
- new net BARO_CS: U4.6 (CSB)
- no-connect marks 6 -> 10
Other:
- note added: "BMI 088 Interial Measurement Unit (IMU)"
- note added: "BMI 390 Barometer"
- note added: "VDD/VDDIO CAPS"
- note removed: "CAN BUS"
- note removed: "TJA1050 CAN Transceiver"
- moved on the sheet: U5, U6

Commit message: 3.0 work
Parts:
- removed J7: RS485 Out, Connector_PinSocket_2.54mm:PinSocket_1x03_P2.54mm_Vertical, symbol Connector:Conn_01x03_Socket
- J1: footprint Connector_PinSocket_2.54mm:PinSocket_1x02_P2.54mm_Vertical -> Connector_PinSocket_2.54mm:PinSocket_1x08_P2.54mm_Vertical; symbol Connector:Conn_01x02_Socket -> Connector:Conn_01x08_Socket
Connections:
- net A: now also J1.6 (Pin_6)
- net B: now also J1.7 (Pin_7)
- net GND: now also J1.8 (Pin_8)
- new net BATT_PWR_SENSE: J1.4 (Pin_4)
- new net EXT_PWR_SENSE: J1.3 (Pin_3)
- no-connect marks 10 -> 11
Other:
- note added: "PIN SOCKET IN/OUT"
- note removed: "PIN SOCKET OUT"
- moved on the sheet: J3

Commit message: HAHAHAH
Parts:
- added D7: D, symbol Device:D
- added U9: MIC5504-3.3YM5, Package_TO_SOT_SMD:SOT-23-5, symbol Regulator_Linear:MIC5504-3.3YM5
- J3: value PT_IN -> ADC_IN
Connections:
- net +3.3V: now also U9.5 (VOUT)
- net +5V: now also D7.1 (K)
- net BUCK_OUT: no longer J2.1 (Pin_1)
- net GND: now also U9.2 (GND)
- net RXD0: now also J2.3 (Pin_3); no longer J2.2 (Pin_2)
- net TXD0: now also J2.2 (Pin_2); no longer J2.3 (Pin_3)
- new net USB_PWR: D7.2 (A), J2.1 (Pin_1), U9.1 (VIN), U9.3 (EN)
Other:
- note added: "ADC OUT"
- note added: "PWR/RS485 OUT"
- note removed: "PROGRAMING CONNECTOR"
- moved on the sheet: J1, J2, J3, J8

Commit message: HEHEHHA
Connections:
- net 485_CONTROL: now also U5.10 (IO25)
- net ACCEL_CS: now also U5.14 (IO12)
- net ADC_CS: now also U5.26 (IO4)
- net ADC_RST: now also U5.12 (IO27)
- net BARO_CS: now also U5.13 (IO14)
- net FLASH_CS: now also U5.11 (IO26)
- net GYRO_CS: now also U5.16 (IO13)
Other:
- moved on the sheet: D7, U9

Commit message: Aaawwww yeah 90% done
Parts:
- removed D7: D, symbol Device:D
- added C22: 10uF, Capacitor_SMD:C_0603_1608Metric, symbol Device:C
- added C23: 0.1uF, Capacitor_SMD:C_0603_1608Metric, symbol Device:C
- added CR1: LSM115JE3/TR13, LSM115JE3_TR13:DO-214BA_MCH-L, symbol LSM115JE3_TR13:LSM115JE3_TR13
Connections:
- net +3.3V: now also C23.1
- net +5V: now also CR1.1
- net BATT_PWR_SENSE: now also U5.7 (IO35)
- net EXT_PWR_SENSE: now also U5.6 (IO34)
- net GND: now also C22.1, C23.2
- net LED_OUT: now also U5.8 (IO32)
- net USB_PWR: now also C22.2, CR1.2
Other:
- note added: "HIGH DURING BOOT"
- note added: "IN ONLY"
- note added: "LOW DURING BOOT"
- note added: "USB POWER CIRCUITRY"
- note removed: "Revert back bc/ off-board programmer"
- moved on the sheet: U9

Commit message: Changes
Parts:
- added J4: MSD-1-A, MSD_1_A:CUI_MSD-1-A, symbol MSD_1_A:MSD-1-A
- added TP12, TP13, TP14, TP15: TestPoint, TestPoint:TestPoint_Pad_D1.5mm, symbol Connector:TestPoint
- J8: footprint Connector_PinSocket_2.54mm:PinSocket_1x14_P2.54mm_Vertical -> Connector_PinSocket_2.54mm:PinSocket_1x08_P2.54mm_Vertical; symbol Connector:Conn_01x14_Socket -> Connector:Conn_01x08_Socket
- TP1, TP2, TP21, TP22, TP3, TP4, TP5, TP6, TP7, TP8, TP9: footprint TestPoint:TestPoint_Loop_D2.60mm_Drill1.6mm_Beaded -> TestPoint:TestPoint_Pad_D1.5mm
- TP10: renamed from TP11; footprint TestPoint:TestPoint_Loop_D2.60mm_Drill1.6mm_Beaded -> TestPoint:TestPoint_Pad_D1.5mm
- TP11: renamed from TP10; footprint TestPoint:TestPoint_Loop_D2.60mm_Drill1.6mm_Beaded -> TestPoint:TestPoint_Pad_D1.5mm
- TP16: renamed from TP12; footprint TestPoint:TestPoint_Loop_D2.60mm_Drill1.6mm_Beaded -> TestPoint:TestPoint_Pad_D1.5mm
- TP17: renamed from TP13; footprint TestPoint:TestPoint_Loop_D2.60mm_Drill1.6mm_Beaded -> TestPoint:TestPoint_Pad_D1.5mm
- TP18: renamed from TP14; footprint TestPoint:TestPoint_Loop_D2.60mm_Drill1.6mm_Beaded -> TestPoint:TestPoint_Pad_D1.5mm
- TP19: renamed from TP15; footprint TestPoint:TestPoint_Loop_D2.60mm_Drill1.6mm_Beaded -> TestPoint:TestPoint_Pad_D1.5mm
- TP20: renamed from TP16; footprint TestPoint:TestPoint_Loop_D2.60mm_Drill1.6mm_Beaded -> TestPoint:TestPoint_Pad_D1.5mm
Connections:
- net GPIO_OUT_6 is gone; now on net GPIO_OUT_5: J8.7 (Pin_7)
- net +3.3V: now also J8.2 (Pin_2), J4.4 (VDD); no longer J8.8 (Pin_8)
- net 485_CONTROL: now also U5.9 (IO33); no longer U5.10 (IO25)
- net ACCEL_CS: now also U5.13 (IO14), TP13.1; no longer U5.14 (IO12)
- net ADC_RST: now also U5.11 (IO26); no longer U5.12 (IO27)
- net BARO_CS: now also U5.12 (IO27), TP15.1; no longer U5.13 (IO14)
- net FLASH_CS: now also U5.10 (IO25); no longer U5.11 (IO26)
- net GND: now also J8.8 (Pin_8), J4.6 (VSS), J4.G1 (COVER_GND), J4.G2 (COVER_GND__1), J4.G3 (COVER_GND__2), J4.G4 (COVER_GND__3); no longer J8.14 (Pin_14)
- net GPIO_OUT_1: now also J8.3 (Pin_3), U5.14 (IO12); no longer J8.2 (Pin_2)
- net GPIO_OUT_2: now also J8.4 (Pin_4), U5.23 (IO15); no longer J8.3 (Pin_3)
- net GPIO_OUT_3: now also J8.5 (Pin_5), U5.24 (IO2); no longer J8.4 (Pin_4)
- net GPIO_OUT_4: now also J8.6 (Pin_6), U5.29 (IO5); no longer J8.5 (Pin_5)
- net GPIO_OUT_5: now also U5.33 (IO21); no longer J8.6 (Pin_6)
- net GYRO_CS: now also TP14.1
- net VSPI_CLK: now also J4.5 (CLK)
- net VSPI_MISO: now also J4.7 (DAT0)
- net VSPI_MOSI: now also J4.3 (CMD)
- net SD_CARD_CS: now reaches U5.36 (IO22)
- net SD_CARD_CS: now also J4.2 (CD/DAT3), TP12.1
- removed net ESP_32_ADC_IN_1: J8.9 (Pin_9)
- removed net ESP_32_ADC_IN_2: J8.10 (Pin_10)
- removed net ESP_32_ADC_IN_3: J8.11 (Pin_11)
- removed net ESP_32_ADC_IN_4: J8.12 (Pin_12)
- removed net ESP_32_ADC_IN_5: J8.13 (Pin_13)
- no-connect marks 11 -> 14
Other:
- note added: "GPIO/ESP_ADC OUT"
- note added: "MSD-1-A Spring SD Card Holder"
- note added: "SPI"
- note removed: "SPI/ADC"
- moved on the sheet: C18, C24, C8, C9, D6, J1, R17, R20, TP1, TP10, TP11, TP16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

Commit message: All the 3.0 files
Parts:
- TP16, TP17, TP19, TP20, TP6, TP7, TP8: footprint TestPoint:TestPoint_Pad_D1.5mm -> TestPoint:TestPoint_Loop_D2.60mm_Drill1.6mm_Beaded
Connections:
- net SD_CARD_DETECT: now reaches J4.CD
- net SD_CARD_DETECT: now also U5.33 (IO21)
- net GPIO_OUT_5: no longer names the net of J8.7 (Pin_7)
- net GPIO_OUT_5: no longer U5.33 (IO21)
Changed lines of the file:
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@@
 	)
 	(no_connect
-		(at 375.285 188.595)
+		(at 407.67 215.9)
 	)
 	(no_connect
-		(at 132.715 204.47)
+		(at 375.285 188.595)
 	)
 	(no_connect
@@
 		)
 	)
+	(wire
+		(pts
+			(xy 130.81 204.47) (xy 132.715 204.47)
+		)
+		(stroke
+			(width 0)
+			(type default)
+		)
+	)
 	(polyline
 		(pts
@@
 		)
 	)
-	(global_label "GPIO_OUT_5"
-		(shape input)
-		(at 226.695 116.84 0)
-		(fields_autoplaced yes)
-		(effects
-			(font
-				(size 1.27 1.27)
-			)
-			(justify left)
-		)
-		(property "Intersheetrefs" "${INTERSHEET_REFS}"
-			(at 240.9288 116.84 0)
-			(effects
-				(font
-					(size 1.27 1.27)
-				)
-				(justify left)
-				(hide yes)
-			)
-		)
-	)
 	(global_label "RXD1"
 		(shape input)
@@
 		)
 	)
+	(global_label "SD_CARD_DETECT"
+		(shape input)
+		(at 226.695 116.84 0)
+		(fields_autoplaced yes)
+		(effects
+			(font
+				(size 1.27 1.27)
+			)
+			(justify left)
+		)
+		(property "Intersheetrefs" "${INTERSHEET_REFS}"
+			(at 245.7667 116.84 0)
+			(effects
+				(font
+					(size 1.27 1.27)
+				)
+				(justify left)
+				(hide yes)
+			)
+		)
+	)
 	(global_label "VSPI_MOSI"
 		(shape input)
@@
 		)
 	)
+	(global_label "SD_CARD_DETECT"
+		(shape input)
+		(at 130.81 204.47 180)
+		(fields_autoplaced yes)
+		(effects
+			(font
+				(size 1.27 1.27)
+			)
+			(justify right)
+		)
+		(property "Intersheetrefs" "${INTERSHEET_REFS}"
+			(at 111.7383 204.47 0)
+			(effects
+				(font
+					(size 1.27 1.27)
+				)
+				(justify right)
+				(hide yes)
+			)
+		)
+	)
 	(global_label "BUCK_OUT"
 		(shape input)
@@
 		)
 	)
-	(global_label "GPIO_OUT_5"
-		(shape input)
-		(at 407.67 215.9 180)
-		(fields_autoplaced yes)
-		(effects
-			(font
-				(size 1.27 1.27)
-			)
-			(justify right)
-		)
-		(property "Intersheetrefs" "${INTERSHEET_REFS}"
-			(at 393.4362 215.9 0)
-			(effects
-				(font
-					(size 1.27 1.27)
-				)
-				(justify right)
-				(hide yes)
-			)
-		)
-	)
 	(global_label "AN_IN_6"
 		(shape input)
@@
 			)
 		)
-		(property "Footprint" "TestPoint:TestPoint_Pad_D1.5mm"
+		(property "Footprint" "TestPoint:TestPoint_Loop_D2.60mm_Drill1.6mm_Beaded"
 			(at 35.56 109.22 0)
 			(effects
@@
 			)
 		)
-		(property "Footprint" "TestPoint:TestPoint_Pad_D1.5mm"
+		(property "Footprint" "TestPoint:TestPoint_Loop_D2.60mm_Drill1.6mm_Beaded"
 			(at 72.39 109.22 0)
 			(effects
@@
 			)
 		)
-		(property "Footprint" "TestPoint:TestPoint_Pad_D1.5mm"
+		(property "Footprint" "TestPoint:TestPoint_Loop_D2.60mm_Drill1.6mm_Beaded"
 			(at 64.77 109.22 0)
 			(effects
@@
 			)
 		)
-		(property "Footprint" "TestPoint:TestPoint_Pad_D1.5mm"
+		(property "Footprint" "TestPoint:TestPoint_Loop_D2.60mm_Drill1.6mm_Beaded"
 			(at 38.1 109.22 0)
 			(effects
@@
 			)
 		)
-		(property "Footprint" "TestPoint:TestPoint_Pad_D1.5mm"
+		(property "Footprint" "TestPoint:TestPoint_Loop_D2.60mm_Drill1.6mm_Beaded"
 			(at 62.23 109.22 0)
 			(effects
@@
 			)
 		)
-		(property "Footprint" "TestPoint:TestPoint_Pad_D1.5mm"
+		(property "Footprint" "TestPoint:TestPoint_Loop_D2.60mm_Drill1.6mm_Beaded"
 			(at 33.02 109.22 0)
 			(effects
@@
 			)
 		)
-		(property "Footprint" "TestPoint:TestPoint_Pad_D1.5mm"
+		(property "Footprint" "TestPoint:TestPoint_Loop_D2.60mm_Drill1.6mm_Beaded"
 			(at 69.85 109.22 0)
 			(effects
