File: Constellation Stack V3.0/Constellation Stack V3.0.kicad_pcb (KiCad board)
At the start: 4 copper layers, 57.1 x 57.1 mm, 87 parts, among them J1 PWR, J2 PROG SOCKET, J3 PT_IN, J5 CAN_TERMINAL, J7 RS485 Out, J8 GPIO/ESP_ADC OUT, Q2 DMP3099L, SW1 RESET, SW2 GPIO_0, SW3 SW_SPST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

Commit message: 3.0 stack
Parts:
- removed C22: 1uF, Capacitor_SMD:C_0603_1608Metric
- removed C23: 47nf, Capacitor_SMD:C_0603_1608Metric
- removed J5: CAN_TERMINAL, Connector_PinSocket_2.54mm:PinSocket_1x02_P2.54mm_Vertical
- removed R18, R19: 60, Resistor_SMD:R_0805_2012Metric
- removed SW3: SW_SPST, Jumper:SolderJumper-2_P1.3mm_Open_RoundedPad1.0x1.5mm
- removed TP17, TP18, TP19, TP20: TestPoint, TestPoint:TestPoint_Loop_D2.60mm_Drill1.6mm_Beaded
- removed U9: TJA1050T_CM_118, Package_SO:SOIC-8_3.9x4.9mm_P1.27mm
- added C11: 100nF, Capacitor_SMD:C_0603_1608Metric, F.Cu at (86.2, 19.8)
- added C12: 100nF, Capacitor_SMD:C_0603_1608Metric, F.Cu at (86.2, 22.3)
- added C15: 100nF, Capacitor_SMD:C_0603_1608Metric, F.Cu at (86.2, 24.8)
- added C16: 100nF, Capacitor_SMD:C_0603_1608Metric, F.Cu at (86.2, 27.3)
- added U4: BMP390, BMP390:10LGA_2X2X0p75_BOS, F.Cu at (72.4, 62.6)
- added U6: BMI088, bmi088:BMI088, F.Cu at (54.0, 54.0)
- SW1, SW2: footprint PTS636SM50JSMTR LFS:SW_PTS636_CNK -> pt36:SW_PTS636_CNK
- TP21, TP22: moved to B.Cu
- moved TP21 40.5 mm to (48.6, 53.3), turned to 180 degrees
- moved TP22 40.5 mm to (48.6, 58.4), turned to 180 degrees
- moved J2 21.8 mm to (40.1, 71.5)
- moved C10 6.35 mm to (93.6, 34.6)
- moved R11 6.35 mm to (90.6, 34.6)
- moved SW1 6.35 mm to (92.0, 39.4)
- moved SW2 6.35 mm to (96.5, 39.5)
Connections:
- J2 pad 2: TXD0 -> RXD0
- J2 pad 3: RXD0 -> TXD0
Routing:
- net CAN_L: track 18.6 -> 0.00 mm
- net CAN_H: track 14.5 -> 0.00 mm, vias 1 -> 0
- net CAN_RX: track 14.5 -> 0.00 mm
- net CAN_TX: track 5.73 -> 0.00 mm
- net GND: track 43.6 -> 40.0 mm, vias 49 -> 45
- net Net-(C23-Pad2): track 3.53 -> 0.00 mm
- net +5V: track 67.2 -> 64.5 mm, vias 3 -> 2
- net Net-(SW3-B): track 2.66 -> 0.00 mm, vias 1 -> 0
Other:
- board text removed: "i cant"

Commit message: 3.0 work
Parts:
- removed J7: RS485 Out, Connector_PinSocket_2.54mm:PinSocket_1x03_P2.54mm_Vertical
- J1: footprint Connector_PinSocket_2.54mm:PinSocket_1x02_P2.54mm_Vertical -> Connector_PinSocket_2.54mm:PinSocket_1x08_P2.54mm_Vertical
- moved G*** 65.5 mm to (35.7, 73.6)
- moved R11 47.3 mm to (67.8, 76.0), turned to 90 degrees
- moved C10 46.3 mm to (67.8, 73.0), turned to 90 degrees
- moved G*** 40.8 mm to (71.5, 63.9)
- moved SW1 40.1 mm to (72.6, 74.5), turned to 180 degrees
- moved D5 38.2 mm to (74.3, 70.2)
- moved R10 38.2 mm to (71.2, 70.2)
- moved TP21 35.3 mm to (16.4, 38.9)
- moved TP9 35.3 mm to (10.1, 41.5)
- moved TP11 35.3 mm to (10.8, 35.1)
- moved TP12 33.9 mm to (17.8, 31.8)
- moved TP13 33.8 mm to (14.8, 28.4)
- moved TP10 30.5 mm to (15.3, 51.4)
- moved TP22 29.0 mm to (21.1, 67.7)
- moved TP2 25.2 mm to (37.7, 28.3)
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Routing:
- net VSPI_MOSI: track 0.00 -> 79.1 mm, vias 0 -> 3
- net VSPI_MISO: track 0.00 -> 77.4 mm, vias 0 -> 2
- net VSPI_CLK: track 0.00 -> 66.5 mm, vias 0 -> 2
- net TXD1: track 0.00 -> 38.3 mm
- net RXD1: track 0.00 -> 29.5 mm
- net +5V: track 64.5 -> 79.2 mm
- net GND: track 40.0 -> 48.4 mm, vias 45 -> 51
- net +3.3V: track 9.43 -> 17.1 mm, vias 10 -> 14
- net B: track 15.0 -> 8.60 mm
- net A: track 12.2 -> 8.01 mm
- net 485_CONTROL: track 14.2 -> 18.2 mm

Commit message: HAHAHAH
Parts:
- J3: value PT_IN -> ADC_IN
- moved TP21 61.6 mm to (66.4, 74.9)
- moved SW2 46.6 mm to (54.4, 59.5), turned to 180 degrees
- moved TP13 38.5 mm to (50.2, 43.6)
- moved TP12 35.5 mm to (49.3, 48.2)
- moved TP3 33.8 mm to (40.0, 28.3)
- moved J2 32.9 mm to (27.9, 73.7), turned to 180 degrees
- moved TP22 28.0 mm to (47.9, 59.6)
- moved G*** 12.1 mm to (37.7, 61.6)
- moved J3 8.89 mm to (27.9, 57.1)
- moved C13 2.47 mm to (35.1, 56.6)
- moved C17 2.47 mm to (36.9, 56.8)
- moved C19 2.47 mm to (33.8, 42.4)
- moved C20 2.47 mm to (35.3, 44.9)
- moved U10 2.47 mm to (34.5, 51.2)
- moved C14 2.47 mm to (33.7, 46.5)
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Connections:
- J2 pad 2: RXD0 -> TXD0
- J2 pad 3: TXD0 -> RXD0
Routing:
- net RESET: track 2.91 -> 63.6 mm
- net GPIO_0: track 0.00 -> 60.5 mm
- net +5V: track 79.2 -> 44.6 mm
- net RXD0: track 0.00 -> 20.2 mm
- net TXD0: track 0.00 -> 19.7 mm
- net AN_IN_6: track 0.00 -> 14.7 mm, vias 0 -> 2
- net AN_IN_7: track 0.00 -> 12.3 mm, vias 0 -> 1
- net AN_IN_5: track 8.04 -> 0.00 mm
- net AN_IN_2: track 5.05 -> 10.9 mm, vias 0 -> 1
- net AN_IN_3: track 5.40 -> 10.9 mm, vias 0 -> 1
- net AN_IN_0: track 5.28 -> 10.5 mm
- net VSPI_CLK: track 66.5 -> 71.1 mm
- net VSPI_MISO: track 77.4 -> 81.1 mm
- net VSPI_MOSI: track 79.1 -> 82.3 mm
- net AN_IN_1: track 4.55 -> 7.53 mm
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
Commit message: HEHEHHA
Parts:
- moved C12 47.5 mm to (53.2, 56.5), turned to 180 degrees
- moved C11 45.3 mm to (53.6, 51.4)
- moved C15 36.9 mm to (67.6, 56.7)
- moved TP11 36.6 mm to (45.5, 46.5)
- moved C16 35.4 mm to (69.6, 58.6)
- moved TP9 35.3 mm to (42.2, 56.2)
- moved TP10 31.0 mm to (40.1, 32.8)
- moved TP12 3.91 mm to (51.5, 44.9)
- moved TP13 2.65 mm to (50.4, 40.9)
- moved TP14 2.38 mm to (57.7, 45.7)
- moved G*** 0.60 mm to (71.0, 64.2)
- moved SW2 0.53 mm to (53.9, 59.6)
Routing:
- net FLASH_CS: track 0.00 -> 58.5 mm, vias 0 -> 1
- net ADC_RST: track 0.00 -> 41.3 mm, vias 0 -> 2
- net +5V: track 44.6 -> 79.2 mm
- net 485_CONTROL: track 18.2 -> 43.2 mm, vias 0 -> 1
- net ADC_CS: track 0.00 -> 17.9 mm, vias 0 -> 1
- net ACCEL_CS: track 0.00 -> 17.4 mm, vias 0 -> 2
- net GYRO_CS: track 0.00 -> 13.7 mm, vias 0 -> 2
- net AN_IN_5: track 0.00 -> 10.2 mm
- net GND: track 48.3 -> 55.5 mm, vias 49 -> 53
- net +3.3V: track 17.6 -> 24.6 mm, vias 14 -> 16
- net VSPI_MISO: track 81.1 -> 87.4 mm
- net BARO_CS: track 0.00 -> 5.42 mm
- net A: track 8.01 -> 10.5 mm
- net B: track 8.60 -> 11.0 mm
- net VSPI_CLK: track 71.1 -> 73.0 mm
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
Commit message: Aaawwww yeah 90% done
Parts:
- added C22: 10uF, Capacitor_SMD:C_0603_1608Metric, F.Cu at (35.8, 73.9)
- added C23: 0.1uF, Capacitor_SMD:C_0603_1608Metric, F.Cu at (34.3, 79.7)
- added CR1: LSM115JE3/TR13, LSM115JE3_TR13:DO-214BA_MCH-L, F.Cu at (32.1, 71.5)
- added U9: MIC5504-3.3YM5, Package_TO_SOT_SMD:SOT-23-5, F.Cu at (34.1, 76.8)
- moved TP3 34.0 mm to (74.0, 27.6)
- moved TP10 11.2 mm to (46.2, 42.1)
- moved TP2 11.0 mm to (31.8, 38.6)
- moved G*** 1.35 mm to (38.1, 62.9)
- moved G*** 0.97 mm to (71.4, 63.4)
- moved TP21 0.65 mm to (66.3, 75.5)
Connections:
- J2 pad 1: BUCK_OUT -> USB_PWR
- U5 pad 10: unconnected-(U5-IO25-Pad10) -> 485_CONTROL
- U5 pad 11: unconnected-(U5-IO26-Pad11) -> FLASH_CS
- U5 pad 12: unconnected-(U5-IO27-Pad12) -> ADC_RST
- U5 pad 13: unconnected-(U5-IO14-Pad13) -> BARO_CS
- U5 pad 14: unconnected-(U5-IO12-Pad14) -> ACCEL_CS
- U5 pad 16: unconnected-(U5-IO13-Pad16) -> GYRO_CS
- U5 pad 26: unconnected-(U5-IO4-Pad26) -> ADC_CS
- U5 pad 6: unconnected-(U5-IO34-Pad6) -> EXT_PWR_SENSE
- U5 pad 7: unconnected-(U5-IO35-Pad7) -> BATT_PWR_SENSE
- U5 pad 8: unconnected-(U5-IO32-Pad8) -> LED_OUT
Routing:
- net EXT_PWR_SENSE: track 0.00 -> 52.5 mm, vias 0 -> 1
- net BATT_PWR_SENSE: track 0.00 -> 51.0 mm, vias 0 -> 1
- net +5V: track 79.2 -> 91.3 mm, vias 2 -> 4
- net USB_PWR: track 0.00 -> 11.9 mm
- net LED_OUT: track 0.00 -> 9.49 mm
- net TXD0: track 19.7 -> 24.7 mm
- net ACCEL_CS: track 17.4 -> 21.0 mm
- net 485_CONTROL: track 43.2 -> 46.7 mm
- net RXD0: track 20.2 -> 22.9 mm
- net +3.3V: track 24.6 -> 27.1 mm, vias 16 -> 17
- net BARO_CS: track 5.42 -> 7.93 mm
- net GND: track 55.5 -> 57.9 mm, vias 53 -> 56
- net GYRO_CS: track 13.7 -> 15.8 mm
- net ADC_RST: track 41.3 -> 43.1 mm
- net GPIO_0: track 60.0 -> 61.2 mm
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
Commit message: Changes
Parts:
- added G***: LOGO, LOGO, B.Cu at (37.1, 62.5)
- added J4: MSD-1-A, MSD_1_A:CUI_MSD-1-A, B.Cu at (40.8, 32.8)
- added TP17: TestPoint, TestPoint:TestPoint_Pad_D1.5mm, B.Cu at (50.9, 43.1)
- added TP18: TestPoint, TestPoint:TestPoint_Pad_D1.5mm, B.Cu at (57.7, 45.7)
- added TP19: TestPoint, TestPoint:TestPoint_Pad_D1.5mm, B.Cu at (57.1, 31.9)
- added TP20: TestPoint, TestPoint:TestPoint_Pad_D1.5mm, B.Cu at (54.6, 31.9)
- J2: moved to B.Cu
- J8: footprint Connector_PinSocket_2.54mm:PinSocket_1x14_P2.54mm_Vertical -> Connector_PinSocket_2.54mm:PinSocket_1x08_P2.54mm_Vertical
- TP1, TP10, TP11, TP12, TP13, TP14, TP15, TP16, TP2, TP21, TP22, TP3, TP4, TP5, TP6, TP7, TP8, TP9: footprint TestPoint:TestPoint_Loop_D2.60mm_Drill1.6mm_Beaded -> TestPoint:TestPoint_Pad_D1.5mm
- moved G*** 45.2 mm to (39.8, 31.0)
- moved TP2 44.3 mm to (74.8, 28.0), turned to 0 degrees
- moved G*** 35.4 mm to (73.3, 67.0)
- moved TP15 31.0 mm to (68.7, 61.0), turned to 0 degrees
- moved G*** 30.5 mm to (59.0, 48.6)
- moved TP13 18.6 mm to (53.0, 59.3), turned to 0 degrees
- moved TP14 15.3 mm to (55.2, 60.8), turned to 0 degrees
- moved TP16 13.2 mm to (52.6, 45.2), turned to 0 degrees
- moved TP12 8.08 mm to (48.1, 52.3), turned to 0 degrees
- moved J8 7.62 mm to (80.0, 44.5)
- moved TP10 4.20 mm to (44.9, 46.1), turned to 0 degrees
- moved C15 4.20 mm to (71.8, 57.4)
- moved U4 4.20 mm to (70.7, 59.7)
- moved C16 4.20 mm to (73.7, 59.2)
- moved TP21 3.90 mm to (69.7, 73.7), turned to 0 degrees
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Connections:
- J8 pad 2: GPIO_OUT_1 -> +3.3V
- J8 pad 3: GPIO_OUT_2 -> GPIO_OUT_1
- J8 pad 4: GPIO_OUT_3 -> GPIO_OUT_2
- J8 pad 5: GPIO_OUT_4 -> GPIO_OUT_3
- J8 pad 6: GPIO_OUT_5 -> GPIO_OUT_4
- J8 pad 7: GPIO_OUT_6 -> GPIO_OUT_5
- J8 pad 8: +3.3V -> GND
- TP10 pad 1: FLASH_CS -> ADC_RST
- TP11 pad 1: ADC_RST -> FLASH_CS
- TP12 pad 1: RXD1 -> SD_CARD_CS
- TP13 pad 1: TXD1 -> ACCEL_CS
- TP14 pad 1: 485_CONTROL -> GYRO_CS
- TP15 pad 1: A -> BARO_CS
- TP16 pad 1: B -> RXD1
- U5 pad 10: 485_CONTROL -> FLASH_CS
- U5 pad 11: FLASH_CS -> ADC_RST
- U5 pad 12: ADC_RST -> BARO_CS
- U5 pad 13: BARO_CS -> ACCEL_CS
- U5 pad 14: ACCEL_CS -> GPIO_OUT_1
- U5 pad 23: unconnected-(U5-IO15-Pad23) -> GPIO_OUT_2
- U5 pad 24: unconnected-(U5-IO2-Pad24) -> GPIO_OUT_3
- U5 pad 29: unconnected-(U5-IO5-Pad29) -> GPIO_OUT_4
- U5 pad 33: unconnected-(U5-IO21-Pad33) -> GPIO_OUT_5
- U5 pad 36: unconnected-(U5-IO22-Pad36) -> SD_CARD_CS
- U5 pad 9: unconnected-(U5-IO33-Pad9) -> 485_CONTROL
Routing:
- net GPIO_OUT_4: track 0.00 -> 48.3 mm, vias 0 -> 1
- net SD_CARD_CS: track 0.00 -> 45.9 mm, vias 0 -> 3
- net GPIO_OUT_5: track 0.00 -> 44.8 mm, vias 0 -> 1
- net GPIO_OUT_3: track 0.00 -> 38.2 mm, vias 0 -> 1
- net GPIO_OUT_2: track 0.00 -> 36.6 mm, vias 0 -> 1
- net GPIO_OUT_1: track 0.00 -> 26.4 mm, vias 0 -> 1
- net VSPI_CLK: track 73.0 -> 83.0 mm, vias 2 -> 4
- net VSPI_MOSI: track 81.3 -> 91.1 mm, vias 3 -> 5
- net VSPI_MISO: track 87.4 -> 96.7 mm, vias 2 -> 4
- net RESET: track 64.4 -> 71.7 mm
- net GND: track 57.9 -> 64.8 mm, vias 56 -> 63
- net BARO_CS: track 7.93 -> 13.5 mm, vias 0 -> 2
- net +5V: track 91.3 -> 95.5 mm, vias 4 -> 6
- net GPIO_0: track 61.2 -> 64.1 mm, vias 0 -> 1
- net B: track 11.0 -> 9.52 mm, vias 0 -> 1
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Other:
- board text added: "0"
- board text added: "1"
- board text added: "2"
- board text added: "3"
- board text added: "3.3V"
- board text added: "3.3V LED"
- board text added: "4"
- board text added: "5"
- board text added: "5V"
- board text added: "6"
- board text added: "7"
- board text added: "A"
- board text added: "ACCEL_CS"
- board text added: "B"
- board text added: "BARO_CS"
- board text added: "BATT"
- board text added: "BUCK_OUT"
- board text added: "CONSTEllaTION STaCK V3.0"
- board text added: "EN"
- board text added: "EXT"
- board text added: "GPIO_0"
- board text added: "GYRO_CS"
- board text added: "G_1"
- board text added: "G_2"
- board text added: "G_3"
- board text added: "G_4"
- board text added: "G_5"
- board text added: "IO_0"
- board text added: "PWR"
- board text added: "RESET"
- board text added: "RX"
- board text added: "SD_CARD_CS"
- board text added: "TX"
- board text added: "hey put that back!"
- board text added: "le game"
- board text removed: "3.3V PWR"
- board text removed: "CAN TERM RES"
- board text removed: "CAN_H"
- board text removed: "CAN_L"
- board text removed: "CAN_RX"
- board text removed: "CAN_TX"

Commit message: All the 3.0 files
Parts:
- TP16, TP17, TP19, TP20, TP6, TP7, TP8: footprint TestPoint:TestPoint_Pad_D1.5mm -> TestPoint:TestPoint_Loop_D2.60mm_Drill1.6mm_Beaded
- moved C22 9.19 mm to (35.8, 64.7)
- moved C23 9.19 mm to (34.2, 70.5)
- moved CR1 9.19 mm to (32.1, 62.3)
- moved U9 9.19 mm to (34.1, 67.6)
- moved G*** 8.66 mm to (72.7, 75.7)
- moved D4 5.41 mm to (33.5, 33.2), turned to -90 degrees
- moved R3 4.78 mm to (80.1, 37.2), turned to 90 degrees
- moved C10 4.66 mm to (71.5, 67.9)
- moved D5 4.66 mm to (79.0, 66.3)
- moved R10 4.66 mm to (75.9, 66.3)
- moved R11 4.66 mm to (71.5, 71.0)
- moved SW1 4.66 mm to (76.4, 69.5)
- moved C16 3.67 mm to (75.8, 62.2)
- moved C15 3.67 mm to (73.9, 60.4)
- moved U4 3.67 mm to (72.8, 62.7)
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Connections:
- J4 pad CD: unconnected-(J4-PadCD) -> SD_CARD_DETECT
- U5 pad 33: GPIO_OUT_5 -> SD_CARD_DETECT
Routing:
- net SD_CARD_DETECT: track 0.00 -> 53.0 mm, vias 0 -> 1
- net GPIO_OUT_5: track 44.8 -> 0.00 mm, vias 1 -> 0
- net +5V: track 95.5 -> 86.0 mm
- net USB_PWR: track 12.0 -> 20.4 mm, vias 0 -> 2
- net RESET: track 71.7 -> 79.8 mm
- net V IN: track 0.00 -> 8.05 mm
- net VSPI_MISO: track 96.7 -> 102.4 mm, vias 4 -> 3
- net TXD0: track 24.7 -> 19.7 mm
- net LED_OUT: track 10.9 -> 15.9 mm
- net VSPI_MOSI: track 91.1 -> 95.7 mm, vias 5 -> 4
- net VSPI_CLK: track 83.0 -> 86.8 mm, vias 4 -> 3
- net RXD0: track 22.9 -> 20.2 mm
- net GND: track 64.8 -> 67.1 mm
- net GPIO_OUT_2: track 36.6 -> 35.4 mm
- net A: track 9.88 -> 10.9 mm, vias 1 -> 0
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Other:
- board text added: "IO1"
- board text added: "IO2"
- board text added: "IO3"
- board text added: "IO4"
- board text added: "X"
- board text added: "even more memes go here"
- board text removed: "G_1"
- board text removed: "G_2"
- board text removed: "G_3"
- board text removed: "G_4"
- board text removed: "G_5"
- board text removed: "hey put that back!"

Commit message: Aaaaaaaa
Connections:
- J8 pad 7: GPIO_OUT_5 -> unconnected-(J8-Pin_7-Pad7)
- U5 pad 6: EXT_PWR_SENSE -> BATT_PWR_SENSE
- U5 pad 7: BATT_PWR_SENSE -> EXT_PWR_SENSE
Changed lines of the file:
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@@
 	(net 19 "AN_IN_3")
 	(net 20 "GPIO_OUT_4")
-	(net 21 "GPIO_OUT_5")
+	(net 21 "unconnected-(J8-Pin_7-Pad7)")
 	(net 22 "GPIO_OUT_1")
 	(net 23 "GPIO_OUT_2")
@@
 			(size 1.5 0.9)
 			(layers "F.Cu" "F.Mask" "F.Paste")
-			(net 73 "EXT_PWR_SENSE")
+			(net 72 "BATT_PWR_SENSE")
 			(pinfunction "IO34")
 			(pintype "input")
@@
 			(size 1.5 0.9)
 			(layers "F.Cu" "F.Mask" "F.Paste")
-			(net 72 "BATT_PWR_SENSE")
+			(net 73 "EXT_PWR_SENSE")
 			(pinfunction "IO35")
 			(pintype "input")
@@
 			(layers "F&B.Cu" "*.Mask")
 			(remove_unused_layers no)
-			(net 21 "GPIO_OUT_5")
+			(net 21 "unconnected-(J8-Pin_7-Pad7)")
 			(pinfunction "Pin_7")
-			(pintype "passive")
+			(pintype "passive+no_connect")
 		)
 		(pad "8" thru_hole rect
@@
 			(type solid)
 		)
-		(fill no)
+		(fill yes)
 		(layer "B.SilkS")
 	)
