File: Constellation Saddle V1.1/Constellation Saddle V1.1.kicad_sch (KiCad schematic)
At the start: 34 parts, among them J1 2601-1104, J15 ADC_IN, J17 PWR, J18 GPIO/ESP_ADC OUT, J2 2601-1104, J3 MTJ-88ARX1-FSM-LG, J4 SIGNAL_OUT, J6 2601-1102, J7 2601-1104, J8 2601-1104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

Commit message: Aaaaaaaa
Parts:
- removed R10: 55, symbol Device:R
- C1: footprint Capacitor_SMD:C_0805_2012Metric_Pad1.18x1.45mm_HandSolder -> Capacitor_SMD:C_0805_2012Metric
- D1, D2, D3: footprint LED_THT:LED_D5.0mm -> LED_SMD:LED_0805_2012Metric
- D4: value 1N007 -> CUS10S30; footprint 1N4007:CR_1N4005_ONS -> Diode_SMD:D_SOD-323
- J1: renamed from J9; footprint (none) -> Connector_Wire:SolderWire-0.75sqmm_1x02_P4.8mm_D1.25mm_OD2.3mm_Relief
- J10: renamed from J7; footprint CONN4_2601-1104_WAG -> WAGO 2601-1104:CONN4_2601-1104_WAG
- J11: renamed from J8; footprint CONN4_2601-1104_WAG -> WAGO 2601-1104:CONN4_2601-1104_WAG
- J2: renamed from J3; footprint MTJ-88ARX1-FSM-LG:ADAMTECH_MTJ-88ARX1-FSM-LG -> MTJ_88ARX1_FSM_LG:ADAMTECH_MTJ-88ARX1-FSM-LG
- J3: renamed from J6; footprint 2601_1102:CONN2_2601-1102_WAG -> WAGO 2601-1102:CONN2_2601-1102_WAG
- J5: renamed from J4; footprint 2601_1108:CONN8_2601-1108_WAG -> WAGO 2601-1108:CONN8_2601-1108_WAG
- J8: renamed from J1; footprint CONN4_2601-1104_WAG -> WAGO 2601-1104:CONN4_2601-1104_WAG
- J9: renamed from J2; footprint CONN4_2601-1104_WAG -> WAGO 2601-1104:CONN4_2601-1104_WAG
- R1: footprint Resistor_THT:R_Axial_DIN0207_L6.3mm_D2.5mm_P7.62mm_Horizontal -> Resistor_SMD:R_0805_2012Metric
- R10: renamed from R5; footprint Resistor_THT:R_Axial_DIN0207_L6.3mm_D2.5mm_P7.62mm_Horizontal -> Resistor_SMD:R_0805_2012Metric
- R2: renamed from R3; footprint Resistor_THT:R_Axial_DIN0207_L6.3mm_D2.5mm_P7.62mm_Horizontal -> Resistor_SMD:R_0805_2012Metric
- R3: renamed from R6; value R -> 51.1k; footprint (none) -> Resistor_SMD:R_0805_2012Metric
- R4: renamed from R8; value R -> 51.1k; footprint (none) -> Resistor_SMD:R_0805_2012Metric
- R5: renamed from R7; value R -> 10k; footprint (none) -> Resistor_SMD:R_0805_2012Metric
- R6: renamed from R9; value R -> 10k; footprint (none) -> Resistor_SMD:R_0805_2012Metric
- R7: renamed from R2; footprint Resistor_THT:R_Axial_DIN0207_L6.3mm_D2.5mm_P7.62mm_Horizontal -> Resistor_SMD:R_0805_2012Metric
- R9: renamed from R4; footprint Resistor_THT:R_Axial_DIN0207_L6.3mm_D2.5mm_P7.62mm_Horizontal -> Resistor_SMD:R_0805_2012Metric
- renumbered J17 to J4, J18 to J6, J15 to J7, Q4 to Q1, Q5 to Q4
Connections:
- net AN_IN_0 is gone; now on net ENG_CHAMBER: J7.8 (Pin_8)
- net AN_IN_1 is gone; now on net F_TANK: J7.7 (Pin_7)
- net AN_IN_2 is gone; now on net O_TANK: J7.6 (Pin_6)
- net AN_IN_3 is gone; now on net HE_TANK: J7.5 (Pin_5)
- net GPIO_OUT_1 is gone; now on net MOV: J6.3 (Pin_3)
- net GPIO_OUT_2 is gone; now on net MFV: J6.4 (Pin_4)
- net GPIO_OUT_3 is gone; now on net F_VENT: J6.5 (Pin_5)
- net GPIO_OUT_4 is gone; now on net O_VENT: J6.6 (Pin_6)
- net VBUS is gone; now on net PWR: C1.1, D4.1 (K), Q3.3 (D), R2.1
- net BATT_PWR_SENSE: now also J4.3 (Pin_3); no longer J4.4 (Pin_4)
- net EXT_PWR_SENSE: now also J4.4 (Pin_4); no longer J4.3 (Pin_3)
- net GND: no longer J2.9
- no-connect marks 6 -> 10
Other:
- moved on the sheet: C1, D1, D2, D3, D4, J2, Q1, Q2, Q3, Q4, R1, R10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
