File: LabJack DB37 PCB/LabJack DB37 PCB.kicad_sch (KiCad schematic)
At the start: 1 part, among them J1 DC37_Pins_MountingHoles

Commit message: DB37
Connections:
- net GND: now also J1.1, J1.10, J1.19, J1.30, J1.8
- net AIN13: now reaches J1.12
- net AIN11: now reaches J1.13
- net AIN9: now reaches J1.14
- net AIN7: now reaches J1.15
- net AIN5: now reaches J1.16
- net AIN3: now reaches J1.17
- net AIN1: now reaches J1.18
- net FIO7: now reaches J1.21
- net FIO5: now reaches J1.22
- net FIO3: now reaches J1.23
- net FIO1: now reaches J1.24
- net MIO0: now reaches J1.25
- net MIO2: now reaches J1.26
- net +5V: now reaches J1.27
- net FIO6: now reaches J1.3
- net AIN12: now reaches J1.31
- net AIN10: now reaches J1.32
- net AIN8: now reaches J1.33
- net AIN6: now reaches J1.34
- net AIN4: now reaches J1.35
- net AIN2: now reaches J1.36
- net AIN0: now reaches J1.37
- net FIO4: now reaches J1.4
- net FIO2: now reaches J1.5
- net FIO0: now reaches J1.6
- net MIO1: now reaches J1.7
- no-connect marks 0 -> 6

Commit message: Push
Parts:
- added J2: 2601-1102, CONN2_2601-1102_WAG, symbol 2601_1102:2601-1102
- added J3: 2601-1103, CONN3_2601-1103_WAG, symbol 2601_1103:2601-1103
Changed lines of the file:
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@@
+	)
+	(symbol
+		(lib_id "2601_1102:2601-1102")
+		(at 161.925 45.72 0)
+		(unit 1)
+		(exclude_from_sim no)
+		(in_bom yes)
+		(on_board yes)
+		(dnp no)
+		(fields_autoplaced yes)
+		(property "Reference" "J2"
+			(at 176.53 48.2599 0)
+			(effects
+				(font
+					(size 1.524 1.524)
+				)
+				(justify left)
+			)
+		)
+		(property "Value" "2601-1102"
+			(at 176.53 50.7999 0)
+			(effects
+				(font
+					(size 1.524 1.524)
+				)
+				(justify left)
+			)
+		)
+		(property "Footprint" "CONN2_2601-1102_WAG"
+			(at 161.925 45.72 0)
+			(effects
+				(font
+					(size 1.27 1.27)
+					(italic yes)
+				)
+				(hide yes)
+			)
+		)
+		(property "Datasheet" "2601-1102"
+			(at 161.925 45.72 0)
+			(effects
+				(font
+					(size 1.27 1.27)
+					(italic yes)
+				)
+				(hide yes)
+			)
+		)
+		(property "Description" ""
+			(at 161.925 45.72 0)
+			(effects
+				(font
+					(size 1.27 1.27)
+				)
+				(hide yes)
+			)
+		)
+		(pin "4"
+		)
+		(pin "2"
+		)
+		(pin "3"
+		)
+		(pin "1"
+		)
+		(instances
+			(project ""
+				(path "/704067de-520d-4444-be45-b08d50d6f95a"
+					(reference "J2")
+					(unit 1)
+				)
+			)
+		)
+	)
+	(symbol
+		(lib_id "2601_1103:2601-1103")
+		(at 169.545 78.105 0)
+		(unit 1)
+		(exclude_from_sim no)
+		(in_bom yes)
+		(on_board yes)
+		(dnp no)
+		(fields_autoplaced yes)
+		(property "Reference" "J3"
+			(at 184.15 83.1849 0)
+			(effects
+				(font
+					(size 1.524 1.524)
+				)
+				(justify left)
+			)
+		)
+		(property "Value" "2601-1103"
+			(at 184.15 85.7249 0)
+			(effects
+				(font
+					(size 1.524 1.524)
+				)
+				(justify left)
+			)
+		)
+		(property "Footprint" "CONN3_2601-1103_WAG"
+			(at 169.545 78.105 0)
+			(effects
+				(font
+					(size 1.27 1.27)
+					(italic yes)
+				)
+				(hide yes)
+			)
+		)
+		(property "Datasheet" "2601-1103"
+			(at 169.545 78.105 0)
+			(effects
+				(font
+					(size 1.27 1.27)
+					(italic yes)
+				)
+				(hide yes)
+			)
+		)
+		(property "Description" ""
+			(at 169.545 78.105 0)
+			(effects
+				(font
+					(size 1.27 1.27)
+				)
+				(hide yes)
+			)
+		)
+		(pin "4"
+		)
+		(pin "6"
+		)
+		(pin "2"
+		)
+		(pin "1"
+		)
+		(pin "5"
+		)
+		(pin "3"
+		)
+		(instances
+			(project ""
+				(path "/704067de-520d-4444-be45-b08d50d6f95a"
+					(reference "J3")
+					(unit 1)
+				)
+			)
+		)
 	)
 	(symbol
