File: 2025-2026 NI Breakout Board/2025-2026 NI Breakout Board.kicad_pcb (KiCad board)
At the start: 2 copper layers, 190.5 x 254 mm, 201 parts, among them J1 NI9205CONN, J10 GNDCONN, J11 AICONN, J12 AICONN, J13 24VCONN, J14 GNDCONN, J15 NI9205CONN, J17 24VCONN, J18 GNDCONN, J19 AICONN, J2 PWRCONN, J20 24VCONN, J21 GNDCONN, J22 AICONN, J23 24VCONN, J24 GNDCONN, J25 AICONN, J26 AICONN, J27 24VCONN, J28 GNDCONN, J29 NI9253CONN, J3 24VCONN, J30 AICONN, J31 VSUPCONN, J32 PWRCONN, J33 NI9237CONN, J34 LC0, J35 LC1, J36 LC2, J37 LC3, J38 NI9485CONN, J39 PWRCONN, J4 GNDCONN, J40 AICONN, J41 GNDCONN, J42 NI9485CONN, J43 PWRCONN, J44 AICONN, J45 GNDCONN, J5 AICONN, J6 24VCONN, J7 GNDCONN, J8 AICONN, J9 24VCONN, Q1 FQP27P06, Q2 FQP27P06, Q3 FQP27P06, Q4 FQP27P06

Commit message: Aaahaha
Parts:
- added J16: PWRCONN, WAGO 2601-1102:CONN2_2601-1102_WAG, F.Cu at (55.9, 165.1)
- added Q5: FQP27P06, Package_TO_SOT_THT:TO-220-3_Horizontal_TabDown, F.Cu at (81.1, 41.6)
- added TP89: TestPoint, TestPoint:TestPoint_THTPad_D2.0mm_Drill1.0mm, F.Cu at (90.8, 169.6)
- added TP90: TestPoint, TestPoint:TestPoint_THTPad_D2.0mm_Drill1.0mm, F.Cu at (50.9, 158.0)
- D12, D7: value LED -> 1N4004; footprint LED_THT:LED_D3.0mm -> Diode_THT:D_DO-41_SOD81_P7.62mm_Horizontal
- D13, D3, D4: value 1N4004 -> LED; footprint Diode_THT:D_DO-41_SOD81_P7.62mm_Horizontal -> LED_THT:LED_D3.0mm
- R12: value 1.1k -> 100K
- R13, R3: value 100K -> 1.1k
- moved R2 220.5 mm to (90.8, 166.4)
- moved J29 213.1 mm to (55.9, 147.3)
- moved J32 213.0 mm to (55.9, 129.8)
- moved J31 206.5 mm to (105.4, 133.3)
- moved J30 206.5 mm to (105.4, 144.8)
- moved D5 205.9 mm to (166.3, 61.9), turned to -135 degrees
- moved Q2 197.3 mm to (85.3, 169.5), turned to 90 degrees
- moved D6 197.1 mm to (166.3, 57.1), turned to -135 degrees
- moved F1 190.5 mm to (93.9, 130.3)
- moved D7 188.4 mm to (166.3, 52.2), turned to -135 degrees
- moved D8 179.7 mm to (166.3, 47.4), turned to -135 degrees
- moved D9 171.1 mm to (166.3, 42.6), turned to -135 degrees
- moved D10 162.5 mm to (166.3, 37.8), turned to -135 degrees
- moved D11 154.0 mm to (166.3, 33.0), turned to -135 degrees
- moved D12 145.5 mm to (166.3, 28.1), turned to -135 degrees
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Connections:
- D10 pad 1: NI9485A_CH6B -> NI9485A_CH5B
- D11 pad 1: NI9485A_CH7B -> NI9485A_CH6B
- D12 pad 1: COM -> NI9485A_CH7B
- D12 pad 2: Net-(D12-A) -> COM
- D13 pad 1: NI9485B_CH0B -> COM
- D13 pad 2: COM -> Net-(D13-A)
- D14 pad 1: NI9485B_CH1B -> NI9485B_CH0B
- D15 pad 1: NI9485B_CH2B -> NI9485B_CH1B
- D16 pad 1: NI9485B_CH3B -> NI9485B_CH2B
- D17 pad 1: NI9485B_CH4B -> NI9485B_CH3B
- D18 pad 1: NI9485B_CH5B -> NI9485B_CH4B
- D19 pad 1: NI9485B_CH6B -> NI9485B_CH5B
- D20 pad 1: NI9485B_CH7B -> NI9485B_CH6B
- D3 pad 1: NI9485A_CH0B -> COM
- D3 pad 2: COM -> Net-(D3-A)
- D4 pad 1: Net-(D4-K) -> COM
- D4 pad 2: COM -> Net-(D4-A)
- D5 pad 1: NI9485A_CH2B -> NI9485A_CH0B
- D6 pad 1: NI9485A_CH3B -> Net-(D6-K)
- D7 pad 1: COM -> NI9485A_CH2B
- D7 pad 2: Net-(D7-A) -> COM
- D8 pad 1: NI9485A_CH4B -> NI9485A_CH3B
- D9 pad 1: NI9485A_CH5B -> NI9485A_CH4B
- F1 pad 1: Net-(Q2-S) -> Net-(Q3-S)
- J13 pad 1: NI9205_PWR -> NI9205A_PWR
- J13 pad 10: NI9205_PWR -> NI9205A_PWR
- J13 pad 11: NI9205_PWR -> NI9205A_PWR
- J13 pad 12: NI9205_PWR -> NI9205A_PWR
- J13 pad 13: NI9205_PWR -> NI9205A_PWR
- J13 pad 14: NI9205_PWR -> NI9205A_PWR
- J13 pad 15: NI9205_PWR -> NI9205A_PWR
- J13 pad 16: NI9205_PWR -> NI9205A_PWR
- J13 pad 2: NI9205_PWR -> NI9205A_PWR
- J13 pad 3: NI9205_PWR -> NI9205A_PWR
- J13 pad 4: NI9205_PWR -> NI9205A_PWR
- J13 pad 5: NI9205_PWR -> NI9205A_PWR
- J13 pad 6: NI9205_PWR -> NI9205A_PWR
- J13 pad 7: NI9205_PWR -> NI9205A_PWR
- J13 pad 8: NI9205_PWR -> NI9205A_PWR
- J13 pad 9: NI9205_PWR -> NI9205A_PWR
- J17 pad 1: NI9205_PWR -> NI9205B_PWR
- J17 pad 10: NI9205_PWR -> NI9205B_PWR
- J17 pad 11: NI9205_PWR -> NI9205B_PWR
- J17 pad 12: NI9205_PWR -> NI9205B_PWR
- J17 pad 13: NI9205_PWR -> NI9205B_PWR
- J17 pad 14: NI9205_PWR -> NI9205B_PWR
- J17 pad 15: NI9205_PWR -> NI9205B_PWR
- J17 pad 16: NI9205_PWR -> NI9205B_PWR
- J17 pad 2: NI9205_PWR -> NI9205B_PWR
- J17 pad 3: NI9205_PWR -> NI9205B_PWR
- J17 pad 4: NI9205_PWR -> NI9205B_PWR
- J17 pad 5: NI9205_PWR -> NI9205B_PWR
- J17 pad 6: NI9205_PWR -> NI9205B_PWR
- J17 pad 7: NI9205_PWR -> NI9205B_PWR
- J17 pad 8: NI9205_PWR -> NI9205B_PWR
- J17 pad 9: NI9205_PWR -> NI9205B_PWR
- J20 pad 1: NI9205_PWR -> NI9205B_PWR
- J20 pad 10: NI9205_PWR -> NI9205B_PWR
- J20 pad 11: NI9205_PWR -> NI9205B_PWR
- J20 pad 12: NI9205_PWR -> NI9205B_PWR
- J20 pad 13: NI9205_PWR -> NI9205B_PWR
- J20 pad 14: NI9205_PWR -> NI9205B_PWR
- J20 pad 15: NI9205_PWR -> NI9205B_PWR
- J20 pad 16: NI9205_PWR -> NI9205B_PWR
- J20 pad 2: NI9205_PWR -> NI9205B_PWR
- J20 pad 3: NI9205_PWR -> NI9205B_PWR
- J20 pad 4: NI9205_PWR -> NI9205B_PWR
- J20 pad 5: NI9205_PWR -> NI9205B_PWR
- J20 pad 6: NI9205_PWR -> NI9205B_PWR
- J20 pad 7: NI9205_PWR -> NI9205B_PWR
- J20 pad 8: NI9205_PWR -> NI9205B_PWR
- J20 pad 9: NI9205_PWR -> NI9205B_PWR
- J23 pad 1: NI9205_PWR -> NI9205B_PWR
- J23 pad 10: NI9205_PWR -> NI9205B_PWR
- J23 pad 11: NI9205_PWR -> NI9205B_PWR
- J23 pad 12: NI9205_PWR -> NI9205B_PWR
- J23 pad 13: NI9205_PWR -> NI9205B_PWR
- J23 pad 14: NI9205_PWR -> NI9205B_PWR
- J23 pad 15: NI9205_PWR -> NI9205B_PWR
- J23 pad 16: NI9205_PWR -> NI9205B_PWR
- J23 pad 2: NI9205_PWR -> NI9205B_PWR
- J23 pad 3: NI9205_PWR -> NI9205B_PWR
- J23 pad 4: NI9205_PWR -> NI9205B_PWR
- J23 pad 5: NI9205_PWR -> NI9205B_PWR
- J23 pad 6: NI9205_PWR -> NI9205B_PWR
- J23 pad 7: NI9205_PWR -> NI9205B_PWR
- J23 pad 8: NI9205_PWR -> NI9205B_PWR
- J23 pad 9: NI9205_PWR -> NI9205B_PWR
- J27 pad 1: NI9205_PWR -> NI9205B_PWR
- J27 pad 10: NI9205_PWR -> NI9205B_PWR
- J27 pad 11: NI9205_PWR -> NI9205B_PWR
- J27 pad 12: NI9205_PWR -> NI9205B_PWR
- J27 pad 13: NI9205_PWR -> NI9205B_PWR
- J27 pad 14: NI9205_PWR -> NI9205B_PWR
- J27 pad 15: NI9205_PWR -> NI9205B_PWR
- J27 pad 16: NI9205_PWR -> NI9205B_PWR
- J27 pad 2: NI9205_PWR -> NI9205B_PWR
- J27 pad 3: NI9205_PWR -> NI9205B_PWR
- J27 pad 4: NI9205_PWR -> NI9205B_PWR
- J27 pad 5: NI9205_PWR -> NI9205B_PWR
- J27 pad 6: NI9205_PWR -> NI9205B_PWR
- J27 pad 7: NI9205_PWR -> NI9205B_PWR
- J27 pad 8: NI9205_PWR -> NI9205B_PWR
- J27 pad 9: NI9205_PWR -> NI9205B_PWR
- J3 pad 1: NI9205_PWR -> NI9205A_PWR
- J3 pad 10: NI9205_PWR -> NI9205A_PWR
- J3 pad 11: NI9205_PWR -> NI9205A_PWR
- J3 pad 12: NI9205_PWR -> NI9205A_PWR
- J3 pad 13: NI9205_PWR -> NI9205A_PWR
- J3 pad 14: NI9205_PWR -> NI9205A_PWR
- J3 pad 15: NI9205_PWR -> NI9205A_PWR
- J3 pad 16: NI9205_PWR -> NI9205A_PWR
- J3 pad 2: NI9205_PWR -> NI9205A_PWR
- J3 pad 3: NI9205_PWR -> NI9205A_PWR
- J3 pad 4: NI9205_PWR -> NI9205A_PWR
- J3 pad 5: NI9205_PWR -> NI9205A_PWR
- J3 pad 6: NI9205_PWR -> NI9205A_PWR
- J3 pad 7: NI9205_PWR -> NI9205A_PWR
- J3 pad 8: NI9205_PWR -> NI9205A_PWR
- J3 pad 9: NI9205_PWR -> NI9205A_PWR
- J6 pad 1: NI9205_PWR -> NI9205A_PWR
- J6 pad 10: NI9205_PWR -> NI9205A_PWR
- J6 pad 11: NI9205_PWR -> NI9205A_PWR
- J6 pad 12: NI9205_PWR -> NI9205A_PWR
- J6 pad 13: NI9205_PWR -> NI9205A_PWR
- J6 pad 14: NI9205_PWR -> NI9205A_PWR
- J6 pad 15: NI9205_PWR -> NI9205A_PWR
- J6 pad 16: NI9205_PWR -> NI9205A_PWR
- J6 pad 2: NI9205_PWR -> NI9205A_PWR
- J6 pad 3: NI9205_PWR -> NI9205A_PWR
- J6 pad 4: NI9205_PWR -> NI9205A_PWR
- J6 pad 5: NI9205_PWR -> NI9205A_PWR
- J6 pad 6: NI9205_PWR -> NI9205A_PWR
- J6 pad 7: NI9205_PWR -> NI9205A_PWR
- J6 pad 8: NI9205_PWR -> NI9205A_PWR
- J6 pad 9: NI9205_PWR -> NI9205A_PWR
- J9 pad 1: NI9205_PWR -> NI9205A_PWR
- J9 pad 10: NI9205_PWR -> NI9205A_PWR
- J9 pad 11: NI9205_PWR -> NI9205A_PWR
- J9 pad 12: NI9205_PWR -> NI9205A_PWR
- J9 pad 13: NI9205_PWR -> NI9205A_PWR
- J9 pad 14: NI9205_PWR -> NI9205A_PWR
- J9 pad 15: NI9205_PWR -> NI9205A_PWR
- J9 pad 16: NI9205_PWR -> NI9205A_PWR
- J9 pad 2: NI9205_PWR -> NI9205A_PWR
- J9 pad 3: NI9205_PWR -> NI9205A_PWR
- J9 pad 4: NI9205_PWR -> NI9205A_PWR
- J9 pad 5: NI9205_PWR -> NI9205A_PWR
- J9 pad 6: NI9205_PWR -> NI9205A_PWR
- J9 pad 7: NI9205_PWR -> NI9205A_PWR
- J9 pad 8: NI9205_PWR -> NI9205A_PWR
- J9 pad 9: NI9205_PWR -> NI9205A_PWR
- Q1 pad 3: NI9205_PWR -> NI9205A_PWR
- Q2 pad 2: Net-(J32-2_1) -> Net-(J16-2_1)
- Q2 pad 3: Net-(Q2-S) -> NI9205B_PWR
- Q3 pad 2: Net-(J39-2_1) -> Net-(J32-2_1)
- Q3 pad 3: NI9485A_24V+ -> Net-(Q3-S)
- Q4 pad 2: Net-(J43-2_1) -> Net-(J39-2_1)
- Q4 pad 3: NI9485B_24V+ -> NI9485A_24V+
- R1 pad 1: NI9205_PWR -> NI9205A_PWR
- R10 pad 1: NI9485A_CH6B -> NI9485A_CH5B
- R11 pad 1: NI9485A_CH7B -> NI9485A_CH6B
- R12 pad 1: NI9485B_24V+ -> NI9485A_CH7B
- R12 pad 2: Net-(D12-A) -> COM
- R13 pad 1: NI9485B_CH0B -> NI9485B_24V+
- R13 pad 2: COM -> Net-(D13-A)
- R14 pad 1: NI9485B_CH1B -> NI9485B_CH0B
- R15 pad 1: NI9485B_CH2B -> NI9485B_CH1B
- R16 pad 1: NI9485B_CH3B -> NI9485B_CH2B
- R17 pad 1: NI9485B_CH4B -> NI9485B_CH3B
- R18 pad 1: NI9485B_CH5B -> NI9485B_CH4B
- R19 pad 1: NI9485B_CH6B -> NI9485B_CH5B
- R2 pad 1: VSUP -> NI9205B_PWR
- R20 pad 1: NI9485B_CH7B -> NI9485B_CH6B
- R3 pad 1: NI9485A_CH0B -> VSUP
- R3 pad 2: COM -> Net-(D3-A)
- R4 pad 2: Net-(D7-A) -> Net-(D4-A)
- R5 pad 1: Net-(D4-K) -> NI9485A_CH0B
- R6 pad 1: NI9485A_CH2B -> Net-(D6-K)
- R7 pad 1: NI9485A_CH3B -> NI9485A_CH2B
- R8 pad 1: NI9485A_CH4B -> NI9485A_CH3B
- R9 pad 1: NI9485A_CH5B -> NI9485A_CH4B
- TP1 pad 1: NI9205_PWR -> NI9205A_PWR
Routing:
- net AI5: track 0.00 -> 102.0 mm
- net AI4: track 0.00 -> 94.6 mm
- net AI3: track 0.00 -> 87.0 mm
- net AI7: track 0.00 -> 86.9 mm
- net AI6: track 0.00 -> 85.6 mm
- net AI2: track 0.00 -> 79.0 mm
- net AI1: track 0.00 -> 70.9 mm
- net AI0: track 0.00 -> 63.5 mm
- net Net-(J16-2_1): track 0.00 -> 36.4 mm
- net Net-(J32-2_1): track 0.00 -> 34.5 mm
- net Net-(Q3-S): track 0.00 -> 7.65 mm
- net Net-(J2-2_1): track 34.2 -> 36.8 mm
- added copper zone on F.Cu, net NI9205A_PWR
- added copper zone on F.Cu, net NI9205B_PWR
- added copper zone on F.Cu, net VSUP
- removed copper zone on F.Cu, net NI9205_PWR
Other:
- board size 190.5 x 254 mm -> 190.5 x 279.4 mm

Commit message: AGS PCBS
Parts:
- added H10: MountingHole_Pad, MountingHole:MountingHole_3.2mm_M3_DIN965_Pad_TopBottom, F.Cu at (71.1, 83.8)
- added H11: MountingHole_Pad, MountingHole:MountingHole_3.2mm_M3_DIN965_Pad_TopBottom, F.Cu at (154.9, 83.8)
- added H12: MountingHole_Pad, MountingHole:MountingHole_3.2mm_M3_DIN965_Pad_TopBottom, F.Cu at (209.6, 83.8)
- added H13: MountingHole_Pad, MountingHole:MountingHole_3.2mm_M3_DIN965_Pad_TopBottom, F.Cu at (31.8, 111.8)
- added H14: MountingHole_Pad, MountingHole:MountingHole_3.2mm_M3_DIN965_Pad_TopBottom, F.Cu at (105.4, 116.8)
- added H15: MountingHole_Pad, MountingHole:MountingHole_3.2mm_M3_DIN965_Pad_TopBottom, F.Cu at (146.1, 116.8)
- added H16: MountingHole_Pad, MountingHole:MountingHole_3.2mm_M3_DIN965_Pad_TopBottom, F.Cu at (209.6, 116.8)
- added H17: MountingHole_Pad, MountingHole:MountingHole_3.2mm_M3_DIN965_Pad_TopBottom, F.Cu at (31.8, 152.4)
- added H18: MountingHole_Pad, MountingHole:MountingHole_3.2mm_M3_DIN965_Pad_TopBottom, F.Cu at (149.9, 146.1)
- added H19: MountingHole_Pad, MountingHole:MountingHole_3.2mm_M3_DIN965_Pad_TopBottom, F.Cu at (165.1, 179.1)
- added H20: MountingHole_Pad, MountingHole:MountingHole_3.2mm_M3_DIN965_Pad_TopBottom, F.Cu at (209.6, 179.1)
- added H21: MountingHole_Pad, MountingHole:MountingHole_3.2mm_M3_DIN965_Pad_TopBottom, F.Cu at (31.8, 215.9)
- added H22: MountingHole_Pad, MountingHole:MountingHole_3.2mm_M3_DIN965_Pad_TopBottom, F.Cu at (109.2, 208.3)
- added H23: MountingHole_Pad, MountingHole:MountingHole_3.2mm_M3_DIN965_Pad_TopBottom, F.Cu at (154.9, 208.3)
- added H24: MountingHole_Pad, MountingHole:MountingHole_3.2mm_M3_DIN965_Pad_TopBottom, F.Cu at (209.6, 208.3)
- added H25: MountingHole_Pad, MountingHole:MountingHole_3.2mm_M3_DIN965_Pad_TopBottom, F.Cu at (165.1, 241.3)
- added H26: MountingHole_Pad, MountingHole:MountingHole_3.2mm_M3_DIN965_Pad_TopBottom, F.Cu at (209.6, 241.3)
- added H27: MountingHole_Pad, MountingHole:MountingHole_3.2mm_M3_DIN965_Pad_TopBottom, F.Cu at (31.8, 273.1)
- added H28: MountingHole_Pad, MountingHole:MountingHole_3.2mm_M3_DIN965_Pad_TopBottom, F.Cu at (105.4, 273.1)
- added H29: MountingHole_Pad, MountingHole:MountingHole_3.2mm_M3_DIN965_Pad_TopBottom, F.Cu at (157.5, 273.1)
- added H30: MountingHole_Pad, MountingHole:MountingHole_3.2mm_M3_DIN965_Pad_TopBottom, F.Cu at (209.6, 273.1)
- added H7: MountingHole_Pad, MountingHole:MountingHole_3.2mm_M3_DIN965_Pad_TopBottom, F.Cu at (177.8, 45.6)
- added H8: MountingHole_Pad, MountingHole:MountingHole_3.2mm_M3_DIN965_Pad_TopBottom, F.Cu at (209.6, 45.7)
- added H9: MountingHole_Pad, MountingHole:MountingHole_3.2mm_M3_DIN965_Pad_TopBottom, F.Cu at (31.8, 83.8)
- added J46: NI_9485A_D-SUB, Connector_Dsub:DSUB-9_Pins_Vertical_P2.77x2.84mm_MountingHoles, F.Cu at (180.3, 71.1)
- added J47: NI_9485B_D-SUB, Connector_Dsub:DSUB-9_Pins_Vertical_P2.77x2.84mm_MountingHoles, F.Cu at (180.3, 31.8)
- moved H4 320.5 mm to (209.6, 6.35)
- moved D2 221.3 mm to (84.4, 158.8)
- moved H5 219.9 mm to (31.8, 45.7)
- moved H6 167.5 mm to (83.8, 45.7)
- moved R3 146.1 mm to (82.8, 119.0), turned to 180 degrees
- moved TP67 142.5 mm to (88.5, 119.0)
- moved TP68 136.6 mm to (55.3, 116.2)
- moved D3 113.3 mm to (70.0, 119.0)
- moved F10 112.6 mm to (97.4, 32.9)
- moved H2 111.5 mm to (82.5, 6.35), turned to 45 degrees
- moved F14 110.5 mm to (97.4, 15.9)
- moved H3 108.1 mm to (177.8, 6.35)
- moved F11 105.0 mm to (97.4, 28.6)
- moved F15 103.4 mm to (97.4, 11.5)
- moved F12 97.6 mm to (97.4, 24.4)
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Connections:
- net Net-(J39-2_1) renamed /V_IN_A
- net Net-(J43-2_1) renamed /V_IN_B
- D6 pad 1: Net-(D6-K) -> NI9485A_CH1B
- J36 pad 1: NI9237_AI2- -> RS2+
- J36 pad 10: RS2- -> NI9237_AI2+
- J36 pad 11: RS2+ -> NI9237_AI2-
- J36 pad 12: RS2+ -> NI9237_AI2-
- J36 pad 2: NI9237_AI2- -> RS2+
- J36 pad 3: NI9237_AI2+ -> RS2-
- J36 pad 4: NI9237_AI2+ -> RS2-
- J36 pad 5: EX2- -> EX2+
- J36 pad 6: EX2- -> EX2+
- J36 pad 7: EX2+ -> EX2-
- J36 pad 8: EX2+ -> EX2-
- J36 pad 9: RS2- -> NI9237_AI2+
- J37 pad 1: NI9237_AI3- -> RS3+
- J37 pad 10: RS3- -> NI9237_AI3+
- J37 pad 11: RS3+ -> NI9237_AI3-
- J37 pad 12: RS3+ -> NI9237_AI3-
- J37 pad 2: NI9237_AI3- -> RS3+
- J37 pad 3: NI9237_AI3+ -> RS3-
- J37 pad 4: NI9237_AI3+ -> RS3-
- J37 pad 5: EX3- -> EX3+
- J37 pad 6: EX3- -> EX3+
- J37 pad 7: EX3+ -> EX3-
- J37 pad 8: EX3+ -> EX3-
- J37 pad 9: RS3- -> NI9237_AI3+
- R6 pad 1: Net-(D6-K) -> NI9485A_CH1B
Routing:
- net NI9485B_CH7B: track 0.00 -> 104.6 mm, vias 0 -> 1
- net NI9485A_CH7B: track 0.00 -> 104.1 mm, vias 0 -> 1
- net NI9485B_CH6B: track 0.00 -> 97.8 mm
- net NI9485A_CH6B: track 0.00 -> 97.2 mm
- net NI9485B_CH5B: track 0.00 -> 96.4 mm
- net NI9485A_CH5B: track 0.00 -> 95.7 mm
- net NI9485B_CH4B: track 0.00 -> 91.1 mm
- net NI9485A_CH0B: track 0.00 -> 82.3 mm
- net NI9485B_CH3B: track 0.00 -> 82.1 mm
- net NI9485A_CH1B: track 0.00 -> 82.1 mm
- net NI9485B_CH2B: track 0.00 -> 81.9 mm
- net NI9485A_CH4B: track 0.00 -> 81.7 mm
- net NI9485B_CH1B: track 0.00 -> 81.7 mm
- net NI9485A_CH2B: track 0.00 -> 81.6 mm
- net NI9485B_CH0B: track 0.00 -> 81.6 mm
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- added copper zone on F.Cu, net /V_IN_A
- added copper zone on F.Cu, net /V_IN_B
- added copper zone on F.Cu, net NI9485A_24V+
- added copper zone on F.Cu, net NI9485B_24V+
Other:
- outline, holes or cut-outs redrawn
- board text added: "1.1K"
- board text added: "100K"
- board text added: "1N4004"
- board text added: "9485A CONN"
- board text added: "9485B CONN"
- board text added: "AI0"
- board text added: "AI0+"
- board text added: "AI0-"
- board text added: "AI1"
- board text added: "AI1+"
- board text added: "AI1-"
- board text added: "AI10"
- board text added: "AI11"
- board text added: "AI12"
- board text added: "AI13"
- board text added: "AI14"
- board text added: "AI15"
- board text added: "AI16"
- board text added: "AI17"
- board text added: "AI18"
- board text added: "AI19"
- board text added: "AI2"
- board text added: "AI2+"
- board text added: "AI2-"
- board text added: "AI20"
- board text added: "AI21"
- board text added: "AI22"
- board text added: "AI23"
- board text added: "AI24"
- board text added: "AI25"
- board text added: "AI26"
- board text added: "AI27"
- board text added: "AI28"
- board text added: "AI29"
- board text added: "AI3"
- board text added: "AI3+"
- board text added: "AI3-"
- board text added: "AI30"
- board text added: "AI31"
- board text added: "AI4"
- board text added: "AI5"
- board text added: "AI6"
- board text added: "AI7"
- board text added: "AI8"
- board text added: "AI9"
- board text added: "A_CH_0"
- board text added: "A_CH_1"
- board text added: "A_CH_2"
- board text added: "A_CH_3"
- board text added: "A_CH_4"
- board text added: "A_CH_5"
- board text added: "A_CH_6"
- board text added: "A_CH_7"
- board text added: "B_CH_0"
- board text added: "B_CH_1"
- board text added: "B_CH_2"
- board text added: "B_CH_3"
- board text added: "B_CH_4"
- board text added: "B_CH_5"
- board text added: "B_CH_6"
- board text added: "B_CH_7"
- board text added: "DC VOLTAGE NO GREATER THAN 60V"
- board text added: "EX0+"
- board text added: "EX0-"
- board text added: "EX1+"
- board text added: "EX1-"
- board text added: "EX2+"
- board text added: "EX2-"
- board text added: "EX3+"
- board text added: "EX3-"
- board text added: "EXPECTED 24V DC IN"
- board text added: "FQP27P06"
- board text added: "LC 0"
- board text added: "LC 1"
- board text added: "LC 2"
- board text added: "LC 3"
- board text added: "NI 9253 PWR"
- board text added: "RELAY_A_PWR"
- board text added: "RELAY_B_PWR"
- board text added: "RS0+"
- board text added: "RS0-"
- board text added: "RS1+"
- board text added: "RS1-"
- board text added: "RS2+"
- board text added: "RS2-"
- board text added: "RS3+"
- board text added: "RS3-"
- board text added: "TP_9205_A_PWR"
- board text added: "TP_9205_B_PWR"
- board text added: "TP_AI_0"
- board text added: "TP_AI_1"
- board text added: "TP_AI_10"
- board text added: "TP_AI_11"
- board text added: "TP_AI_12"
- board text added: "TP_AI_13"
- board text added: "TP_AI_14"
- board text added: "TP_AI_15"
- board text added: "TP_AI_16"
- board text added: "TP_AI_17"
- board text added: "TP_AI_18"
- board text added: "TP_AI_19"
- board text added: "TP_AI_2"
- board text added: "TP_AI_20"
- board text added: "TP_AI_21"
- board text added: "TP_AI_22"
- board text added: "TP_AI_23"
- board text added: "TP_AI_24"
- board text added: "TP_AI_25"
- board text added: "TP_AI_26"
- board text added: "TP_AI_27"
- board text added: "TP_AI_28"
- board text added: "TP_AI_29"
- board text added: "TP_AI_3"
- board text added: "TP_AI_30"
- board text added: "TP_AI_31"
- board text added: "TP_AI_4"
- board text added: "TP_AI_5"
- board text added: "TP_AI_6"
- board text added: "TP_AI_7"
- board text added: "TP_AI_8"
- board text added: "TP_AI_9"
- board text added: "TP_GND"
- board text added: "TP_RELAY_A_PWR"
- board text added: "TP_RELAY_B_PWR"
- board text added: "TP_V_SUP"
- board text added: "V SUP"
- board text added: "VIN"

Commit message: Producation files
Parts:
- added G***: LOGO, LOGO, F.Cu at (85.3, 144.1)
- added G***: LOGO, LOGO, F.Cu at (170.2, 134.6)
- added G***: LOGO, LOGO, F.Cu at (180.8, 117.5)
- added G***: LOGO, LOGO, F.Cu at (192.3, 270.6)
- added H31: MountingHole_Pad, MountingHole:MountingHole_3.2mm_M3_DIN965_Pad_TopBottom, F.Cu at (104.1, 273.1)
- added H32: MountingHole_Pad, MountingHole:MountingHole_3.2mm_M3_DIN965_Pad_TopBottom, F.Cu at (139.7, 273.1)
- added H33: MountingHole_Pad, MountingHole:MountingHole_3.2mm_M3_DIN965_Pad_TopBottom, F.Cu at (177.8, 273.1)
- added H34: MountingHole_Pad, MountingHole:MountingHole_3.2mm_M3_DIN965_Pad_TopBottom, F.Cu at (209.6, 273.1)
- moved H20 177.8 mm to (31.8, 182.9)
- moved H30 177.8 mm to (31.8, 273.1)
- moved H21 138.0 mm to (165.1, 180.3)
- moved H23 123.3 mm to (31.8, 213.4)
- moved H22 104.1 mm to (209.6, 180.3)
- moved H24 82.6 mm to (127.0, 208.3)
- moved H28 69.9 mm to (167.6, 241.3)
- moved H29 61.0 mm to (209.6, 241.3)
- moved H19 55.4 mm to (209.6, 146.1)
- moved H17 42.1 mm to (73.7, 156.2)
- moved H7 33.4 mm to (144.8, 40.6), turned to 0 degrees
- moved H25 33.1 mm to (162.6, 208.3)
- moved H26 33.0 mm to (209.6, 208.3)
- moved H27 29.2 mm to (31.8, 243.8)
- moved H15 6.35 mm to (152.4, 116.8)
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Connections:
- H1 pad 1: COM -> unconnected-(H1-Pad1)_1
- H10 pad 1: COM -> unconnected-(H10-Pad1)_1
- H11 pad 1: COM -> unconnected-(H11-Pad1)_2
- H12 pad 1: COM -> unconnected-(H12-Pad1)
- H13 pad 1: COM -> unconnected-(H13-Pad1)_1
- H14 pad 1: COM -> unconnected-(H14-Pad1)
- H15 pad 1: COM -> unconnected-(H15-Pad1)
- H16 pad 1: COM -> unconnected-(H16-Pad1)_2
- H17 pad 1: COM -> unconnected-(H17-Pad1)_1
- H18 pad 1: COM -> unconnected-(H18-Pad1)
- H19 pad 1: COM -> unconnected-(H19-Pad1)_2
- H2 pad 1: COM -> unconnected-(H2-Pad1)
- H20 pad 1: COM -> unconnected-(H20-Pad1)_2
- H21 pad 1: COM -> unconnected-(H21-Pad1)
- H22 pad 1: COM -> unconnected-(H22-Pad1)
- H23 pad 1: COM -> unconnected-(H23-Pad1)_2
- H24 pad 1: COM -> unconnected-(H24-Pad1)
- H25 pad 1: COM -> unconnected-(H25-Pad1)
- H26 pad 1: COM -> unconnected-(H26-Pad1)_1
- H27 pad 1: COM -> unconnected-(H27-Pad1)
- H28 pad 1: COM -> unconnected-(H28-Pad1)
- H29 pad 1: COM -> unconnected-(H29-Pad1)
- H3 pad 1: COM -> unconnected-(H3-Pad1)
- H30 pad 1: COM -> unconnected-(H30-Pad1)
- H4 pad 1: COM -> unconnected-(H4-Pad1)_1
- H5 pad 1: COM -> unconnected-(H5-Pad1)_1
- H6 pad 1: COM -> unconnected-(H6-Pad1)
- H7 pad 1: COM -> unconnected-(H7-Pad1)_1
- H8 pad 1: COM -> unconnected-(H8-Pad1)_2
- H9 pad 1: COM -> unconnected-(H9-Pad1)
Other:
- board text added: "BOTTOM TEXT"
- board text added: "Click Clack these valves are WACK"
- board text added: "GET IT?"
- board text added: "PAPER AH BOARD"
- board text added: "Please work"
- board text added: "THE WHOLE BOARD IS A MEME"
