File: 2025-2026 NI Breakout Board/2025-2026 NI Breakout Board.kicad_sch (KiCad schematic)
At the start: 31 parts, among them J1 NI9205CONN, J10 GNDCONN, J11 GNDCONN, J12 GNDCONN, J13 24VCONN, J14 GNDCONN, J15 NI9205CONN, J16 PWRCONN, J17 24VCONN, J18 GNDCONN, J19 GNDCONN, J2 PWRCONN, J20 24VCONN, J21 GNDCONN, J22 GNDCONN, J23 24VCONN, J24 GNDCONN, J25 GNDCONN, J26 GNDCONN, J27 24VCONN, J28 GNDCONN, J29 NI9253CONN, J3 24VCONN, J4 GNDCONN, J5 GNDCONN, J6 24VCONN, J7 GNDCONN, J8 GNDCONN, J9 24VCONN

Commit message: Ni breakout
Parts:
- added J30: PWRCONN, WAGO 2601-1102:CONN2_2601-1102_WAG, symbol 2602_1102:2601-1102
- added J31: GNDCONN, TBLH10V-350-08BK:RHDR16W80P550X350_2X8_2870X850X1420P, symbol TBLH10V-350-08BK:TBLH10V-350-08BK
Connections:
- net GND: now also J29.2, J30.1 (1_1), J30.2 (1_2)
- net NI9205A_AI0: now also J31.1, J31.2
- net NI9205A_AI1: now also J31.3, J31.4
- net NI9205A_AI2: now also J31.5, J31.6
- net NI9205A_AI3: now also J31.7, J31.8
- net NI9205A_AI4: now also J31.10, J31.9
- net NI9205A_AI5: now also J31.11, J31.12
- net NI9205A_AI6: now also J31.13, J31.14
- net NI9205A_AI7: now also J31.15, J31.16
- net NI9253_VSUP: now reaches J29.1
- net NI9253_VSUP: now also J29.4, J30.3 (2_1), J30.4 (2_2)

Commit message: kkkkkkkkkkkkkk
Parts:
- removed J29: NI9253CONN, symbol Connector:DB25_Socket
- removed J30: PWRCONN, WAGO 2601-1102:CONN2_2601-1102_WAG, symbol 2602_1102:2601-1102
- removed JX1: NI 9205 REF, symbol Connector_Generic:Conn_02x18_Counter_Clockwise
- removed JX2: JX2, symbol Connector_Generic:Conn_02x14_Counter_Clockwise
- added D1, D13, D2, D3, D4: LED, symbol Device:LED
- added D10, D11, D12, D14, D15, D16, D17, D18, D19, D20, D21, D5, D6, D7, D8, D9: 1N4004, Diode_THT:D_DO-41_SOD81_P7.62mm_Horizontal, symbol Diode:1N4004
- added F10, F11, F12, F13, F14, F15, F16, F17, F18, F19, F4, F5, F6, F7, F8, F9: Polyfuse, symbol Device:Polyfuse
- added H1, H2, H3, H4, H5, H6: MountingHole_Pad, MountingEquipment:DINRailAdapter_3xM3_PhoenixContact_1201578, symbol Mechanical:MountingHole_Pad
- added J29: NI9253CONN, symbol Connector:DA15_Pins_MountingHoles
- added J30, J40, J44: AICONN, TBLH10V-350-08BK:RHDR16W80P550X350_2X8_2870X850X1420P, symbol TBLH10V-350-08BK:TBLH10V-350-08BK
- added J32, J39, J43: PWRCONN, WAGO 2601-1102:CONN2_2601-1102_WAG, symbol 2602_1102:2601-1102
- added J33: NI9205CONN, Connector_Dsub:DSUB-37_Socket_Vertical_P2.77x2.84mm_MountingHoles, symbol Connector:DC37_Pins_MountingHoles
- added J34: LC0, CONN6_2601-3106_WAG, symbol 2601-3106:2601-3106
- added J35: LC1, CONN6_2601-3106_WAG, symbol 2601-3106:2601-3106
- added J36: LC2, CONN6_2601-3106_WAG, symbol 2601-3106:2601-3106
- added J37: LC3, CONN6_2601-3106_WAG, symbol 2601-3106:2601-3106
- added J38, J42: NI9485CONN, symbol Connector:DB25_Pins_MountingHoles
- added J41, J45: GNDCONN, TBLH10V-350-08BK:RHDR16W80P550X350_2X8_2870X850X1420P, symbol TBLH10V-350-08BK:TBLH10V-350-08BK
- added Q1: FQP27P06, Package_TO_SOT_THT:TO-220-3_Horizontal_TabDown, symbol Transistor_FET:FQP27P06
- added Q2, Q3, Q4, Q5: FQP27P06, Package_TO_SOT_THT:TO-220-3_Vertical, symbol Transistor_FET:FQP27P06
- added R1, R13, R2, R3, R4: R, symbol Device:R
- added R10, R11, R12, R14, R15, R16, R17, R18, R19, R20, R21, R5, R6, R7, R8, R9: 100K, Resistor_THT:R_Axial_DIN0207_L6.3mm_D2.5mm_P7.62mm_Horizontal, symbol Device:R
- J1, J15: symbol Connector:DC37_Socket_MountingHoles -> Connector:DC37_Pins_MountingHoles
- J11, J12, J19, J22, J25, J26, J5, J8: value GNDCONN -> AICONN
- J31: value GNDCONN -> VSUPCONN
Connections:
- net AI0: now also J29.3, J30.1, J30.2
- net AI1: now also J29.4, J30.3, J30.4
- net AI2: now also J29.5, J30.5, J30.6
- net AI3: now also J29.6, J30.7, J30.8
- net AI4: now also J29.7, J30.10, J30.9
- net AI5: now also J29.8, J30.11, J30.12
- net AI6: now also J29.10 (P10), J30.13, J30.14
- net AI7: now also J29.9 (P9), J30.15, J30.16
- net GND: now also D1.1 (K), D10.2 (A), D11.2 (A), D12.2 (A), D13.1 (K), D14.2 (A), D15.2 (A), D16.2 (A), D17.2 (A), D18.2 (A), D19.2 (A), D2.1 (K), D20.2 (A), D21.2 (A), D3.1 (K), D4.1 (K), D5.2 (A), D6.2 (A), D7.2 (A), D8.2 (A), D9.2 (A), H1.1, H2.1, H3.1, H4.1, H5.1, H6.1, J29.0 (PAD), J29.2, J32.1 (1_1), J32.2 (1_2), J38.0 (PAD), J39.1 (1_1), J39.2 (1_2), J41.1, J41.10, J41.11, J41.12, J41.13, J41.14, J41.15, J41.16, J41.2, J41.3, J41.4, J41.5, J41.6, J41.7, J41.8, J41.9, J42.0 (PAD), J43.1 (1_1), J43.2 (1_2), J45.1, J45.10, J45.11, J45.12, J45.13, J45.14, J45.15, J45.16, J45.2, J45.3, J45.4, J45.5, J45.6, J45.7, J45.8, J45.9, Q1.1 (G), Q2.1 (G), Q3.1 (G), Q4.1 (G), Q5.1 (G), R10.2, R11.2, R12.2, R14.2, R15.2, R16.2, R17.2, R18.2, R19.2, R20.2, R21.2, R5.2, R6.2, R7.2, R8.2, R9.2
- net NI9205A_AI0: no longer J31.1, J31.2
- net NI9205A_AI1: no longer J31.3, J31.4
- net NI9205A_AI2: no longer J31.5, J31.6
- net NI9205A_AI3: no longer J31.7, J31.8
- net NI9205A_AI4: no longer J31.10, J31.9
- net NI9205A_AI5: no longer J31.11, J31.12
- net NI9205A_AI6: no longer J31.13, J31.14
- net NI9205A_AI7: no longer J31.15, J31.16
- net VSUP: now also J31.1, J31.10, J31.11, J31.12, J31.13, J31.14, J31.15, J31.16, J31.2, J31.3, J31.4, J31.5, J31.6, J31.7, J31.8, J31.9, J29.1, R3.1
- removed net +24V: J13.1, J13.10, J13.11, J13.12, J13.13, J13.14, J13.15, J13.16, J13.2, J13.3, J13.4, J13.5, J13.6, J13.7, J13.8, J13.9, J16.3 (2_1), J16.4 (2_2), J17.1, J17.10, J17.11, J17.12, J17.13, J17.14, J17.15, J17.16, J17.2, J17.3, J17.4, J17.5, J17.6, J17.7, J17.8, J17.9, J2.3 (2_1), J2.4 (2_2), J20.1, J20.10, J20.11, J20.12, J20.13, J20.14, J20.15, J20.16, J20.2, J20.3, J20.4, J20.5, J20.6, J20.7, J20.8, J20.9, J23.1, J23.10, J23.11, J23.12, J23.13, J23.14, J23.15, J23.16, J23.2, J23.3, J23.4, J23.5, J23.6, J23.7, J23.8, J23.9, J27.1, J27.10, J27.11, J27.12, J27.13, J27.14, J27.15, J27.16, J27.2, J27.3, J27.4, J27.5, J27.6, J27.7, J27.8, J27.9, J3.1, J3.10, J3.11, J3.12, J3.13, J3.14, J3.15, J3.16, J3.2, J3.3, J3.4, J3.5, J3.6, J3.7, J3.8, J3.9, J6.1, J6.10, J6.11, J6.12, J6.13, J6.14, J6.15, J6.16, J6.2, J6.3, J6.4, J6.5, J6.6, J6.7, J6.8, J6.9, J9.1, J9.10, J9.11, J9.12, J9.13, J9.14, J9.15, J9.16, J9.2, J9.3, J9.4, J9.5, J9.6, J9.7, J9.8, J9.9
- new net: F8.1, J38.4
- new net: F11.1, J38.1
- new net: F10.1, J38.2
- new net: F9.1, J38.3
- new net: F7.1, J38.5
- new net: F6.1, J38.6
- new net: F5.1, J38.7
- new net: F4.1, J38.8
- new net: D13.2 (A), R13.2
- new net: D6.1 (K), R6.1
- new net: J32.3 (2_1), J32.4 (2_2), Q3.2 (D)
- new net: J16.3 (2_1), J16.4 (2_2), Q2.2 (D)
- new net: J39.3 (2_1), J39.4 (2_2), Q4.2 (D)
- new net: D1.2 (A), R1.2
- new net: F15.1, J42.5
- new net: D2.2 (A), R2.2
- new net: F12.1, J42.8
- new net: F18.1, J42.2
- new net: J43.3 (2_1), J43.4 (2_2), Q5.2 (D)
- new net: J2.3 (2_1), J2.4 (2_2), Q1.2 (D)
- new net: D4.2 (A), R4.2
- new net: F14.1, J42.6
- new net: D3.2 (A), R3.2
- new net: F16.1, J42.4
- new net: F13.1, J42.7
- new net: F17.1, J42.3
- new net: F19.1, J42.1
- new net EX0+: J33.2, J34.1 (1_1), J34.2 (1_2)
- new net EX0-: J33.21, J34.3 (2_1), J34.4 (2_2)
- new net EX1+: J33.6, J35.1 (1_1), J35.2 (1_2)
- new net EX1-: J33.25, J35.3 (2_1), J35.4 (2_2)
- new net EX2+: J33.12, J36.1 (1_1), J36.2 (1_2)
- new net EX2-: J33.31, J36.3 (2_1), J36.4 (2_2)
- new net EX3+: J33.16, J37.1 (1_1), J37.2 (1_2)
- new net EX3-: J33.35, J37.3 (2_1), J37.4 (2_2)
- new net NI9205A_PWR: J13.1, J13.10, J13.11, J13.12, J13.13, J13.14, J13.15, J13.16, J13.2, J13.3, J13.4, J13.5, J13.6, J13.7, J13.8, J13.9, J3.1, J3.10, J3.11, J3.12, J3.13, J3.14, J3.15, J3.16, J3.2, J3.3, J3.4, J3.5, J3.6, J3.7, J3.8, J3.9, J6.1, J6.10, J6.11, J6.12, J6.13, J6.14, J6.15, J6.16, J6.2, J6.3, J6.4, J6.5, J6.6, J6.7, J6.8, J6.9, J9.1, J9.10, J9.11, J9.12, J9.13, J9.14, J9.15, J9.16, J9.2, J9.3, J9.4, J9.5, J9.6, J9.7, J9.8, J9.9, Q1.3 (S), R1.1
- new net NI9205B_PWR: J17.1, J17.10, J17.11, J17.12, J17.13, J17.14, J17.15, J17.16, J17.2, J17.3, J17.4, J17.5, J17.6, J17.7, J17.8, J17.9, J20.1, J20.10, J20.11, J20.12, J20.13, J20.14, J20.15, J20.16, J20.2, J20.3, J20.4, J20.5, J20.6, J20.7, J20.8, J20.9, J23.1, J23.10, J23.11, J23.12, J23.13, J23.14, J23.15, J23.16, J23.2, J23.3, J23.4, J23.5, J23.6, J23.7, J23.8, J23.9, J27.1, J27.10, J27.11, J27.12, J27.13, J27.14, J27.15, J27.16, J27.2, J27.3, J27.4, J27.5, J27.6, J27.7, J27.8, J27.9, Q2.3 (S), Q3.3 (S), Q4.3 (S), Q5.3 (S), R2.1
- new net NI9237_AI0+: J33.3, J34.5 (3_1), J34.6 (3_2)
- new net NI9237_AI0-: J33.22, J34.7 (4_1), J34.8 (4_2)
- new net NI9237_AI1+: J33.7, J35.5 (3_1), J35.6 (3_2)
- new net NI9237_AI1-: J33.26, J35.7 (4_1), J35.8 (4_2)
- new net NI9237_AI2+: J33.13, J36.5 (3_1), J36.6 (3_2)
- new net NI9237_AI2-: J33.32, J36.7 (4_1), J36.8 (4_2)
- new net NI9237_AI3+: J33.17, J37.5 (3_1), J37.6 (3_2)
- new net NI9237_AI3-: J33.36, J37.7 (4_1), J37.8 (4_2)
- new net NI9485A_24V+: J38.14 (P14), J38.15 (P15), J38.16 (P16), J38.17 (P17), J38.18 (P18), J38.19 (P19), J38.20 (P20), J38.21 (P21), R4.1
- new net NI9485A_CH0B: D5.1 (K), F4.2, J40.1, J40.2, R5.1
- new net NI9485A_CH1B: F5.2, J40.3, J40.4
- new net NI9485A_CH2B: D7.1 (K), F6.2, J40.5, J40.6, R7.1
- new net NI9485A_CH3B: D8.1 (K), F7.2, J40.7, J40.8, R8.1
- new net NI9485A_CH4B: D9.1 (K), F8.2, J40.10, J40.9, R9.1
- new net NI9485A_CH5B: D10.1 (K), F9.2, J40.11, J40.12, R10.1
- new net NI9485A_CH6B: D11.1 (K), F10.2, J40.13, J40.14, R11.1
- new net NI9485A_CH7B: D12.1 (K), F11.2, J40.15, J40.16, R12.1
- new net NI9485B_24V+: J42.14 (P14), J42.15 (P15), J42.16 (P16), J42.17 (P17), J42.18 (P18), J42.19 (P19), J42.20 (P20), J42.21 (P21), R13.1
- new net NI9485B_CH0B: D14.1 (K), F12.2, J44.1, J44.2, R14.1
- new net NI9485B_CH1B: D15.1 (K), F13.2, J44.3, J44.4, R15.1
- new net NI9485B_CH2B: D16.1 (K), F14.2, J44.5, J44.6, R16.1
- new net NI9485B_CH3B: D17.1 (K), F15.2, J44.7, J44.8, R17.1
- new net NI9485B_CH4B: D18.1 (K), F16.2, J44.10, J44.9, R18.1
- new net NI9485B_CH5B: D19.1 (K), F17.2, J44.11, J44.12, R19.1
- new net NI9485B_CH6B: D20.1 (K), F18.2, J44.13, J44.14, R20.1
- new net NI9485B_CH7B: D21.1 (K), F19.2, J44.15, J44.16, R21.1
- new net RS0+: J33.1, J34.10 (5_2), J34.9 (5_1)
- new net RS0-: J33.20, J34.11 (6_1), J34.12 (6_2)
- new net RS1+: J33.5, J35.10 (5_2), J35.9 (5_1)
- new net RS1-: J33.24, J35.11 (6_1), J35.12 (6_2)
- new net RS2+: J33.11, J36.10 (5_2), J36.9 (5_1)
- new net RS2-: J33.30, J36.11 (6_1), J36.12 (6_2)
- new net RS3+: J33.15, J37.10 (5_2), J37.9 (5_1)
- new net RS3-: J33.34, J37.11 (6_1), J37.12 (6_2)
- no-connect marks 4 -> 39
Other:
- note added: "NI 9205 A SCHEMATIC (V_AI)"
- note added: "NI 9205 B SCHEMATIC (V_AI)"
- note added: "NI 9237 SCHEMATIC (LC_AI)"
- note added: "NI 9253 SCHEMATIC (C_AI)"
- note added: "NI 9485 A SCHEMATIC (RELAY)"
- note added: "NI 9485 B SCHEMATIC (RELAY)"
- note removed: "NI 9205 A SCHEMATIC"
- note removed: "NI 9205 B SCHEMATIC"
- moved on the sheet: J11, J12, J13, J14, J16, J17, J2, J20, J21, J22, J24, J26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

Commit message: KID
Parts:
- removed D2: LED, symbol Device:LED
- removed F18, F19: Polyfuse, symbol Device:Polyfuse
- removed J16: PWRCONN, WAGO 2601-1102:CONN2_2601-1102_WAG, symbol 2602_1102:2601-1102
- removed Q2: FQP27P06, Package_TO_SOT_THT:TO-220-3_Vertical, symbol Transistor_FET:FQP27P06
- removed R2: R, symbol Device:R
- added F1: 0ZCF0100AF2A, Fuse:Fuse_2920_7451Metric_Pad2.10x5.45mm_HandSolder, symbol Device:Polyfuse
- added F3, F4: 0ZRP0065FF1E, Fuse:Fuse_Bourns_MF-RG300, symbol Device:Polyfuse
- added TP1, TP10, TP11, TP12, TP13, TP14, TP15, TP16, TP17, TP18, TP19, TP2, TP20, TP21, TP22, TP23, TP24, TP25, TP26, TP27, TP28, TP29, TP3, TP30, TP31, TP32, TP33, TP34, TP35, TP36, TP37, TP38, TP39, TP4, TP40, TP41, TP42, TP43, TP44, TP45, TP46, TP47, TP48, TP49, TP5, TP50, TP51, TP52, TP53, TP54, TP55, TP56, TP57, TP58, TP59, TP6, TP60, TP61, TP62, TP63, TP64, TP65, TP66, TP67, TP68, TP69, TP7, TP70, TP71, TP72, TP73, TP74, TP75, TP76, TP77, TP78, TP79, TP8, TP80, TP81, TP82, TP83, TP84, TP85, TP86, TP87, TP88, TP9: TestPoint, TestPoint:TestPoint_THTPad_D2.0mm_Drill1.0mm, symbol Connector:TestPoint
- D1: footprint (none) -> LED_THT:LED_D3.0mm
- D12: renamed from D13; footprint (none) -> LED_THT:LED_D3.0mm
- D2: renamed from D3; footprint (none) -> LED_THT:LED_D3.0mm
- D7: renamed from D4; footprint (none) -> LED_THT:LED_D3.0mm
- F10, F11, F12, F13, F14, F15, F16, F17, F5, F6, F7, F8, F9: value Polyfuse -> 0ZRP0065FF1E; footprint (none) -> Fuse:Fuse_Bourns_MF-RG300
- F2: renamed from F4; value Polyfuse -> 0ZRP0065FF1E; footprint (none) -> Fuse:Fuse_Bourns_MF-RG300
- H1, H2, H3, H4, H5, H6: footprint MountingEquipment:DINRailAdapter_3xM3_PhoenixContact_1201578 -> MountingHole:MountingHole_3.2mm_M3_DIN965_Pad_TopBottom
- J1, J15: footprint Connector_Dsub:DSUB-37_Socket_Vertical_P2.77x2.84mm_MountingHoles -> Connector_Dsub:DSUB-37_Pins_Vertical_P2.77x2.84mm_MountingHoles
- J29: footprint (none) -> Connector_Dsub:DSUB-15_Pins_Vertical_P2.77x2.84mm_MountingHoles
- J33: value NI9205CONN -> NI9237CONN; footprint Connector_Dsub:DSUB-37_Socket_Vertical_P2.77x2.84mm_MountingHoles -> Connector_Dsub:DSUB-37_Pins_Vertical_P2.77x2.84mm_MountingHoles
- J34, J35, J36, J37: footprint CONN6_2601-3106_WAG -> 2601-3106:CONN6_2601-3106_WAG
- J38, J42: footprint (none) -> Connector_Dsub:DSUB-25_Pins_Vertical_P2.77x2.84mm_MountingHoles
- Q2: renamed from Q3; footprint Package_TO_SOT_THT:TO-220-3_Vertical -> Package_TO_SOT_THT:TO-220-3_Horizontal_TabDown
- Q3: renamed from Q4; footprint Package_TO_SOT_THT:TO-220-3_Vertical -> Package_TO_SOT_THT:TO-220-3_Horizontal_TabDown
- Q4: renamed from Q5; footprint Package_TO_SOT_THT:TO-220-3_Vertical -> Package_TO_SOT_THT:TO-220-3_Horizontal_TabDown
- R1, R4: value R -> 1.1k; footprint (none) -> Resistor_THT:R_Axial_DIN0207_L6.3mm_D2.5mm_P7.62mm_Horizontal
- R12: renamed from R13; value R -> 1.1k; footprint (none) -> Resistor_THT:R_Axial_DIN0207_L6.3mm_D2.5mm_P7.62mm_Horizontal
- R2: renamed from R3; value R -> 1.1k; footprint (none) -> Resistor_THT:R_Axial_DIN0207_L6.3mm_D2.5mm_P7.62mm_Horizontal
- renumbered D11 to D10, D12 to D11, D14 to D13, D15 to D14, D16 to D15, D17 to D16, D18 to D17, D19 to D18, D20 to D19, D21 to D20, D5 to D3, D6 to D4, D7 to D5, D8 to D6, D9 to D8, D10 to D9, R11 to R10, R12 to R11, R14 to R13, R15 to R14, R16 to R15, R17 to R16, R18 to R17, R19 to R18, R20 to R19, R21 to R20, R5 to R3, R6 to R5, R7 to R6, R8 to R7, R9 to R8, R10 to R9
Connections:
- net EX0+: now also J34.5 (3_1), J34.6 (3_2); no longer J34.1 (1_1), J34.2 (1_2)
- net EX0-: now also J34.7 (4_1), J34.8 (4_2); no longer J34.3 (2_1), J34.4 (2_2)
- net EX1+: now also J35.5 (3_1), J35.6 (3_2); no longer J35.1 (1_1), J35.2 (1_2)
- net EX1-: now also J35.7 (4_1), J35.8 (4_2); no longer J35.3 (2_1), J35.4 (2_2)
- net EX2+: now also J36.7 (4_1), J36.8 (4_2); no longer J36.1 (1_1), J36.2 (1_2)
- net EX2-: now also J36.5 (3_1), J36.6 (3_2); no longer J36.3 (2_1), J36.4 (2_2)
- net EX3+: now also J37.7 (4_1), J37.8 (4_2); no longer J37.1 (1_1), J37.2 (1_2)
- net EX3-: now also J37.5 (3_1), J37.6 (3_2); no longer J37.3 (2_1), J37.4 (2_2)
- net GND: now also TP2.1, TP68.1, TP70.1, TP80.1
- net NI9205A_AI0: now also TP3.1
- net NI9205A_AI1: now also TP4.1
- net NI9205A_AI10: now also TP13.1
- net NI9205A_AI11: now also TP14.1
- net NI9205A_AI12: now also TP15.1
- net NI9205A_AI13: now also TP16.1
- net NI9205A_AI14: now also TP17.1
- net NI9205A_AI15: now also TP18.1
- net NI9205A_AI16: now also TP19.1
- net NI9205A_AI17: now also TP20.1
- net NI9205A_AI18: now also TP21.1
- net NI9205A_AI19: now also TP22.1
- net NI9205A_AI2: now also TP5.1
- net NI9205A_AI20: now also TP23.1
- net NI9205A_AI21: now also TP24.1
- net NI9205A_AI22: now also TP25.1
- net NI9205A_AI23: now also TP26.1
- net NI9205A_AI24: now also TP27.1
- net NI9205A_AI25: now also TP28.1
- net NI9205A_AI26: now also TP29.1
- net NI9205A_AI27: now also TP30.1
- net NI9205A_AI28: now also TP31.1
- net NI9205A_AI29: now also TP32.1
- net NI9205A_AI3: now also TP6.1
- net NI9205A_AI30: now also TP33.1
- net NI9205A_AI31: now also TP34.1
- net NI9205A_AI4: now also TP7.1
- net NI9205A_AI5: now also TP8.1
- net NI9205A_AI6: now also TP9.1
- net NI9205A_AI7: now also TP10.1
- net NI9205A_AI8: now also TP11.1
- net NI9205A_AI9: now also TP12.1
- net NI9205B_AI0: now also TP35.1
- net NI9205B_AI1: now also TP36.1
- net NI9205B_AI10: now also TP45.1
- net NI9205B_AI11: now also TP46.1
- net NI9205B_AI12: now also TP47.1
- net NI9205B_AI13: now also TP48.1
- net NI9205B_AI14: now also TP49.1
- net NI9205B_AI15: now also TP50.1
- net NI9205B_AI16: now also TP51.1
- net NI9205B_AI17: now also TP52.1
- net NI9205B_AI18: now also TP53.1
- net NI9205B_AI19: now also TP54.1
- net NI9205B_AI2: now also TP37.1
- net NI9205B_AI20: now also TP55.1
- net NI9205B_AI21: now also TP56.1
- net NI9205B_AI22: now also TP57.1
- net NI9205B_AI23: now also TP58.1
- net NI9205B_AI24: now also TP59.1
- net NI9205B_AI25: now also TP60.1
- net NI9205B_AI26: now also TP61.1
- net NI9205B_AI27: now also TP62.1
- net NI9205B_AI28: now also TP63.1
- net NI9205B_AI29: now also TP64.1
- net NI9205B_AI3: now also TP38.1
- net NI9205B_AI30: now also TP65.1
- net NI9205B_AI31: now also TP66.1
- net NI9205B_AI4: now also TP39.1
- net NI9205B_AI5: now also TP40.1
- net NI9205B_AI6: now also TP41.1
- net NI9205B_AI7: now also TP42.1
- net NI9205B_AI8: now also TP43.1
- net NI9205B_AI9: now also TP44.1
- net NI9237_AI0+: now also J34.10 (5_2), J34.9 (5_1); no longer J34.5 (3_1), J34.6 (3_2)
- net NI9237_AI0-: now also J34.11 (6_1), J34.12 (6_2); no longer J34.7 (4_1), J34.8 (4_2)
- net NI9237_AI1+: now also J35.10 (5_2), J35.9 (5_1); no longer J35.5 (3_1), J35.6 (3_2)
- net NI9237_AI1-: now also J35.11 (6_1), J35.12 (6_2); no longer J35.7 (4_1), J35.8 (4_2)
- net NI9237_AI2+: now also J36.3 (2_1), J36.4 (2_2); no longer J36.5 (3_1), J36.6 (3_2)
- net NI9237_AI2-: now also J36.1 (1_1), J36.2 (1_2); no longer J36.7 (4_1), J36.8 (4_2)
- net NI9237_AI3+: now also J37.3 (2_1), J37.4 (2_2); no longer J37.5 (3_1), J37.6 (3_2)
- net NI9237_AI3-: now also J37.1 (1_1), J37.2 (1_2); no longer J37.7 (4_1), J37.8 (4_2)
- net NI9485A_24V+: now also Q3.3 (S), TP69.1
- net NI9485A_CH0B: now also TP71.1
- net NI9485A_CH1B: now also F3.2, TP72.1; no longer F5.2
- net NI9485A_CH2B: now also F4.2, TP73.1; no longer F6.2
- net NI9485A_CH3B: now also F5.2, TP74.1; no longer F7.2
- net NI9485A_CH4B: now also F6.2, TP75.1; no longer F8.2
- net NI9485A_CH5B: now also F7.2, TP76.1; no longer F9.2
- net NI9485A_CH6B: now also F8.2, TP77.1; no longer F10.2
- net NI9485A_CH7B: now also F9.2, TP78.1; no longer F11.2
- net NI9485B_24V+: now also Q4.3 (S), TP79.1
- net NI9485B_CH0B: now also F10.2, TP81.1; no longer F12.2
- net NI9485B_CH1B: now also F11.2, TP82.1; no longer F13.2
- net NI9485B_CH2B: now also F12.2, TP83.1; no longer F14.2
- net NI9485B_CH3B: now also F13.2, TP84.1; no longer F15.2
- net NI9485B_CH4B: now also F14.2, TP85.1; no longer F16.2
- net NI9485B_CH5B: now also F15.2, TP86.1; no longer F17.2
- net NI9485B_CH6B: now also F16.2, TP87.1
- net NI9485B_CH7B: now also F17.2, TP88.1
- net RS0+: now also J34.1 (1_1), J34.2 (1_2); no longer J34.10 (5_2), J34.9 (5_1)
- net RS0-: now also J34.3 (2_1), J34.4 (2_2); no longer J34.11 (6_1), J34.12 (6_2)
- net RS1+: now also J35.1 (1_1), J35.2 (1_2); no longer J35.10 (5_2), J35.9 (5_1)
- net RS1-: now also J35.3 (2_1), J35.4 (2_2); no longer J35.11 (6_1), J35.12 (6_2)
- net RS2+: now also J36.11 (6_1), J36.12 (6_2); no longer J36.10 (5_2), J36.9 (5_1)
- net RS2-: now also J36.10 (5_2), J36.9 (5_1); no longer J36.11 (6_1), J36.12 (6_2)
- net RS3+: now also J37.11 (6_1), J37.12 (6_2); no longer J37.10 (5_2), J37.9 (5_1)
- net RS3-: now also J37.10 (5_2), J37.9 (5_1); no longer J37.11 (6_1), J37.12 (6_2)
- net VSUP: now also F1.2, TP67.1
- net at F8.1: now also J38.2; no longer J38.4
- net at J38.1: now also F9.1; no longer F11.1
- net at F10.1: now also J42.8; no longer J38.2
- net at J38.3: now also F7.1; no longer F9.1
- net at J38.5: now also F5.1; no longer F7.1
- net at F6.1: now also J38.4; no longer J38.6
- net at J38.7: now also F3.1; no longer F5.1
- net at J42.5: now also F13.1; no longer F15.1
- net at F12.1: now also J42.6; no longer J42.8
- net at J42.2: now also F16.1
- net at F14.1: now also J42.4; no longer J42.6
- net at J42.7: now also F11.1; no longer F13.1
- net at J42.3: now also F15.1; no longer F17.1
- net at J42.1: now also F17.1
- net NI9205A_PWR renamed NI9205_PWR
- net NI9205_PWR: now also J17.1, J17.10, J17.11, J17.12, J17.13, J17.14, J17.15, J17.16, J17.2, J17.3, J17.4, J17.5, J17.6, J17.7, J17.8, J17.9, J20.1, J20.10, J20.11, J20.12, J20.13, J20.14, J20.15, J20.16, J20.2, J20.3, J20.4, J20.5, J20.6, J20.7, J20.8, J20.9, J23.1, J23.10, J23.11, J23.12, J23.13, J23.14, J23.15, J23.16, J23.2, J23.3, J23.4, J23.5, J23.6, J23.7, J23.8, J23.9, J27.1, J27.10, J27.11, J27.12, J27.13, J27.14, J27.15, J27.16, J27.2, J27.3, J27.4, J27.5, J27.6, J27.7, J27.8, J27.9, TP1.1
- removed net NI9205B_PWR: J17.1, J17.10, J17.11, J17.12, J17.13, J17.14, J17.15, J17.16, J17.2, J17.3, J17.4, J17.5, J17.6, J17.7, J17.8, J17.9, J20.1, J20.10, J20.11, J20.12, J20.13, J20.14, J20.15, J20.16, J20.2, J20.3, J20.4, J20.5, J20.6, J20.7, J20.8, J20.9, J23.1, J23.10, J23.11, J23.12, J23.13, J23.14, J23.15, J23.16, J23.2, J23.3, J23.4, J23.5, J23.6, J23.7, J23.8, J23.9, J27.1, J27.10, J27.11, J27.12, J27.13, J27.14, J27.15, J27.16, J27.2, J27.3, J27.4, J27.5, J27.6, J27.7, J27.8, J27.9, Q2.3 (S), Q3.3 (S), Q4.3 (S)
- new net: F4.1, J38.6
- new net: F1.1, Q2.3 (S)

Commit message: Aaahaha
Parts:
- added D2: LED, LED_THT:LED_D3.0mm, symbol Device:LED
- added J16: PWRCONN, WAGO 2601-1102:CONN2_2601-1102_WAG, symbol 2602_1102:2601-1102
- added Q2: FQP27P06, Package_TO_SOT_THT:TO-220-3_Horizontal_TabDown, symbol Transistor_FET:FQP27P06
- added R2: 1.1k, Resistor_THT:R_Axial_DIN0207_L6.3mm_D2.5mm_P7.62mm_Horizontal, symbol Device:R
- added TP89, TP90: TestPoint, TestPoint:TestPoint_THTPad_D2.0mm_Drill1.0mm, symbol Connector:TestPoint
- renumbered D9 to D10, D10 to D11, D11 to D12, D12 to D13, D13 to D14, D14 to D15, D15 to D16, D16 to D17, D17 to D18, D18 to D19, D19 to D20, D20 to D21, D2 to D3, D7 to D4, D3 to D5, D4 to D6, D5 to D7, D6 to D8, D8 to D9, Q2 to Q3, Q3 to Q4, Q4 to Q5, R9 to R10, R10 to R11, R11 to R12, R12 to R13, R13 to R14, R14 to R15, R15 to R16, R16 to R17, R17 to R18, R18 to R19, R19 to R20, R20 to R21, R2 to R3, R3 to R5, R5 to R6, R6 to R7, R7 to R8, R8 to R9
Connections:
- net GND: now also D2.1 (K), J16.1 (1_1), J16.2 (1_2), Q2.1 (G), TP90.1
- net NI9205_PWR renamed NI9205A_PWR
- net NI9205A_PWR: no longer J17.1, J17.10, J17.11, J17.12, J17.13, J17.14, J17.15, J17.16, J17.2, J17.3, J17.4, J17.5, J17.6, J17.7, J17.8, J17.9, J20.1, J20.10, J20.11, J20.12, J20.13, J20.14, J20.15, J20.16, J20.2, J20.3, J20.4, J20.5, J20.6, J20.7, J20.8, J20.9, J23.1, J23.10, J23.11, J23.12, J23.13, J23.14, J23.15, J23.16, J23.2, J23.3, J23.4, J23.5, J23.6, J23.7, J23.8, J23.9, J27.1, J27.10, J27.11, J27.12, J27.13, J27.14, J27.15, J27.16, J27.2, J27.3, J27.4, J27.5, J27.6, J27.7, J27.8, J27.9
- new net: J16.3 (2_1), J16.4 (2_2), Q2.2 (D)
- new net: D2.2 (A), R2.2
- new net NI9205B_PWR: J17.1, J17.10, J17.11, J17.12, J17.13, J17.14, J17.15, J17.16, J17.2, J17.3, J17.4, J17.5, J17.6, J17.7, J17.8, J17.9, J20.1, J20.10, J20.11, J20.12, J20.13, J20.14, J20.15, J20.16, J20.2, J20.3, J20.4, J20.5, J20.6, J20.7, J20.8, J20.9, J23.1, J23.10, J23.11, J23.12, J23.13, J23.14, J23.15, J23.16, J23.2, J23.3, J23.4, J23.5, J23.6, J23.7, J23.8, J23.9, J27.1, J27.10, J27.11, J27.12, J27.13, J27.14, J27.15, J27.16, J27.2, J27.3, J27.4, J27.5, J27.6, J27.7, J27.8, J27.9, Q2.3 (S), R2.1, TP89.1

Commit message: AGS PCBS
Parts:
- added H10, H11, H12, H13, H14, H15, H16, H17, H18, H19, H20, H21, H22, H23, H24, H25, H26, H27, H28, H29, H30, H7, H8, H9: MountingHole_Pad, MountingHole:MountingHole_3.2mm_M3_DIN965_Pad_TopBottom, symbol Mechanical:MountingHole_Pad
- added J46: NI_9485A_D-SUB, Connector_Dsub:DSUB-9_Pins_Vertical_P2.77x2.84mm_MountingHoles, symbol Connector:DE9_Pins_MountingHoles
- added J47: NI_9485B_D-SUB, Connector_Dsub:DSUB-9_Pins_Vertical_P2.77x2.84mm_MountingHoles, symbol Connector:DE9_Pins_MountingHoles
Connections:
- net EX2+: now also J36.5 (3_1), J36.6 (3_2); no longer J36.7 (4_1), J36.8 (4_2)
- net EX2-: now also J36.7 (4_1), J36.8 (4_2); no longer J36.5 (3_1), J36.6 (3_2)
- net EX3+: now also J37.5 (3_1), J37.6 (3_2); no longer J37.7 (4_1), J37.8 (4_2)
- net EX3-: now also J37.7 (4_1), J37.8 (4_2); no longer J37.5 (3_1), J37.6 (3_2)
- net GND: now also H10.1, H11.1, H12.1, H13.1, H14.1, H15.1, H16.1, H17.1, H18.1, H19.1, H20.1, H21.1, H22.1, H23.1, H24.1, H25.1, H26.1, H27.1, H28.1, H29.1, H30.1, H7.1, H8.1, H9.1, J46.0 (PAD), J46.9, J47.0 (PAD), J47.9
- net NI9237_AI2+: now also J36.10 (5_2), J36.9 (5_1); no longer J36.3 (2_1), J36.4 (2_2)
- net NI9237_AI2-: now also J36.11 (6_1), J36.12 (6_2); no longer J36.1 (1_1), J36.2 (1_2)
- net NI9237_AI3+: now also J37.10 (5_2), J37.9 (5_1); no longer J37.3 (2_1), J37.4 (2_2)
- net NI9237_AI3-: now also J37.11 (6_1), J37.12 (6_2); no longer J37.1 (1_1), J37.2 (1_2)
- net NI9485A_CH0B: now also J46.1
- net NI9485A_CH1B: now also D6.1 (K), R6.1, J46.2
- net NI9485A_CH2B: now also J46.3
- net NI9485A_CH3B: now also J46.4
- net NI9485A_CH4B: now also J46.5
- net NI9485A_CH5B: now also J46.6
- net NI9485A_CH6B: now also J46.7
- net NI9485A_CH7B: now also J46.8
- net NI9485B_CH0B: now also J47.1
- net NI9485B_CH1B: now also J47.2
- net NI9485B_CH2B: now also J47.3
- net NI9485B_CH3B: now also J47.4
- net NI9485B_CH4B: now also J47.5
- net NI9485B_CH5B: now also J47.6
- net NI9485B_CH6B: now also J47.7
- net NI9485B_CH7B: now also J47.8
- net RS2+: now also J36.1 (1_1), J36.2 (1_2); no longer J36.11 (6_1), J36.12 (6_2)
- net RS2-: now also J36.3 (2_1), J36.4 (2_2); no longer J36.10 (5_2), J36.9 (5_1)
- net RS3+: now also J37.1 (1_1), J37.2 (1_2); no longer J37.11 (6_1), J37.12 (6_2)
- net RS3-: now also J37.3 (2_1), J37.4 (2_2); no longer J37.10 (5_2), J37.9 (5_1)
- net V_IN_A: now reaches J39.3 (2_1), J39.4 (2_2), Q4.2 (D)
- net V_IN_B: now reaches J43.3 (2_1), J43.4 (2_2), Q5.2 (D)
Other:
- moved on the sheet: H1, H2, H3, H4, H5, H6, TP1, TP10, TP11, TP12, TP13, TP14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

Commit message: Producation files
Parts:
- added H31, H32, H33, H34: MountingHole_Pad, MountingHole:MountingHole_3.2mm_M3_DIN965_Pad_TopBottom, symbol Mechanical:MountingHole_Pad
Connections:
- net GND: no longer H1.1, H10.1, H11.1, H12.1, H13.1, H14.1, H15.1, H16.1, H17.1, H18.1, H19.1, H2.1, H20.1, H21.1, H22.1, H23.1, H24.1, H25.1, H26.1, H27.1, H28.1, H29.1, H3.1, H30.1, H4.1, H5.1, H6.1, H7.1, H8.1, H9.1
- no-connect marks 39 -> 73
