File: AGS Solenoid Breakout D9/AGS Solenoid Breakout D9.kicad_pcb (KiCad board)
At the start: 2 copper layers, 50.8 x 63.5 mm, 24 parts, among them J1 DB9_INPUT, J2 SOL. CHANS., J3 SOL. CHANS.

Commit message: Producation files
Parts:
- removed the G*** at (51.9, 62.6)
- added G***: LOGO, LOGO, B.Cu at (50.9, 62.5)
