File: Test Stand Limit Switch/Test Stand Limit Switch.kicad_sch (KiCad schematic)
At the start: 4 parts, among them J1 PIN_OUT, SW1 SW_SPDT_312

Commit message: AGS PCBS
Parts:
- removed D1: LED, symbol Device:LED
- removed J1: PIN_OUT, symbol Connector:Conn_01x03_Pin
- removed SW1: SW_SPDT_312, symbol Switch:SW_SPDT_312
- added C1: .33uF, Capacitor_THT:C_Disc_D5.0mm_W2.5mm_P2.50mm, symbol Device:C
- added C2: .1uF, Capacitor_THT:C_Disc_D5.0mm_W2.5mm_P2.50mm, symbol Device:C
- added D1: 1N4004, Diode_THT:D_DO-41_SOD81_P7.62mm_Horizontal, symbol Diode:1N4004
- added D2: RED, LED_THT:LED_D3.0mm, symbol Device:LED
- added H1, H2: MountingHole_Pad, MountingHole:MountingHole_3.2mm_M3_DIN965_Pad_TopBottom, symbol Mechanical:MountingHole_Pad
- added J1: IN, TerminalBlock_Phoenix:TerminalBlock_Phoenix_PT-1,5-3-3.5-H_1x03_P3.50mm_Horizontal, symbol Connector:Screw_Terminal_01x03
- added R2: 10K, Resistor_THT:R_Axial_DIN0207_L6.3mm_D2.5mm_P7.62mm_Horizontal, symbol Device:R
- added R3: 12K, Resistor_THT:R_Axial_DIN0207_L6.3mm_D2.5mm_P7.62mm_Horizontal, symbol Device:R
- added R4: 6.6K, Resistor_THT:R_Axial_DIN0207_L6.3mm_D2.5mm_P7.62mm_Horizontal, symbol Device:R
- added R5: 1.7K, Resistor_THT:R_Axial_DIN0207_L6.3mm_D2.5mm_P7.62mm_Horizontal, symbol Device:R
- added SW1: OPEN, TerminalBlock_Phoenix:TerminalBlock_Phoenix_PT-1,5-3-3.5-H_1x03_P3.50mm_Horizontal, symbol Switch:SW_SPDT
- added SW2: CLOSE, TerminalBlock_Phoenix:TerminalBlock_Phoenix_PT-1,5-3-3.5-H_1x03_P3.50mm_Horizontal, symbol Switch:SW_SPDT
- added U1: L78L09_TO92, Package_TO_SOT_THT:TO-92L_Inline, symbol Regulator_Linear:L78L09_TO92
- R1: value R -> 1.1K; footprint (none) -> Resistor_THT:R_Axial_DIN0207_L6.3mm_D2.5mm_P7.62mm_Horizontal
Connections:
- net GND: now also C1.2, C2.2, D2.1 (K), J1.2 (Pin_2), R3.2, R4.2, R5.2, U1.2 (GND)
- net SIGNAL: now also J1.1 (Pin_1), R2.2, R3.1, SW1.2 (B), SW2.2 (B)
- net +9V: now reaches R1.1
- net +9V: now also C2.1, R2.1, U1.1 (VO)
- net +24V: no longer names the net of R1.2
- net +24V: now also D2.2 (A)
- new net: R5.1, SW2.3 (C)
- new net: D1.2 (A), J1.3 (Pin_3)
- new net: R4.1, SW1.3 (C)
- new net VCC: C1.1, D1.1 (K), U1.3 (VI)
- no-connect marks 0 -> 4
Other:
- note added: "9V OUT LDO 30V Max V IN 100mA Max Out"
- note added: "Operating Circuitry"
- note added: "Power LED"
- note added: "Terminal In"
- note added: "~1 volt = Valve Close"
- note added: "~3 volts = Valve Open"
- note added: "~5 volts = Valve Moving"
- note removed: "PIN OUT"
- note removed: "PWR LED"

Commit message: Stuff
Parts:
- R4: value 6.6K -> 6.8k
- R5: value 1.7K -> 1.5k
Changed lines of the file:
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@@
 			)
 		)
-		(property "Value" "1.7K"
+		(property "Value" "1.5k"
 			(at 146.05 67.3099 0)
 			(effects
@@
 			)
 		)
-		(property "Value" "6.6K"
+		(property "Value" "6.8k"
 			(at 130.81 67.3099 0)
 			(effects
